File: simulation/vco/vco.sch (KiCad schematic (older format))
At the start: 43 parts, among them Q1 BC546, Q2 BC546, Q3 BC546, Q4 BC546, U1 LM324, U2 LM324, U3 LM324, U4 LM324, U5 LM324, U6 LM324, U7 LM324, U8 LM324

Commit message: vco: adapt sawtooth generation to actual ciruitry on the breadboard
Parts:
- V2: value 2 -> 4
Connections:
- net GNDREF: now also Q2.3 (E); no longer R13.1
- net triangle: now also R13.2; no longer Q2.1 (C)
- new net: Q2.1 (C), R13.1, U4.1 (+)
Other:
- moved on the sheet: Q2, R10, R13
Changed lines of the file:
@@
 $EndComp
-Wire Wire Line
-	4700 5400 4650 5400
 Wire Wire Line
 	4600 5200 4650 5200
@@
 Wire Wire Line
 	4150 5200 4300 5200
-Wire Wire Line
-	4400 5900 4400 5400
 $Comp
 L power:GNDREF #PWR012
 U 1 1 5CF85DC5
-P 4650 5700
-F 0 "#PWR012" H 4650 5450 50  0001 C CNN
-F 1 "GNDREF" H 4655 5527 50  0001 C CNN
-F 2 "" H 4650 5700 50  0001 C CNN
-F 3 "" H 4650 5700 50  0001 C CNN
-	1    4650 5700
+P 4650 6100
+F 0 "#PWR012" H 4650 5850 50  0001 C CNN
+F 1 "GNDREF" H 4655 5927 50  0001 C CNN
+F 2 "" H 4650 6100 50  0001 C CNN
+F 3 "" H 4650 6100 50  0001 C CNN
+	1    4650 6100
 	-1   0    0    -1
 $EndComp
@@
 L Device:R R13
 U 1 1 5CF81086
-P 4650 5550
-F 0 "R13" V 4550 5550 50  0000 C CNN
-F 1 "100k" V 4650 5550 50  0000 C CNN
-F 2 "" V 4580 5550 50  0001 C CNN
-F 3 "~" H 4650 5550 50  0001 C CNN
-	1    4650 5550
-	1    0    0    1
-$EndComp
-Wire Wire Line
-	4150 5900 4400 5900
-Connection ~ 4650 5400
-Wire Wire Line
-	4650 5400 4400 5400
-Wire Wire Line
-	3700 5550 3600 5550
+P 4450 5400
+F 0 "R13" V 4350 5400 50  0000 C CNN
+F 1 "100k" V 4450 5400 50  0000 C CNN
+F 2 "" V 4380 5400 50  0001 C CNN
+F 3 "~" H 4450 5400 50  0001 C CNN
+	1    4450 5400
+	0    1    -1   0
+$EndComp
 Text GLabel 5700 5300 2    50   Input ~ 0
 sawtooth
@@
 Connection ~ 5400 5300
 Wire Wire Line
-	3500 6300 3600 6300
-Wire Wire Line
-	3600 5550 3600 5750
-Wire Wire Line
-	3600 6050 3600 6300
-Connection ~ 3600 6300
-Wire Wire Line
-	3600 6300 5650 6300
+	3500 6300 3800 6300
+Wire Wire Line
+	3800 6150 3800 6300
+Connection ~ 3800 6300
+Wire Wire Line
+	3800 6300 5650 6300
 $Comp
 L pspice:QNPN Q2
 U 1 1 5CF6A60E
-P 4000 5550
-F 0 "Q2" H 3700 5850 50  0000 L CNN
-F 1 "BC546" H 3700 5750 50  0000 L CNN
-F 2 "" H 4000 5550 50  0001 C CNN
-F 3 "~" H 4000 5550 50  0001 C CNN
-F 4 "Q" H 4000 5550 50  0001 C CNN "Spice_Primitive"
-F 5 "BC546B" H 4000 5550 50  0001 C CNN "Spice_Model"
-F 6 "Y" H 4000 5550 50  0001 C CNN "Spice_Netlist_Enabled"
-F 7 "BC546.lib" H 4000 5550 50  0001 C CNN "Spice_Lib_File"
-	1    4000 5550
+P 4500 5750
+F 0 "Q2" H 4200 5600 50  0000 L CNN
+F 1 "BC546" H 4050 5500 50  0000 L CNN
+F 2 "" H 4500 5750 50  0001 C CNN
+F 3 "~" H 4500 5750 50  0001 C CNN
+F 4 "Q" H 4500 5750 50  0001 C CNN "Spice_Primitive"
+F 5 "BC546B" H 4500 5750 50  0001 C CNN "Spice_Model"
+F 6 "Y" H 4500 5750 50  0001 C CNN "Spice_Netlist_Enabled"
+F 7 "BC546.lib" H 4500 5750 50  0001 C CNN "Spice_Lib_File"
+	1    4500 5750
 	1    0    0    -1
 $EndComp
 Wire Wire Line
 	4150 5200 4150 4650
-Connection ~ 4150 5200
 Connection ~ 4150 4650
 Wire Wire Line
@@
 L Device:R R10
 U 1 1 5CF9A0F2
-P 3600 5900
-F 0 "R10" V 3500 5900 50  0000 C CNN
-F 1 "10k" V 3600 5900 50  0000 C CNN
-F 2 "" V 3530 5900 50  0001 C CNN
-F 3 "~" H 3600 5900 50  0001 C CNN
-	1    3600 5900
+P 3800 6000
+F 0 "R10" V 3700 6000 50  0000 C CNN
+F 1 "10k" V 3800 6000 50  0000 C CNN
+F 2 "" V 3730 6000 50  0001 C CNN
+F 3 "~" H 3800 6000 50  0001 C CNN
+	1    3800 6000
 	1    0    0    -1
 $EndComp
@@
 P 7200 3350
 F 0 "V2" H 6800 3450 50  0000 L CNN
-F 1 "2" H 6800 3200 50  0000 L CNN
+F 1 "4" H 6800 3200 50  0000 L CNN
 F 2 "" H 7200 3350 50  0001 C CNN
 F 3 "~" H 7200 3350 50  0001 C CNN
@@
 Text Notes 800  6900 0    50   ~ 0
 use 2N7000\nMOSFET instead
+Wire Wire Line
+	4600 5400 4650 5400
+Wire Wire Line
+	4300 5400 4150 5400
+Wire Wire Line
+	4150 5400 4150 5200
+Connection ~ 4150 5200
+Connection ~ 4650 5400
+Wire Wire Line
+	4650 5400 4700 5400
+Wire Wire Line
+	4200 5750 3800 5750
+Wire Wire Line
+	3800 5750 3800 5850
 $EndSCHEMATC

Commit message: more comments
Parts:
- R16: value 1Meg -> 100k
- R19: value 200k -> 534k
- R20: value 3.3k -> 10k
- R21: value 200k -> 220k
- R4, R5, R6: value 50k -> 47k
- V2: value 4 -> 1
Other:
- note added: ".tran 10u 10m"
- note added: "10k / 534k = 0.0187\ni.e. for 1V on V_control, the output\nwill change by 18.7mV."
- note added: "R16 determines the I_C current through\nQ4 when Q4's base is at GNDREF.\nTogether with V_tune, it determines the pitch.\nChoose R16 and V_tune such, that U8's output needs\nto be at around GNDREF for "sane" pitches."
- note added: "for Q4, the following holds true:\nI_C = const * exp(V_B / VT) with VT=26mV\n(thermal voltage of a transistor)\nnow this means that Vout will double\nevery (log(2) * 26mV) = 18mV."
- note added: "or use\nBCM847"
- note removed: ".tran 0.1u 10m"
Changed lines of the file:
@@
 P 3400 1400
 F 0 "R16" H 3470 1446 50  0000 L CNN
-F 1 "1Meg" H 3470 1355 50  0000 L CNN
+F 1 "100k" H 3470 1355 50  0000 L CNN
 F 2 "" V 3330 1400 50  0001 C CNN
 F 3 "~" H 3400 1400 50  0001 C CNN
@@
 U 1 1 5D054548
 P 1100 1800
-F 0 "R19" V 950 1800 50  0000 C CNN
-F 1 "200k" V 1100 1800 50  0000 C CNN
+F 0 "R19" V 1000 1800 50  0000 C CNN
+F 1 "534k" V 1100 1800 50  0000 C CNN
 F 2 "" V 1030 1800 50  0001 C CNN
 F 3 "~" H 1100 1800 50  0001 C CNN
@@
 P 1100 2000
 F 0 "R21" V 1200 2000 50  0000 C CNN
-F 1 "200k" V 1100 2000 50  0000 C CNN
+F 1 "220k" V 1100 2000 50  0000 C CNN
 F 2 "" V 1030 2000 50  0001 C CNN
 F 3 "~" H 1100 2000 50  0001 C CNN
@@
 Connection ~ 9900 3700
 Text Notes 7050 600  0    50   ~ 0
-.tran 0.1u 10m
+.tran 10u 10m
 $Comp
 L Device:R R20
 U 1 1 5D054E64
 P 1450 1650
-F 0 "R20" H 1380 1604 50  0000 R CNN
-F 1 "3.3k" H 1380 1695 50  0000 R CNN
+F 0 "R20" V 1550 1700 50  0000 R CNN
+F 1 "10k" V 1450 1700 50  0000 R CNN
 F 2 "" V 1380 1650 50  0001 C CNN
 F 3 "~" H 1450 1650 50  0001 C CNN
@@
 P 7200 3350
 F 0 "V2" H 6800 3450 50  0000 L CNN
-F 1 "4" H 6800 3200 50  0000 L CNN
+F 1 "1" H 6800 3200 50  0000 L CNN
 F 2 "" H 7200 3350 50  0001 C CNN
 F 3 "~" H 7200 3350 50  0001 C CNN
@@
 P 1850 6150
 F 0 "R6" V 1750 6150 50  0000 C CNN
-F 1 "50k" V 1850 6150 50  0000 C CNN
+F 1 "47k" V 1850 6150 50  0000 C CNN
 F 2 "" V 1780 6150 50  0001 C CNN
 F 3 "~" H 1850 6150 50  0001 C CNN
@@
 P 1650 6250
 F 0 "R5" V 1750 6250 50  0000 C CNN
-F 1 "50k" V 1650 6250 50  0000 C CNN
+F 1 "47k" V 1650 6250 50  0000 C CNN
 F 2 "" V 1580 6250 50  0001 C CNN
 F 3 "~" H 1650 6250 50  0001 C CNN
@@
 P 1400 6000
 F 0 "R4" V 1500 6000 50  0000 C CNN
-F 1 "50k" V 1400 6000 50  0000 C CNN
+F 1 "47k" V 1400 6000 50  0000 C CNN
 F 2 "" V 1330 6000 50  0001 C CNN
 F 3 "~" H 1400 6000 50  0001 C CNN
@@
 U 1 1 5CFF1629
 P 5350 1050
-F 0 "R18" V 5143 1050 50  0000 C CNN
-F 1 "10k" V 5234 1050 50  0000 C CNN
+F 0 "R18" V 5250 1050 50  0000 C CNN
+F 1 "10k" V 5350 1050 50  0000 C CNN
 F 2 "" V 5280 1050 50  0001 C CNN
 F 3 "~" H 5350 1050 50  0001 C CNN
@@
 Wire Wire Line
 	3800 5750 3800 5850
+Text Notes 3500 2050 0    50   ~ 0
+or use\nBCM847
+Text Notes 900  1350 0    50   ~ 0
+10k / 534k = 0.0187\ni.e. for 1V on V_control, the output\nwill change by 18.7mV.
+Text Notes 3950 2850 0    50   ~ 0
+for Q4, the following holds true:\nI_C = const * exp(V_B / VT) with VT=26mV\n(thermal voltage of a transistor)\nnow this means that Vout will double\nevery (log(2) * 26mV) = 18mV.
+Text Notes 2700 950  0    50   ~ 0
+R16 determines the I_C current through\nQ4 when Q4's base is at GNDREF.\nTogether with V_tune, it determines the pitch.\nChoose R16 and V_tune such, that U8's output needs\nto be at around GNDREF for "sane" pitches.
 $EndSCHEMATC
