File: simulation/filter_feedback/filter_feedback.sch (KiCad schematic (older format))
At the start: 37 parts, among them Q1 QNPN, U1 LM324, U2 LM324, U3 LM324, U4 LM324, U5 LM324, U6 LM324, U7 LM324

Commit message: various simulations
Parts:
- removed C7, C8: 100n, symbol Device:C
- removed C9: 10n, symbol Device:C
- removed Q1: QNPN, symbol pspice:QNPN
- removed R10, R14: 100k, symbol Device:R
- removed R12: 1G, symbol Device:R
- removed R9004: 10Meg, symbol Device:R
- removed U7: LM324, symbol pspice:OPAMP
- removed V5: pulse (0 20m 0 0 0 10m 20m) ac 1, symbol pspice:VSOURCE
- removed V6: 5, symbol pspice:VSOURCE
- V4: value ac 0.1 -> ac 10
