File: hardware/vco_mk1/vco_mk1/vco_mk1.sch (KiCad schematic (older format))
At the start: 87 parts

Commit message: remove duplicate solder bridges
Parts:
- removed SB? (x2): SolderJumper_2_Open, symbol Jumper:SolderJumper_2_Open
Connections:
- wire segments 232 -> 224
Other:
- moved on the sheet: JP?
Changed lines of the file:
@@
 Wire Notes Line
 	10000 5075 10000 6475
-Wire Wire Line
-	3975 4175 4025 4175
-Wire Wire Line
-	4375 4175 4325 4175
 Text GLabel 9400 2900 0    50   Input ~ 0
 ctl_override
@@
 L Jumper:Jumper_2_Open JP?
 U 1 1 5E0BADDE
-P 3475 2275
-F 0 "JP?" H 3300 2325 50  0000 C CNN
-F 1 "Rossum override" H 3475 2400 50  0000 C CNN
-F 2 "" H 3475 2275 50  0001 C CNN
-F 3 "~" H 3475 2275 50  0001 C CNN
-	1    3475 2275
-	1    0    0    -1
-$EndComp
-Wire Wire Line
-	3275 2275 3125 2275
-Wire Wire Line
-	3125 2275 3125 2425
-Connection ~ 3125 2800
-Wire Wire Line
-	3125 2800 3250 2800
-Wire Wire Line
-	3675 2275 3800 2275
-Wire Wire Line
-	3800 2275 3800 2425
-Connection ~ 3800 2925
-Wire Wire Line
-	3800 2925 3975 2925
-Wire Wire Line
-	4125 4050 3975 4050
-$Comp
-L Jumper:SolderJumper_2_Open SB?
-U 1 1 5E0F0CDF
-P 4325 4175
-F 0 "SB?" H 4325 4075 50  0000 C CNN
-F 1 "SolderJumper_2_Open" H 4300 4050 50  0001 C CNN
-F 2 "" H 4325 4175 50  0001 C CNN
-F 3 "~" H 4325 4175 50  0001 C CNN
-	1    4325 4175
-	1    0    0    -1
-$EndComp
-Wire Wire Line
-	4125 4050 4125 4175
-Connection ~ 4125 4050
-Wire Wire Line
-	4525 4050 4525 4175
-Connection ~ 4525 4050
-$Comp
-L Jumper:SolderJumper_2_Open SB?
-U 1 1 5E106B1B
 P 3475 2425
-F 0 "SB?" H 3475 2325 50  0000 C CNN
-F 1 "SolderJumper_2_Open" H 3450 2300 50  0001 C CNN
+F 0 "JP?" H 3300 2475 50  0000 C CNN
+F 1 "Rossum override" H 3475 2550 50  0000 C CNN
 F 2 "" H 3475 2425 50  0001 C CNN
 F 3 "~" H 3475 2425 50  0001 C CNN
@@
 	1    0    0    -1
 $EndComp
-Wire Wire Line
-	3325 2425 3125 2425
-Connection ~ 3125 2425
+Connection ~ 3125 2800
+Wire Wire Line
+	3125 2800 3250 2800
+Connection ~ 3800 2925
+Wire Wire Line
+	3800 2925 3975 2925
+Wire Wire Line
+	4125 4050 3975 4050
 Wire Wire Line
 	3125 2425 3125 2800
-Wire Wire Line
-	3625 2425 3800 2425
-Connection ~ 3800 2425
 Wire Wire Line
 	3800 2425 3800 2925
@@
 	1    0    0    -1
 $EndComp
+Wire Wire Line
+	3275 2425 3125 2425
+Wire Wire Line
+	3675 2425 3800 2425
 $EndSCHEMATC

Commit message: consistent naming
Parts:
- gave numbers to parts that had none: 1
Changed lines of the file:
@@
 	6725 5200 7300 5200
 $Comp
-L Connector:Conn_01x04_Male J?
+L Connector:Conn_01x04_Male JP?
 U 1 1 5D8F200D
 P 9300 5400
-F 0 "J?" V 9325 5625 50  0000 R CNN
+F 0 "JP?" V 9325 5675 50  0000 R CNN
 F 1 "ringmod config" V 9225 5725 50  0000 R CNN
 F 2 "" H 9300 5400 50  0001 C CNN
@@
 Wire Wire Line
 	10475 5650 10675 5650
-$Comp
-L Connector_Generic:Conn_02x03_Counter_Clockwise J?
-U 1 1 5DED6187
-P 10525 6050
-F 0 "J?" H 10575 6250 50  0000 C CNN
-F 1 "BCM847 breakout socket" H 10600 5850 50  0000 C CNN
-F 2 "" H 10525 6050 50  0001 C CNN
-F 3 "~" H 10525 6050 50  0001 C CNN
-	1    10525 6050
-	1    0    0    -1
-$EndComp
 Text GLabel 10325 5950 0    50   Input ~ 0
 E
@@
 	1175 3000 1175 3025
 $Comp
-L Connector:Conn_01x02_Male J?
+L Connector:Conn_01x02_Male JP?
 U 1 1 5DDEFD28
 P 3975 1575
-F 0 "J?" V 4025 1450 50  0000 R CNN
+F 0 "JP?" V 4025 1450 50  0000 R CNN
 F 1 "expo in" V 3900 1675 50  0000 R CNN
 F 2 "" H 3975 1575 50  0001 C CNN
@@
 Wire Wire Line
 	3675 2425 3800 2425
+$Comp
+L Connector_Generic:Conn_02x03_Counter_Clockwise J?
+U 1 1 5DED6187
+P 10525 6050
+F 0 "J?" H 10575 6250 50  0000 C CNN
+F 1 "BCM847 breakout socket" H 10600 5850 50  0000 C CNN
+F 2 "" H 10525 6050 50  0001 C CNN
+F 3 "~" H 10525 6050 50  0001 C CNN
+	1    10525 6050
+	1    0    0    -1
+$EndComp
 $EndSCHEMATC

Commit message: pre-name some components
Parts:
- J4: renamed from J?; value Conn_01x04_Male -> ringmod in
- R?: value R_POT -> TODO
- gave numbers to parts that had none: 9
Other:
- moved on the sheet: J1, R?

Commit message: annotate all components
Parts:
- Q1: value 1/2 BCM847 -> BCM847
- gave numbers to parts that had none: 64

Commit message: component selection 80%
Parts:
- C1, C10, C11, C2, C3, C4, C5, C6, C7, C8, C9: footprint (none) -> Capacitor_SMD:C_0805_2012Metric_Pad1.15x1.40mm_HandSolder
- J1: footprint (none) -> Connector_PinHeader_2.54mm:PinHeader_1x03_P2.54mm_Vertical
- J2: footprint (none) -> Connector_PinHeader_2.54mm:PinHeader_2x07_P2.54mm_Vertical
- J3: footprint (none) -> Connector_PinHeader_2.54mm:PinHeader_2x06_P2.54mm_Vertical
- J4: footprint (none) -> Connector_PinHeader_2.54mm:PinHeader_1x04_P2.54mm_Vertical
- J5: footprint (none) -> Connector_Samtec_HLE_SMD:Samtec_HLE-103-02-xxx-DV-BE-LC_2x03_P2.54mm_Horizontal
- R1, R11: footprint (none) -> Potentiometer_THT:Potentiometer_Bourns_3296W_Vertical
- R10, R12, R14, R15, R16, R17, R18, R19, R2, R20, R21, R22, R24, R25, R27, R28, R3, R30, R31, R32, R33, R34, R35, R36, R37, R38, R39, R4, R40, R41, R5, R6, R8, R9: footprint (none) -> Resistor_SMD:R_0805_2012Metric_Pad1.15x1.40mm_HandSolder
- R13, R23, R29: footprint (none) -> Resistor_THT:R_Axial_DIN0918_L18.0mm_D9.0mm_P22.86mm_Horizontal
- R26, R42: footprint (none) -> Potentiometer_THT:Potentiometer_Runtron_RM-065_Vertical
- R7: footprint (none) -> Resistor_THT:R_Axial_DIN0204_L3.6mm_D1.6mm_P2.54mm_Vertical
- U1, U2, U3: footprint (none) -> Package_DIP:DIP-14_W7.62mm

Commit message: layout wip
Parts:
- J5: footprint Connector_Samtec_HLE_SMD:Samtec_HLE-103-02-xxx-DV-BE-LC_2x03_P2.54mm_Horizontal -> Package_DIP:DIP-6_W7.62mm_Socket
- JP1, JP2, JP3: footprint (none) -> footprints:SolderDipJumper2alt
- JP4: footprint (none) -> footprints:SolderDipJumper3alt
- JP5: footprint (none) -> footprints:SolderDipJumper4alt
- R13: footprint Resistor_THT:R_Axial_DIN0918_L18.0mm_D9.0mm_P22.86mm_Horizontal -> Resistor_SMD:R_0805_2012Metric_Pad1.15x1.40mm_HandSolder
- R19: footprint Resistor_SMD:R_0805_2012Metric_Pad1.15x1.40mm_HandSolder -> Potentiometer_THT:Potentiometer_Runtron_RM-065_Vertical
- R23: footprint Resistor_THT:R_Axial_DIN0918_L18.0mm_D9.0mm_P22.86mm_Horizontal -> Potentiometer_THT:Potentiometer_Bourns_3296W_Vertical
- R29: footprint Resistor_THT:R_Axial_DIN0918_L18.0mm_D9.0mm_P22.86mm_Horizontal -> Potentiometer_THT:Potentiometer_Runtron_RM-065_Vertical
Changed lines of the file:
@@
 F 0 "JP5" V 9325 5675 50  0000 R CNN
 F 1 "ringmod config" V 9225 5725 50  0000 R CNN
-F 2 "" H 9300 5400 50  0001 C CNN
+F 2 "footprints:SolderDipJumper4alt" H 9300 5400 50  0001 C CNN
 F 3 "~" H 9300 5400 50  0001 C CNN
 	1    9300 5400
@@
 Text GLabel 10175 5450 0    50   Input ~ 0
 B1
-Text GLabel 10975 5450 2    50   Input ~ 0
-B2
 Text GLabel 10575 5650 3    50   Input ~ 0
 E
@@
 Text GLabel 10325 6150 0    50   Input ~ 0
 C2
-Text GLabel 10825 6050 2    50   Input ~ 0
-B2
 Text Notes 10025 6450 0    50   ~ 0
 alternative transistors\nonly equip one pair
@@
 F 0 "R29" V 2675 6775 50  0000 L CNN
 F 1 "1Meg" V 2525 6800 50  0000 L CNN
-F 2 "Resistor_THT:R_Axial_DIN0918_L18.0mm_D9.0mm_P22.86mm_Horizontal" V 2530 6850 50  0001 C CNN
+F 2 "Potentiometer_THT:Potentiometer_Runtron_RM-065_Vertical" V 2530 6850 50  0001 C CNN
 F 3 "~" H 2600 6850 50  0001 C CNN
 	1    2600 6850
@@
 F 0 "R23" H 1475 6950 50  0000 L CNN
 F 1 "10k" H 1400 6850 50  0000 L CNN
-F 2 "Resistor_THT:R_Axial_DIN0918_L18.0mm_D9.0mm_P22.86mm_Horizontal" V 1555 6900 50  0001 C CNN
+F 2 "Potentiometer_THT:Potentiometer_Bourns_3296W_Vertical" V 1555 6900 50  0001 C CNN
 F 3 "~" H 1625 6900 50  0001 C CNN
 	1    1625 6900
@@
 F 0 "JP4" H 1525 7525 50  0000 C CNN
 F 1 "gnd adjust" H 1625 7700 50  0000 C CNN
-F 2 "" H 1625 7600 50  0001 C CNN
+F 2 "footprints:SolderDipJumper3alt" H 1625 7600 50  0001 C CNN
 F 3 "~" H 1625 7600 50  0001 C CNN
 	1    1625 7600
@@
 F 0 "J5" H 10575 6250 50  0000 C CNN
 F 1 "BCM847 breakout socket" H 10600 5850 50  0000 C CNN
-F 2 "Connector_Samtec_HLE_SMD:Samtec_HLE-103-02-xxx-DV-BE-LC_2x03_P2.54mm_Horizontal" H 10525 6050 50  0001 C CNN
+F 2 "Package_DIP:DIP-6_W7.62mm_Socket" H 10525 6050 50  0001 C CNN
 F 3 "~" H 10525 6050 50  0001 C CNN
 	1    10525 6050
@@
 F 0 "R19" V 7525 1425 50  0000 C CNN
 F 1 "50k" V 7450 1450 50  0000 C CNN
-F 2 "Resistor_SMD:R_0805_2012Metric_Pad1.15x1.40mm_HandSolder" V 7280 1475 50  0001 C CNN
+F 2 "Potentiometer_THT:Potentiometer_Runtron_RM-065_Vertical" V 7280 1475 50  0001 C CNN
 F 3 "~" H 7350 1475 50  0001 C CNN
 	1    7350 1475
@@
 F 0 "JP3" V 4025 1450 50  0000 R CNN
 F 1 "expo in" V 3900 1675 50  0000 R CNN
-F 2 "" H 3975 1575 50  0001 C CNN
+F 2 "footprints:SolderDipJumper2alt" H 3975 1575 50  0001 C CNN
 F 3 "~" H 3975 1575 50  0001 C CNN
 	1    3975 1575
@@
 F 0 "JP1" H 3300 2475 50  0000 C CNN
 F 1 "Rossum override" H 3475 2550 50  0000 C CNN
-F 2 "" H 3475 2425 50  0001 C CNN
+F 2 "footprints:SolderDipJumper2alt" H 3475 2425 50  0001 C CNN
 F 3 "~" H 3475 2425 50  0001 C CNN
 	1    3475 2425
@@
 F 0 "JP2" H 4325 4200 50  0000 C CNN
 F 1 "Rossum connect" H 4325 4125 50  0000 C CNN
-F 2 "" H 4325 4050 50  0001 C CNN
+F 2 "footprints:SolderDipJumper2alt" H 4325 4050 50  0001 C CNN
 F 3 "~" H 4325 4050 50  0001 C CNN
 	1    4325 4050
@@
 Text GLabel 5650 2325 1    50   Input ~ 0
 E
-Text GLabel 6200 2125 1    50   Input ~ 0
-B2
 Text GLabel 5100 2125 1    50   Input ~ 0
 B1
@@
 F 0 "R13" V 3300 3050 50  0000 C CNN
 F 1 "100k" V 3400 3050 50  0000 C CNN
-F 2 "Resistor_THT:R_Axial_DIN0918_L18.0mm_D9.0mm_P22.86mm_Horizontal" V 3330 3050 50  0001 C CNN
+F 2 "Resistor_SMD:R_0805_2012Metric_Pad1.15x1.40mm_HandSolder" V 3330 3050 50  0001 C CNN
 F 3 "~" H 3400 3050 50  0001 C CNN
 	1    3400 3050
@@
 	1    0    0    -1
 $EndComp
+Text GLabel 10825 6050 2    50   Input ~ 0
+GND
+Text GLabel 10975 5450 2    50   Input ~ 0
+GND
+Text GLabel 6200 2125 1    50   Input ~ 0
+GND
+Text GLabel 1400 1075 1    50   Input ~ 0
+GNDREF
+$Comp
+L power:GNDREF #PWR0106
+U 1 1 5EC060DD
+P 1400 1075
+F 0 "#PWR0106" H 1400 825 50  0001 C CNN
+F 1 "GNDREF" H 1405 902 50  0001 C CNN
+F 2 "" H 1400 1075 50  0001 C CNN
+F 3 "" H 1400 1075 50  0001 C CNN
+	1    1400 1075
+	1    0    0    -1
+$EndComp
+Text GLabel 1275 1075 1    50   Input ~ 0
+GNDREF
+$Comp
+L power:GNDREF #PWR0105
+U 1 1 5EBF8868
+P 1275 1075
+F 0 "#PWR0105" H 1275 825 50  0001 C CNN
+F 1 "GNDREF" H 1280 902 50  0001 C CNN
+F 2 "" H 1275 1075 50  0001 C CNN
+F 3 "" H 1275 1075 50  0001 C CNN
+	1    1275 1075
+	1    0    0    -1
+$EndComp
+Text GLabel 1150 1075 1    50   Input ~ 0
+GNDREF
+$Comp
+L power:GNDREF #PWR0104
+U 1 1 5EBEB0EB
+P 1150 1075
+F 0 "#PWR0104" H 1150 825 50  0001 C CNN
+F 1 "GNDREF" H 1155 902 50  0001 C CNN
+F 2 "" H 1150 1075 50  0001 C CNN
+F 3 "" H 1150 1075 50  0001 C CNN
+	1    1150 1075
+	1    0    0    -1
+$EndComp
+Text GLabel 1025 1075 1    50   Input ~ 0
+GNDREF
+$Comp
+L power:GNDREF #PWR0103
+U 1 1 5EBDD8AA
+P 1025 1075
+F 0 "#PWR0103" H 1025 825 50  0001 C CNN
+F 1 "GNDREF" H 1030 902 50  0001 C CNN
+F 2 "" H 1025 1075 50  0001 C CNN
+F 3 "" H 1025 1075 50  0001 C CNN
+	1    1025 1075
+	1    0    0    -1
+$EndComp
+Text GLabel 900  1075 1    50   Input ~ 0
+GNDREF
+$Comp
+L power:GNDREF #PWR0102
+U 1 1 5EBCFF9F
+P 900 1075
+F 0 "#PWR0102" H 900 825 50  0001 C CNN
+F 1 "GNDREF" H 905 902 50  0001 C CNN
+F 2 "" H 900 1075 50  0001 C CNN
+F 3 "" H 900 1075 50  0001 C CNN
+	1    900  1075
+	1    0    0    -1
+$EndComp
+Text GLabel 775  1075 1    50   Input ~ 0
+GNDREF
+$Comp
+L power:GNDREF #PWR0101
+U 1 1 5EB79DB0
+P 775 1075
+F 0 "#PWR0101" H 775 825 50  0001 C CNN
+F 1 "GNDREF" H 780 902 50  0001 C CNN
+F 2 "" H 775 1075 50  0001 C CNN
+F 3 "" H 775 1075 50  0001 C CNN
+	1    775  1075
+	1    0    0    -1
+$EndComp

Commit message: layout wip2
Parts:
- removed J2: control in, Connector_PinHeader_2.54mm:PinHeader_2x07_P2.54mm_Vertical, symbol Connector_Generic:Conn_02x07_Counter_Clockwise
- added J2: control in, Connector_PinHeader_2.54mm:PinHeader_2x07_P2.54mm_Vertical, symbol Connector_Generic:Conn_02x07_Odd_Even
Connections:
- net C2: now also J2.10 (Pin_10)
- net GNDREF: now also J2.1 (Pin_1), J2.13 (Pin_13), J2.14 (Pin_14), J2.2 (Pin_2)
- net V_control: now also J2.3 (Pin_3)
- net V_control_2: now also J2.5 (Pin_5)
- net V_control_3: now also J2.7 (Pin_7)
- net V_control_raw: now also J2.9 (Pin_9)
- net V_lin_pitchmod_1: now also J2.4 (Pin_4)
- net V_lin_pitchmod_2: now also J2.6 (Pin_6)
- net V_lin_pitchmod_3: now also J2.8 (Pin_8)
- net V_pwm: now also J2.12 (Pin_12)
- net ctl_override: now also J2.11 (Pin_11)
Changed lines of the file:
@@
 	1    0    0    -1
-$EndComp
-$Comp
-L Diode:1N4148 D1
-U 1 1 5E16153A
-P 3550 3350
-F 0 "D1" H 3550 3250 50  0000 C CNN
-F 1 "1N4148" H 3550 3450 50  0000 C CNN
-F 2 "Diode_THT:D_DO-35_SOD27_P7.62mm_Horizontal" H 3550 3175 50  0001 C CNN
-F 3 "https://assets.nexperia.com/documents/data-sheet/1N4148_1N4448.pdf" H 3550 3350 50  0001 C CNN
-	1    3550 3350
-	-1   0    0    1
 $EndComp
 Wire Wire Line
@@
 F 3 "~" H 3475 2425 50  0001 C CNN
 	1    3475 2425
-	1    0    0    -1
-$EndComp
-$Comp
-L Jumper:Jumper_2_Bridged JP2
-U 1 1 5E0B9FA6
-P 4325 4050
-F 0 "JP2" H 4325 4200 50  0000 C CNN
-F 1 "Rossum connect" H 4325 4125 50  0000 C CNN
-F 2 "footprints:SolderDipJumper2alt" H 4325 4050 50  0001 C CNN
-F 3 "~" H 4325 4050 50  0001 C CNN
-	1    4325 4050
 	1    0    0    -1
 $EndComp
@@
 Wire Notes Line
 	2950 2625 2950 3850
-Wire Wire Line
-	3700 3350 3975 3350
 Wire Notes Line
 	2950 2625 3725 2625
@@
 Wire Wire Line
 	9400 2400 9400 2300
-$Comp
-L Connector_Generic:Conn_02x07_Counter_Clockwise J2
-U 1 1 5D5F57E8
-P 9600 2700
-F 0 "J2" H 9575 3150 50  0000 C CNN
-F 1 "control in" V 9650 2700 50  0000 C CNN
-F 2 "Connector_PinHeader_2.54mm:PinHeader_2x07_P2.54mm_Vertical" H 9600 2700 50  0001 C CNN
-F 3 "~" H 9600 2700 50  0001 C CNN
-	1    9600 2700
-	1    0    0    -1
-$EndComp
 Text GLabel 9900 2900 2    50   Input ~ 0
 V_pwm
@@
 	1    0    0    -1
 $EndComp
+Wire Wire Line
+	3700 3350 3975 3350
+$Comp
+L Jumper:Jumper_2_Bridged JP2
+U 1 1 5E0B9FA6
+P 4325 4050
+F 0 "JP2" H 4325 4200 50  0000 C CNN
+F 1 "Rossum connect" H 4325 4125 50  0000 C CNN
+F 2 "footprints:SolderDipJumper2alt" H 4325 4050 50  0001 C CNN
+F 3 "~" H 4325 4050 50  0001 C CNN
+	1    4325 4050
+	1    0    0    -1
+$EndComp
+$Comp
+L Diode:1N4148 D1
+U 1 1 5E16153A
+P 3550 3350
+F 0 "D1" H 3550 3250 50  0000 C CNN
+F 1 "1N4148" H 3550 3450 50  0000 C CNN
+F 2 "Diode_THT:D_DO-35_SOD27_P7.62mm_Horizontal" H 3550 3175 50  0001 C CNN
+F 3 "https://assets.nexperia.com/documents/data-sheet/1N4148_1N4448.pdf" H 3550 3350 50  0001 C CNN
+	1    3550 3350
+	-1   0    0    1
+$EndComp
+$Comp
+L Connector_Generic:Conn_02x07_Odd_Even J2
+U 1 1 5D76A0AB
+P 9600 2700
+F 0 "J2" H 9575 3175 50  0000 C CNN
+F 1 "control in" V 9650 2700 50  0000 C CNN
+F 2 "Connector_PinHeader_2.54mm:PinHeader_2x07_P2.54mm_Vertical" H 9600 2700 50  0001 C CNN
+F 3 "~" H 9600 2700 50  0001 C CNN
+	1    9600 2700
+	1    0    0    -1
+$EndComp

Commit message: fix XOR schematic
Parts:
- added R? (x5): 10k, Resistor_SMD:R_0805_2012Metric_Pad1.15x1.40mm_HandSolder, symbol Device:R
Connections:
- net GNDREF: now also C11.1, R37.2, R38.2, R39.2, R40.2, R41.2, U3.7 (GND)
- net VEE: no longer C11.1, R37.2, R38.2, R39.2, R40.2, R41.2, U3.7 (GND)
- net at R37.1, U3.1: now also R?.1; no longer J4.1 (Pin_1)
- net at R38.1, U3.2: now also R?.1; no longer J4.2 (Pin_2)
- net at R41.1, U3.10: now also R?.2; no longer JP5.4 (Pin_4)
- net at R39.1, U3.12: now also R?.1; no longer J4.3 (Pin_3)
- net at R40.1, U3.13: now also R?.1; no longer J4.4 (Pin_4)
- net VCC renamed +5V
- new net: JP5.4 (Pin_4), R?.1
- new net: J4.1 (Pin_1), R?.2
- new net: J4.2 (Pin_2), R?.2
- new net: J4.3 (Pin_3), R?.2
- new net: J4.4 (Pin_4), R?.2
Other:
- note added: "Q5 cannot be\nreplaced by a \nmosfet due to\nthe parasitic\ndiode inside a\nFET. Do replace\nit for some\ncrunchy wave-\nshaping, though."
- note added: "TODO\nor 470"
- note added: "VCC-GND should be <= 6V \nabsolute maximum: 7V).\nOtherwise, 5V and VCC\nmust be separated"
- note removed: "Q? cannot be\nreplaced by a \nmosfet due to\nthe parasitic\ndiode inside a\nFET. Do replace\nit for some\ncrunchy wave-\nshaping, though."
- moved on the sheet: C11, C4, C5, C6, C7, J2, J3, J4, J5, JP5, Q2, Q3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
