File: hardware/vco_mk1/vco_mk1/vco_mk1.sch (KiCad schematic (older format))
At the start: 77 parts, among them J1 power supply, J2 control in, J3 signal out, J4 ringmod in, J5 BCM847 breakout socket, Q1 BCM847, Q2 BC547, Q3 BC547, Q4 2N7000, Q5 BC547, U1 LM324, U2 LM324, U3 74HC86

Commit message: better ring modulation. improved comments
Parts:
- removed J1: power supply, Connector_PinHeader_2.54mm:PinHeader_1x03_P2.54mm_Vertical, symbol Connector_Generic:Conn_01x03
- removed J3: signal out, Connector_PinHeader_2.54mm:PinHeader_2x06_P2.54mm_Vertical, symbol Connector_Generic:Conn_02x06_Odd_Even
- removed J4: ringmod in, Connector_PinHeader_2.54mm:PinHeader_1x04_P2.54mm_Vertical, symbol Connector:Conn_01x04_Male
- removed R37, R38, R41: 100k, Resistor_SMD:R_0805_2012Metric_Pad1.15x1.40mm_HandSolder, symbol Device:R
- removed R? (x2): 10k, Resistor_SMD:R_0805_2012Metric_Pad1.15x1.40mm_HandSolder, symbol Device:R
- added C?: 100n, Capacitor_SMD:C_0805_2012Metric_Pad1.15x1.40mm_HandSolder, symbol Device:C
- added J1: power supply, symbol Connector_Generic:Conn_02x03_Odd_Even
- added J3: signal out, symbol Connector_Generic:Conn_02x07_Odd_Even
- added J4: Conn_01x03_Male, symbol Connector:Conn_01x03_Male
- added Q?: BC327, Package_TO_SOT_THT:TO-92_Inline, symbol Transistor_BJT:BC327
- added R? (x2): 100k, Resistor_SMD:R_0805_2012Metric_Pad1.15x1.40mm_HandSolder, symbol Device:R
- added R? (x2): 10k, Resistor_SMD:R_0805_2012Metric_Pad1.15x1.40mm_HandSolder, symbol Device:R
- renumbered R40 to R?, R39 to R?
Connections:
- net +5V: now also R?.2, R?.2, J1.2 (Pin_2), R?.2, R?.2; no longer C1.2, C10.2, R1.1, R14.1, R27.2, R42.1, U1.4 (V+), U2.11 (V-)
- net GNDREF: now also J1.3 (Pin_3), J3.1 (Pin_1), J3.13 (Pin_13), J3.14 (Pin_14), J3.2 (Pin_2); no longer C11.1, R?.2, R?.2, U3.7 (GND)
- net VEE: now also J1.5 (Pin_5), R?.1
- net pulse: now also C6.1, U3.9, J3.5 (Pin_5); no longer C4.1
- net sawtooth: now also C7.1, J3.9 (Pin_9); no longer C5.1
- net square_ctl: now also C?.1, J3.11 (Pin_11); no longer C7.1
- net triangle: now also C5.1, J3.7 (Pin_7); no longer C6.1
- net at U3.1: now also R?.1, R?.1; no longer R?.1
- net at U3.2: now also R?.1, R?.1
- net at U3.5: now also R?.1, R?.1; no longer U3.11
- net at U3.6: now also U3.10, U3.12; no longer U3.9
- net at JP5.1 (Pin_1): now also Q?.1 (C), R?.2; no longer U3.8
- net at JP5.4 (Pin_4): now also U3.13, R?.1
- net at R?.2: now also U3.11
- net at R?.2: now also J4.2 (Pin_2)
- net at R?.2: now also J4.3 (Pin_3)
- net at C7.2: now also J3.10 (Pin_10)
- net at C4.2: now also J3.4 (Pin_4)
- net at C6.2: now also J3.6 (Pin_6)
- net at C5.2: now also J3.8 (Pin_8)
- new net: Q?.2 (B), R?.1
- new net: J4.1 (Pin_1), R?.2
- new net: C?.2, J3.12 (Pin_12)
- new net GNDD: C11.1, J1.4 (Pin_4), U3.7 (GND)
- new net VCC: C1.2, C10.2, J1.1 (Pin_1), Q?.3 (E), R1.1, R14.1, R27.2, R42.1, U1.4 (V+), U2.11 (V-)
- new net rmpulse: C4.1, J3.3 (Pin_3), U3.8
- no-connect marks 0 -> 1
Other:
- note added: "GNDREF and GNDD may be\nconnected, but this might have\na negative impact on the\nfrequency stability."
- note added: "Jumper configurations for JP5:\n12 + 34: sawtooth wave with 4x ringmod\n12: triangle wave with 4x ringmod\n (pin 4 can be used as fifth ringmod)\n23: sawtooth, no ring mod. Choose this\n when no 74HC86 is installed."
- note added: "Just a hacky way of applying an\nadjustable voltage with an adjustable\ninner resistance. Replace R26-R28\nby a 100-200k trimmer and leave\nout R29 completely if you want.\nOr just spare everything and connect\nthe (+) pin to GNDREF.\nThat will cause a slightly off-center\ntriangle wave and a shifted sawtooth,\nat least with the LM324."
- note added: "Optional components:\n\nRossum compensation: can be left out, you must close JP1 then.\n Effect: No precise 1V/oct tuning possible (stable, but non-linear\n frequency response; requires digital compensation)\n\nSawtooth gen / dig.ring.mod.: can be left out, you must connect JP5's pin2+3. \n Effect: No ring modulation features. Sawtooth still works.\n\nWaveform generation: can be left out (togethe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"
- note added: "R14 determines the I_C current through\nQ1B when Q1B's base is at GNDREF.\nTogether with V_tune, it determines the pitch.\nChoose R14 and V_tune such, that Q1A's base is\nat around GNDREF for "sane" pitches."
- note added: "R20 * C8 should be 100µs, this affects the freq. range\nR20 : R22+R23 must be 2:1, this affects the triangle shape\nR21 : R24 must be 1:1, this affects the triangle shape\nR29 : R30 should be 1:2, this affects the tri amplitude and\nfrequency range. Too large R29 may cause distortion\nR32 : R34 should be 1:1, this affects sawtooth amplitude"
- note added: "TODO:\nor 1k?"
- note added: "for Q1B, the following holds true:\nI_C = const * exp(V_B / VT) with VT=26mV\n(thermal voltage of a transistor)\nnow this means that V_expo will double\nevery (log(2) * 26mV) = 18mV.\n\nNote that VT is temperature dependent.\nWhen the temperature rises, VT rises and so\nthe input voltage must rise too. The thermal\ncompensation consisting of R7-10 does that.\n\nAdditionally, Q1A and Q1B have a bu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"
- note added: "shift the 0/5V levels up to Vcc / Vee\nlevels. Q5 wants to be driven with these"
- note added: "to put the pulse signal roughly at the same\nlevel as the others (ca. 3V peak-peak.\nothers can range from 1.5V to ca. 7V)"
- note removed: "If R8 was connected to GNDREF, the triangle would be\ncentered around GNDREF, but only if the output of the\ncomparator U3 would swing between Vcc and Vee.\nHowever, U3 swings between less-than-Vcc and\nexactly Vee, so the triangle isn't centered.\nR14 and R15 comprise a poti to compensate for that."
- note removed: "Jumper configurations:\n12 + 34: sawtooth wave with 4x ringmod\n12: triangle wave with 4x ringmod\n (pin 4 can be used as fifth ringmod)\n23: sawtooth, no ring mod. Choose this\n when no 74HC86 is installed."
- note removed: "Just a hacky way of applying an\nadjustable voltage with an adjustable\ninner resistance. Replace R?+R?+R?\nby a 100-200k trimmer and leave\nout R? completely if you want.\nOr just spare everything and connect\nthe (+) pin to GNDREF.\nThis will cause a slightly off-center\ntriangle wave and a shifted sawtooth,\nat least with the LM324."
- note removed: "R16 determines the I_C current through\nQ4 when Q4's base is at GNDREF.\nTogether with V_tune, it determines the pitch.\nChoose R16 and V_tune such, that U8's output needs\nto be at around GNDREF for "sane" pitches."
- note removed: "R3 * C1 should be 100µs, this affects the frequency range\nR3 : R5 must be 2:1, this affects the triangle shape\nR4 : R6 must be 1:1, this affects the triangle shape\nR8 : R9 should be 1:2, this affects the triangle amplitude and\nfrequency range. If R9 is too large, this may cause distortion\nR11 : R12 should be 1:1, this affects sawtooth amplitude"
- note removed: "TODO\nor 470"
- note removed: "do not use"
- note removed: "for Q4, the following holds true:\nI_C = const * exp(V_B / VT) with VT=26mV\n(thermal voltage of a transistor)\nnow this means that Vout will double\nevery (log(2) * 26mV) = 18mV.\n\nNote that VT is temperature dependent.\nWhen the temperature rises, VT rises and so\nthe input voltage must rise too. The thermal\ncompensation consisting of TODO does that.\n\nAdditionally, Q3 and Q4 have a bulk res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"
- note removed: "to put the pulse signal roughly at the same level as the others\n(ca. 3V peak-peak. others can range from 1.5V to ca. 7V)"
- moved on the sheet: C11, C4, C5, C6, C7, J2, JP5, R42, R?, U3A, U3B, U3C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

Commit message: annotate and add footprints
Parts:
- J1: footprint (none) -> Connector_PinHeader_2.54mm:PinHeader_2x03_P2.54mm_Vertical
- J3: footprint (none) -> Connector_PinHeader_2.54mm:PinHeader_2x07_P2.54mm_Vertical
- J4: footprint (none) -> Connector_PinHeader_2.54mm:PinHeader_1x03_P2.54mm_Vertical
- gave numbers to parts that had none: 11
Changed lines of the file:
@@
 $EndComp
 $Comp
-L power:+5V #PWR?
+L power:+5V #PWR039
 U 1 1 5D87E356
 P 9800 1125
-F 0 "#PWR?" H 9800 975 50  0001 C CNN
+F 0 "#PWR039" H 9800 975 50  0001 C CNN
 F 1 "+5V" H 9815 1298 50  0000 C CNN
 F 2 "" H 9800 1125 50  0001 C CNN
@@
 VCC-GND should be <= 6V \nabsolute maximum: 7V).\nOtherwise, 5V and VCC\nmust be separated
 $Comp
-L Device:R R?
+L Device:R R39
 U 1 1 5DA160FA
 P 6675 5450
-F 0 "R?" V 6625 5550 50  0000 L CNN
+F 0 "R39" V 6625 5550 50  0000 L CNN
 F 1 "10k" V 6675 5375 50  0000 L CNN
 F 2 "Resistor_SMD:R_0805_2012Metric_Pad1.15x1.40mm_HandSolder" V 6605 5450 50  0001 C CNN
@@
 $EndComp
 $Comp
-L Device:R R?
+L Device:R R38
 U 1 1 5DA129CE
 P 6675 5250
-F 0 "R?" V 6625 5350 50  0000 L CNN
+F 0 "R38" V 6625 5350 50  0000 L CNN
 F 1 "10k" V 6675 5175 50  0000 L CNN
 F 2 "Resistor_SMD:R_0805_2012Metric_Pad1.15x1.40mm_HandSolder" V 6605 5250 50  0001 C CNN
@@
 $EndComp
 $Comp
-L Device:R R?
+L Device:R R45
 U 1 1 5D9D225A
 P 9175 5450
-F 0 "R?" V 9075 5425 50  0000 L CNN
+F 0 "R45" V 9075 5375 50  0000 L CNN
 F 1 "10k" V 9175 5375 50  0000 L CNN
 F 2 "Resistor_SMD:R_0805_2012Metric_Pad1.15x1.40mm_HandSolder" V 9105 5450 50  0001 C CNN
@@
 Connection ~ 6400 4500
 $Comp
-L power:+5V #PWR?
+L power:+5V #PWR031
 U 1 1 5D8888E9
 P 6400 4500
-F 0 "#PWR?" H 6400 4350 50  0001 C CNN
+F 0 "#PWR031" H 6400 4350 50  0001 C CNN
 F 1 "+5V" H 6415 4673 50  0000 C CNN
 F 2 "" H 6400 4500 50  0001 C CNN
@@
 Connection ~ 8425 5250
 $Comp
-L Device:R R?
+L Device:R R43
 U 1 1 5D937375
 P 7275 5700
-F 0 "R?" H 7225 5475 50  0000 L CNN
+F 0 "R43" V 7275 5375 50  0000 L CNN
 F 1 "100k" V 7275 5600 50  0000 L CNN
 F 2 "Resistor_SMD:R_0805_2012Metric_Pad1.15x1.40mm_HandSolder" V 7205 5700 50  0001 C CNN
@@
 $EndComp
 $Comp
-L Device:R R?
+L Device:R R41
 U 1 1 5D985574
 P 7125 5700
-F 0 "R?" H 7075 5475 50  0000 L CNN
+F 0 "R41" V 7125 5375 50  0000 L CNN
 F 1 "100k" V 7125 5600 50  0000 L CNN
 F 2 "Resistor_SMD:R_0805_2012Metric_Pad1.15x1.40mm_HandSolder" V 7055 5700 50  0001 C CNN
@@
 	6825 5250 7125 5250
 $Comp
-L Device:R R?
+L Device:R R40
 U 1 1 5DF424B1
 P 6975 5700
-F 0 "R?" H 6925 5475 50  0000 L CNN
+F 0 "R40" V 6975 5375 50  0000 L CNN
 F 1 "100k" V 6975 5600 50  0000 L CNN
 F 2 "Resistor_SMD:R_0805_2012Metric_Pad1.15x1.40mm_HandSolder" V 6905 5700 50  0001 C CNN
@@
 F 0 "J4" H 6300 5450 50  0000 C CNN
 F 1 "Conn_01x03_Male" H 6275 5775 50  0001 C CNN
-F 2 "" H 6250 5250 50  0001 C CNN
+F 2 "Connector_PinHeader_2.54mm:PinHeader_1x03_P2.54mm_Vertical" H 6250 5250 50  0001 C CNN
 F 3 "~" H 6250 5250 50  0001 C CNN
 	1    6250 5250
@@
 	8425 6325 9025 6325
 $Comp
-L Device:R R?
+L Device:R R44
 U 1 1 5E0DCE8F
 P 7425 5700
-F 0 "R?" H 7375 5475 50  0000 L CNN
+F 0 "R44" V 7425 5375 50  0000 L CNN
 F 1 "100k" V 7425 5600 50  0000 L CNN
 F 2 "Resistor_SMD:R_0805_2012Metric_Pad1.15x1.40mm_HandSolder" V 7355 5700 50  0001 C CNN
@@
 	7425 5550 8425 5550
 $Comp
-L power:GNDD #PWR?
+L power:GNDD #PWR033
 U 1 1 5E183D97
 P 7400 4500
-F 0 "#PWR?" H 7400 4250 50  0001 C CNN
+F 0 "#PWR033" H 7400 4250 50  0001 C CNN
 F 1 "GNDD" H 7375 4375 50  0000 C CNN
 F 2 "" H 7400 4500 50  0001 C CNN
@@
 Connection ~ 7400 4500
 $Comp
-L power:+5V #PWR?
+L power:+5V #PWR032
 U 1 1 5E1D5BED
 P 6850 5850
-F 0 "#PWR?" H 6850 5700 50  0001 C CNN
+F 0 "#PWR032" H 6850 5700 50  0001 C CNN
 F 1 "+5V" H 6825 6000 50  0000 C CNN
 F 2 "" H 6850 5850 50  0001 C CNN
@@
 F 0 "J3" H 9675 4050 50  0000 C CNN
 F 1 "signal out" V 9750 3600 50  0000 C CNN
-F 2 "" H 9700 3600 50  0001 C CNN
+F 2 "Connector_PinHeader_2.54mm:PinHeader_2x07_P2.54mm_Vertical" H 9700 3600 50  0001 C CNN
 F 3 "~" H 9700 3600 50  0001 C CNN
 	1    9700 3600
@@
 rmpulse
 $Comp
-L Device:C C?
+L Device:C C12
 U 1 1 5E406B46
 P 10150 3800
-F 0 "C?" V 10100 3700 50  0000 C CNN
+F 0 "C12" V 10100 3700 50  0000 C CNN
 F 1 "100n" V 10100 3950 50  0000 C CNN
 F 2 "Capacitor_SMD:C_0805_2012Metric_Pad1.15x1.40mm_HandSolder" H 10188 3650 50  0001 C CNN
@@
 rmpulse
 $Comp
-L Transistor_BJT:BC327 Q?
+L Transistor_BJT:BC327 Q6
 U 1 1 5E4891B8
 P 9525 5450
-F 0 "Q?" H 9450 5275 50  0000 L CNN
+F 0 "Q6" H 9450 5275 50  0000 L CNN
 F 1 "BC327" H 9350 5625 50  0000 L CNN
 F 2 "Package_TO_SOT_THT:TO-92_Inline" H 9725 5375 50  0001 L CIN
@@
 Connection ~ 9625 5725
 $Comp
-L Device:R R?
+L Device:R R46
 U 1 1 5E4AF968
 P 9625 5950
-F 0 "R?" H 9725 5950 50  0000 L CNN
+F 0 "R46" H 9700 5950 50  0000 L CNN
 F 1 "10k" V 9625 5875 50  0000 L CNN
 F 2 "Resistor_SMD:R_0805_2012Metric_Pad1.15x1.40mm_HandSolder" V 9555 5950 50  0001 C CNN
@@
 $EndComp
 $Comp
-L power:VCC #PWR?
+L power:VCC #PWR037
 U 1 1 5E4C09F3
 P 9625 5250
-F 0 "#PWR?" H 9625 5100 50  0001 C CNN
+F 0 "#PWR037" H 9625 5100 50  0001 C CNN
 F 1 "VCC" H 9642 5423 50  0000 C CNN
 F 2 "" H 9625 5250 50  0001 C CNN
@@
 $EndComp
 $Comp
-L power:VEE #PWR?
+L power:VEE #PWR038
 U 1 1 5E4C205B
 P 9625 6100
-F 0 "#PWR?" H 9625 5950 50  0001 C CNN
+F 0 "#PWR038" H 9625 5950 50  0001 C CNN
 F 1 "VEE" H 9643 6273 50  0000 C CNN
 F 2 "" H 9625 6100 50  0001 C CNN
@@
 	6200 4225 9925 4225
 $Comp
-L Device:R R?
+L Device:R R37
 U 1 1 5E576FD2
 P 6675 5050
-F 0 "R?" V 6625 5150 50  0000 L CNN
+F 0 "R37" V 6625 5150 50  0000 L CNN
 F 1 "10k" V 6675 4975 50  0000 L CNN
 F 2 "Resistor_SMD:R_0805_2012Metric_Pad1.15x1.40mm_HandSolder" V 6605 5050 50  0001 C CNN
@@
 Optional components:\n\nRossum compensation: can be left out, you must close JP1 then.\n    Effect: No precise 1V/oct tuning possible (stable, but non-linear\n           frequency response; requires digital compensation)\n\nSawtooth gen / dig.ring.mod.: can be left out, you must connect JP5's pin2+3. \n    Effect: No ring modulation features. Sawtooth still works.\n\nWaveform generation: can be left out (together with saw gen (above))\n    Effect: Only the triangle and square_ctl waves are available.
 $Comp
-L power:GNDD #PWR?
+L power:GNDD #PWR040
 U 1 1 5E7FD69F
 P 9925 1225
-F 0 "#PWR?" H 9925 975 50  0001 C CNN
+F 0 "#PWR040" H 9925 975 50  0001 C CNN
 F 1 "GNDD" H 9975 1100 50  0000 C CNN
 F 2 "" H 9925 1225 50  0001 C CNN
@@
 F 0 "J1" H 9550 1542 50  0000 C CNN
 F 1 "power supply" H 9700 1000 50  0000 C CNN
-F 2 "" H 9500 1225 50  0001 C CNN
+F 2 "Connector_PinHeader_2.54mm:PinHeader_2x03_P2.54mm_Vertical" H 9500 1225 50  0001 C CNN
 F 3 "~" H 9500 1225 50  0001 C CNN
 	1    9500 1225

Commit message: add high pass filter for sawtooth/square generation
this fixes sawtooth/square generation when running
in DCO mode.
Parts:
- added C?: 100n, Capacitor_SMD:C_0805_2012Metric_Pad1.15x1.40mm_HandSolder, symbol Device:C
- added R?: none, symbol Device:R
Connections:
- net GNDREF: now also R?.2
- net triangle: now also C?.2; no longer R32.1, R33.2, U2.9 (-)
- new net: C?.1, R32.1, R33.2, R?.1, U2.9 (-)
Other:
- note added: "do not equip R?\n10-100k are fine,\nbut R33+Q5 are\nenough for our\npurpose."
- note added: "or 470n"
- note added: "remove the DC offset. This doesn't matter for normal\noperation, but for DCO operation, where R27-R30 have\nno effect and thus, the signal is not centered."
Changed lines of the file:
@@
 Text GLabel 5625 6700 2    50   Input ~ 0
 square_ctl
-Text GLabel 5675 5250 2    50   Input ~ 0
+Text GLabel 5675 5200 2    50   Input ~ 0
 triangle
 $Comp
@@
 $EndComp
 Wire Wire Line
-	5675 5250 4125 5250
-Wire Wire Line
 	2375 7400 3475 7400
 Wire Wire Line
@@
 Text GLabel 5675 5800 2    50   Input ~ 0
 sawtooth
-Wire Wire Line
-	4125 5700 4125 5250
-Connection ~ 4125 5250
-Wire Wire Line
-	4125 5250 2875 5250
 $Comp
 L Device:R R32
@@
 $EndComp
 Connection ~ 2875 6300
-Wire Wire Line
-	2875 5250 2875 6300
 $Comp
 L Device:R R31
@@
 Wire Wire Line
 	4675 5075 4125 5075
-Wire Wire Line
-	4125 5075 4125 5250
 Text GLabel 1025 4875 0    50   Input ~ 0
 V_pwm
@@
 Text Notes 9050 1875 0    50   ~ 0
 GNDREF and GNDD may be\nconnected, but this might have\na negative impact on the\nfrequency stability.
+Text Notes 3150 5300 0    50   ~ 0
+or 470n
+Wire Wire Line
+	4125 5075 4125 5325
+Wire Wire Line
+	5675 5200 2875 5200
+Wire Wire Line
+	2875 5200 2875 5325
+Wire Wire Line
+	2950 5325 2875 5325
+Connection ~ 2875 5325
+Wire Wire Line
+	2875 5325 2875 6300
+Wire Wire Line
+	3250 5325 3325 5325
+Connection ~ 4125 5325
+Wire Wire Line
+	4125 5325 4125 5700
+$Comp
+L Device:R R?
+U 1 1 5D53B3BE
+P 3325 5475
+F 0 "R?" H 3175 5525 50  0000 L CNN
+F 1 "none" V 3325 5375 50  0000 L CNN
+F 2 "" V 3255 5475 50  0001 C CNN
+F 3 "~" H 3325 5475 50  0001 C CNN
+	1    3325 5475
+	1    0    0    -1
+$EndComp
+Connection ~ 3325 5325
+Wire Wire Line
+	3325 5325 4125 5325
+$Comp
+L power:GNDREF #PWR?
+U 1 1 5D54168D
+P 3325 5625
+F 0 "#PWR?" H 3325 5375 50  0001 C CNN
+F 1 "GNDREF" H 3330 5452 50  0001 C CNN
+F 2 "" H 3325 5625 50  0001 C CNN
+F 3 "" H 3325 5625 50  0001 C CNN
+	1    3325 5625
+	-1   0    0    -1
+$EndComp
+Text Notes 2925 5675 0    25   ~ 0
+do not equip R?\n10-100k are fine,\nbut R33+Q5 are\nenough for our\npurpose.
+$Comp
+L Device:C C?
+U 1 1 5D49B6B5
+P 3100 5325
+F 0 "C?" V 3150 5225 50  0000 C CNN
+F 1 "100n" V 3050 5200 50  0000 C CNN
+F 2 "Capacitor_SMD:C_0805_2012Metric_Pad1.15x1.40mm_HandSolder" H 3138 5175 50  0001 C CNN
+F 3 "~" H 3100 5325 50  0001 C CNN
+	1    3100 5325
+	0    1    1    0
+$EndComp
+Text Notes 2800 5175 0    25   ~ 0
+remove the DC offset. This doesn't matter for normal\noperation, but for DCO operation, where R27-R30 have\nno effect and thus, the signal is not centered.
 $EndSCHEMATC

Commit message: add comment about deepmind-ish square variation
Other:
- note added: "For another interesting square wave\nvariation, connect ctl_override (JP5,\npin 3) to J4. Then play around with\nthe PWM voltage and watch rmpulse."
- note added: "TODO:\nraw pulse?"
Changed lines of the file:
@@
 Text Notes 2800 5175 0    25   ~ 0
 remove the DC offset. This doesn't matter for normal\noperation, but for DCO operation, where R27-R30 have\nno effect and thus, the signal is not centered.
+Text Notes 5725 5050 0    50   ~ 0
+TODO:\nraw pulse?
+Text Notes 5300 7475 0    50   ~ 0
+For another interesting square wave\nvariation, connect ctl_override (JP5,\npin 3) to J4. Then play around with\nthe PWM voltage and watch rmpulse.
 $EndSCHEMATC

Commit message: more comments
Parts:
- added JP?: Jumper_2_Open, symbol Jumper:Jumper_2_Open
Connections:
- net triangle: now also JP?.1 (A)
- net at C?.1, R32.1, R33.2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: now also JP?.2 (B)
Other:
- note added: "Just a hacky way of applying an\nadjustable voltage with an adjustable\ninner resistance. Replace R26-R28\nby a 100-200k trimmer and leave\nout R29 completely if you want.\nOr just spare everything and connect\nthe (+) pin via 100k to GNDREF.\nThat will cause a slightly off-center\ntriangle wave and a shifted sawtooth,\nat least with the LM324."
- note added: "Q5 cannot be replaced by a \nmosfet due to the parasitic\ndiode inside a FET. Do replace\nit for some crunchy wave-\nshaping, though."
- note added: "TODO: jumper?"
- note added: "remove the DC offset. This doesn't matter for normal\noperation, but for DCO operation, where R26-R29 have\nno effect and thus, the signal is not centered."
- note removed: "Just a hacky way of applying an\nadjustable voltage with an adjustable\ninner resistance. Replace R26-R28\nby a 100-200k trimmer and leave\nout R29 completely if you want.\nOr just spare everything and connect\nthe (+) pin to GNDREF.\nThat will cause a slightly off-center\ntriangle wave and a shifted sawtooth,\nat least with the LM324."
- note removed: "Q5 cannot be\nreplaced by a \nmosfet due to\nthe parasitic\ndiode inside a\nFET. Do replace\nit for some\ncrunchy wave-\nshaping, though."
- note removed: "remove the DC offset. This doesn't matter for normal\noperation, but for DCO operation, where R27-R30 have\nno effect and thus, the signal is not centered."
- moved on the sheet: C1, C2, C?, D1, JP1, R1, R10, R11, R12, R13, R2, R3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

Commit message: soft sync
Parts:
- added J?: Conn_01x01_Male, symbol Connector:Conn_01x01_Male
Connections:
- net at R29.1, R30.1, U2.5 (+): now also J?.1 (Pin_1)
Other:
- note added: "For another interesting square wave\nvariation, connect ctl_override (JP5,\npin 3) to J4. Then play around with\nthe PWM voltage and watch rmpulse.\n\nApply narrow periodic pull-to-GND\npulse to U2's pin5 (J?) for soft sync."
- note removed: "For another interesting square wave\nvariation, connect ctl_override (JP5,\npin 3) to J4. Then play around with\nthe PWM voltage and watch rmpulse."
Changed lines of the file:
@@
 TODO:\nraw pulse?
 Text Notes 5300 7475 0    50   ~ 0
-For another interesting square wave\nvariation, connect ctl_override (JP5,\npin 3) to J4. Then play around with\nthe PWM voltage and watch rmpulse.
+For another interesting square wave\nvariation, connect ctl_override (JP5,\npin 3) to J4. Then play around with\nthe PWM voltage and watch rmpulse.\n\nApply narrow periodic pull-to-GND\npulse to U2's pin5 (J?) for soft sync.
 Wire Notes Line
 	6075 6625 3650 6625
@@
 Text Notes 2725 6725 1    50   ~ 0
 TODO: jumper?
+$Comp
+L Connector:Conn_01x01_Male J?
+U 1 1 5D4BF3A9
+P 2825 6600
+F 0 "J?" V 2775 6550 50  0000 L CNN
+F 1 "Conn_01x01_Male" V 2978 6644 50  0001 L CNN
+F 2 "" H 2825 6600 50  0001 C CNN
+F 3 "~" H 2825 6600 50  0001 C CNN
+	1    2825 6600
+	0    1    1    0
+$EndComp
+Connection ~ 2825 6800
 $EndSCHEMATC
