File: hardware/vco_mk1/vco_mk1/vco_mk1.sch (KiCad schematic (older format))
At the start: 82 parts, among them J1 power supply, J2 control in, J3 signal out, J4 Conn_01x03_Male, J5 BCM847 breakout socket, Q1 BCM847, Q2 BC547, Q3 BC547, Q4 2N7000, Q5 BC547, Q6 BC327, U1 LM324, U2 LM324, U3 74HC86

Commit message: confirmed: vco core and waveform generation (and fixes)
Parts:
- added R48: 10k, Resistor_SMD:R_0805_2012Metric_Pad1.15x1.40mm_HandSolder, symbol Device:R
- gave numbers to parts that had none: 4
Connections:
- net V_pwm: now also U2.9 (-); no longer U2.10 (+)
- net at C13.1, JP6.2 (B), R32.1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: now also U2.10 (+); no longer U2.9 (-)
- net at R44.1, U3.13: now also R48.2; no longer JP5.4 (Pin_4)
- new net: JP5.4 (Pin_4), R48.1
Other:
- note added: "For another interesting square wave\nvariation, connect ctl_override (JP5,\npin 3) to J4. Then play around with\nthe PWM voltage and watch rmpulse.\n\nApply narrow periodic pull-to-GND\npulse to U2's pin5 (J6) for soft sync."
- note added: "connected to var_vsource\n(probably in error)"
- note added: "todo: maybe 47n?"
- note removed: "For another interesting square wave\nvariation, connect ctl_override (JP5,\npin 3) to J4. Then play around with\nthe PWM voltage and watch rmpulse.\n\nApply narrow periodic pull-to-GND\npulse to U2's pin5 (J?) for soft sync."
Changed lines of the file:
@@
-$Comp
-L Amplifier_Operational:LM324 U2
-U 3 1 5D62893A
-P 4975 4975
-F 0 "U2" H 5050 5150 50  0000 C CNN
-F 1 "LM324" H 4950 4975 50  0000 C CNN
-F 2 "Package_DIP:DIP-14_W7.62mm" H 4925 5075 50  0001 C CNN
-F 3 "http://www.ti.com/lit/ds/symlink/lm2902-n.pdf" H 5025 5175 50  0001 C CNN
-	3    4975 4975
-	1    0    0    -1
-$EndComp
 $Comp
 L Amplifier_Operational:LM324 U2
@@
 pulse
 Wire Wire Line
-	8425 5550 8425 6325
+	8425 5550 8425 5800
 Wire Wire Line
 	8425 6325 9025 6325
@@
 	5675 5200 2875 5200
 $Comp
-L Device:R R?
+L Device:R R47
 U 1 1 5D53B3BE
 P 3550 5825
-F 0 "R?" H 3425 5975 50  0000 L CNN
+F 0 "R47" H 3425 5975 50  0000 L CNN
 F 1 "none" V 3550 5725 50  0000 L CNN
 F 2 "" V 3480 5825 50  0001 C CNN
@@
 $EndComp
 $Comp
-L power:GNDREF #PWR?
+L power:GNDREF #PWR041
 U 1 1 5D54168D
 P 3550 5975
-F 0 "#PWR?" H 3550 5725 50  0001 C CNN
+F 0 "#PWR041" H 3550 5725 50  0001 C CNN
 F 1 "GNDREF" H 3555 5802 50  0001 C CNN
 F 2 "" H 3550 5975 50  0001 C CNN
@@
 do not equip R?\n10-100k are fine,\nbut R33+Q5 are\nenough for our\npurpose.
 $Comp
-L Device:C C?
+L Device:C C13
 U 1 1 5D49B6B5
 P 3225 5600
-F 0 "C?" V 3275 5700 50  0000 C CNN
+F 0 "C13" V 3275 5700 50  0000 C CNN
 F 1 "100n" V 3175 5475 50  0000 C CNN
 F 2 "Capacitor_SMD:C_0805_2012Metric_Pad1.15x1.40mm_HandSolder" H 3263 5450 50  0001 C CNN
@@
 TODO:\nraw pulse?
 Text Notes 5300 7475 0    50   ~ 0
-For another interesting square wave\nvariation, connect ctl_override (JP5,\npin 3) to J4. Then play around with\nthe PWM voltage and watch rmpulse.\n\nApply narrow periodic pull-to-GND\npulse to U2's pin5 (J?) for soft sync.
+For another interesting square wave\nvariation, connect ctl_override (JP5,\npin 3) to J4. Then play around with\nthe PWM voltage and watch rmpulse.\n\nApply narrow periodic pull-to-GND\npulse to U2's pin5 (J6) for soft sync.
 Wire Notes Line
 	6075 6625 3650 6625
@@
 	2875 5200 2875 5500
 $Comp
-L Jumper:Jumper_2_Open JP?
+L Jumper:Jumper_2_Open JP6
 U 1 1 5D692292
 P 3225 5400
-F 0 "JP?" H 3050 5475 50  0000 C CNN
+F 0 "JP6" H 3050 5475 50  0000 C CNN
 F 1 "Jumper_2_Open" H 3225 5544 50  0001 C CNN
 F 2 "" H 3225 5400 50  0001 C CNN
@@
 TODO: jumper?
 $Comp
-L Connector:Conn_01x01_Male J?
+L Connector:Conn_01x01_Male J6
 U 1 1 5D4BF3A9
 P 2825 6600
-F 0 "J?" V 2775 6550 50  0000 L CNN
+F 0 "J6" V 2775 6550 50  0000 L CNN
 F 1 "Conn_01x01_Male" V 2978 6644 50  0001 L CNN
 F 2 "" H 2825 6600 50  0001 C CNN
@@
 $EndComp
 Connection ~ 2825 6800
+$Comp
+L Device:R R48
+U 1 1 5D58016A
+P 8425 5950
+F 0 "R48" H 8450 5800 50  0000 L CNN
+F 1 "10k" V 8425 5875 50  0000 L CNN
+F 2 "Resistor_SMD:R_0805_2012Metric_Pad1.15x1.40mm_HandSolder" V 8355 5950 50  0001 C CNN
+F 3 "~" H 8425 5950 50  0001 C CNN
+	1    8425 5950
+	-1   0    0    1
+$EndComp
+Wire Wire Line
+	8425 6100 8425 6325
+Wire Notes Line
+	1825 7450 1625 7450
+Wire Notes Line
+	1825 6800 1825 7450
+Text Notes 1900 7225 1    20   ~ 0
+connected to var_vsource\n(probably in error)
+Text Notes 10500 3275 0    50   ~ 0
+todo: maybe 47n?
+$Comp
+L Amplifier_Operational:LM324 U2
+U 3 1 5D62893A
+P 4975 4975
+F 0 "U2" H 5075 4825 50  0000 C CNN
+F 1 "LM324" H 4950 4975 50  0000 C CNN
+F 2 "Package_DIP:DIP-14_W7.62mm" H 4925 5075 50  0001 C CNN
+F 3 "http://www.ti.com/lit/ds/symlink/lm2902-n.pdf" H 5025 5175 50  0001 C CNN
+	3    4975 4975
+	1    0    0    1
+$EndComp
 $EndSCHEMATC

Commit message: confirmed: expo
Parts:
- added R? (x2): 1Meg, Resistor_SMD:R_0805_2012Metric_Pad1.15x1.40mm_HandSolder, symbol Device:R
- C3: value 1n -> 2.2n
- R42: value TODO -> 1k
Connections:
- net VCC: now also R?.1; no longer R1.1
- net VEE: now also R?.2; no longer R1.3
- new net: R1.1, R?.2
- new net: R1.3, R?.1
Other:
- note added: "10k"
- note added: "111k"
- note added: "1Meg"
- note added: "2x 1Meg for Q4 compensation\nless (possibly 0 Ohm) for other\npurposes"
- note added: "Rs that can scale together:\nx: R14, x: R19, 1/x: R13\nTODO test!"
- note added: "TODO: test 1n"
Changed lines of the file:
@@
 P 10650 1200
 F 0 "R42" H 10581 1246 50  0000 R CNN
-F 1 "TODO" V 10650 1300 50  0000 R CNN
+F 1 "1k" V 10650 1250 50  0000 R CNN
 F 2 "Potentiometer_THT:Potentiometer_Runtron_RM-065_Vertical" H 10650 1200 50  0001 C CNN
 F 3 "~" H 10650 1200 50  0001 C CNN
@@
 L power:VCC #PWR01
 U 1 1 5E0402DF
-P 825 3350
-F 0 "#PWR01" H 825 3200 50  0001 C CNN
-F 1 "VCC" H 725 3425 50  0000 C CNN
-F 2 "" H 825 3350 50  0001 C CNN
-F 3 "" H 825 3350 50  0001 C CNN
-	1    825  3350
+P 825 3050
+F 0 "#PWR01" H 825 2900 50  0001 C CNN
+F 1 "VCC" H 725 3125 50  0000 C CNN
+F 2 "" H 825 3050 50  0001 C CNN
+F 3 "" H 825 3050 50  0001 C CNN
+	1    825  3050
 	1    0    0    -1
 $EndComp
@@
 L power:VEE #PWR02
 U 1 1 5E03FE83
-P 825 3650
-F 0 "#PWR02" H 825 3500 50  0001 C CNN
-F 1 "VEE" H 925 3725 50  0000 C CNN
-F 2 "" H 825 3650 50  0001 C CNN
-F 3 "" H 825 3650 50  0001 C CNN
-	1    825  3650
+P 825 3950
+F 0 "#PWR02" H 825 3800 50  0001 C CNN
+F 1 "VEE" H 925 4025 50  0000 C CNN
+F 2 "" H 825 3950 50  0001 C CNN
+F 3 "" H 825 3950 50  0001 C CNN
+	1    825  3950
 	-1   0    0    1
 $EndComp
@@
 P 4900 2900
 F 0 "C3" V 4648 2900 50  0000 C CNN
-F 1 "1n" V 4739 2900 50  0000 C CNN
+F 1 "2.2n" V 4739 2900 50  0000 C CNN
 F 2 "Capacitor_SMD:C_0805_2012Metric_Pad1.15x1.40mm_HandSolder" H 4938 2750 50  0001 C CNN
 F 3 "~" H 4900 2900 50  0001 C CNN
@@
 U 1 1 5D41CBAE
 P 5650 2725
-F 0 "R15" H 5720 2771 50  0000 L CNN
-F 1 "1k" H 5720 2680 50  0000 L CNN
+F 0 "R15" H 5725 2725 50  0000 L CNN
+F 1 "1k" V 5650 2675 50  0000 L CNN
 F 2 "Resistor_SMD:R_0805_2012Metric_Pad1.15x1.40mm_HandSolder" V 5580 2725 50  0001 C CNN
 F 3 "~" H 5650 2725 50  0001 C CNN
@@
 	1    0    0    1
 $EndComp
+Text Notes 4650 2600 0    50   ~ 0
+TODO: test 1n
+$Comp
+L Device:R R?
+U 1 1 5D73F6A7
+P 825 3200
+F 0 "R?" H 650 3200 50  0000 L CNN
+F 1 "1Meg" V 825 3100 50  0000 L CNN
+F 2 "Resistor_SMD:R_0805_2012Metric_Pad1.15x1.40mm_HandSolder" V 755 3200 50  0001 C CNN
+F 3 "~" H 825 3200 50  0001 C CNN
+	1    825  3200
+	1    0    0    -1
+$EndComp
+$Comp
+L Device:R R?
+U 1 1 5D7480C4
+P 825 3800
+F 0 "R?" H 650 3800 50  0000 L CNN
+F 1 "1Meg" V 825 3700 50  0000 L CNN
+F 2 "Resistor_SMD:R_0805_2012Metric_Pad1.15x1.40mm_HandSolder" V 755 3800 50  0001 C CNN
+F 3 "~" H 825 3800 50  0001 C CNN
+	1    825  3800
+	1    0    0    -1
+$EndComp
+Text Notes 675  3750 1    25   ~ 0
+2x 1Meg for Q4 compensation\nless (possibly 0 Ohm) for other\npurposes
+Text Notes 5500 1625 0    50   ~ 0
+1Meg
+Text Notes 7225 1250 0    50   ~ 0
+111k
+Text Notes 7875 2325 0    50   ~ 0
+Rs that can scale together:\nx: R14, x: R19, 1/x: R13\nTODO test!
+Text Notes 3525 3400 0    50   ~ 0
+10k
 $EndSCHEMATC
