File: hardware/vco_mk1/vco_mk1/vco_mk1.sch (KiCad schematic (older format))
At the start: 87 parts, among them J1 power supply, J2 control in, J3 signal out, J4 Conn_01x03_Male, J5 BCM847 breakout socket, J6 Conn_01x01_Male, Q1 BCM847, Q2 BC547, Q3 BC547, Q4 2N7000, Q5 BC547, Q6 BC327, U1 LM324, U2 LM324, U3 74HC86

Commit message: footprints
Parts:
- J6: footprint (none) -> Connector_PinHeader_2.54mm:PinHeader_1x01_P2.54mm_Vertical
- JP5: footprint (none) -> footprints:SolderDipJumper2alt
- R34: footprint (none) -> Resistor_SMD:R_0805_2012Metric_Pad1.15x1.40mm_HandSolder
Changed lines of the file:
@@
 F 0 "R34" H 3425 5975 50  0000 L CNN
 F 1 "none" V 3550 5725 50  0000 L CNN
-F 2 "" V 3480 5825 50  0001 C CNN
+F 2 "Resistor_SMD:R_0805_2012Metric_Pad1.15x1.40mm_HandSolder" V 3480 5825 50  0001 C CNN
 F 3 "~" H 3550 5825 50  0001 C CNN
 	1    3550 5825
@@
 F 0 "JP5" H 3050 5475 50  0000 C CNN
 F 1 "Jumper_2_Open" H 3225 5544 50  0001 C CNN
-F 2 "" H 3225 5400 50  0001 C CNN
+F 2 "footprints:SolderDipJumper2alt" H 3225 5400 50  0001 C CNN
 F 3 "~" H 3225 5400 50  0001 C CNN
 	1    3225 5400
@@
 F 0 "J6" V 2775 6550 50  0000 L CNN
 F 1 "Conn_01x01_Male" V 2978 6644 50  0001 L CNN
-F 2 "" H 2825 6600 50  0001 C CNN
+F 2 "Connector_PinHeader_2.54mm:PinHeader_1x01_P2.54mm_Vertical" H 2825 6600 50  0001 C CNN
 F 3 "~" H 2825 6600 50  0001 C CNN
 	1    2825 6600

Commit message: placement 1/3
Connections:
- net C2: now also U1.2 (-); no longer U1.9 (-)
- net V_control_raw: now also U1.9 (-); no longer U1.2 (-)
- net V_expo: now also U1.1; no longer U1.8
- net at R8.2, R9.1: now also U1.8; no longer U1.1
Other:
- moved on the sheet: U1A, U1C
Changed lines of the file:
@@
 L Amplifier_Operational:LM324 U1
 U 3 1 5D5EBF6F
-P 7350 1825
-F 0 "U1" H 7450 1675 50  0000 C CNN
-F 1 "LM324" H 7325 1825 50  0000 C CNN
-F 2 "Package_DIP:DIP-14_W7.62mm" H 7300 1925 50  0001 C CNN
-F 3 "http://www.ti.com/lit/ds/symlink/lm2902-n.pdf" H 7400 2025 50  0001 C CNN
-	3    7350 1825
+P 2050 2400
+F 0 "U1" H 2150 2250 50  0000 C CNN
+F 1 "LM324" H 2025 2400 50  0000 C CNN
+F 2 "Package_DIP:DIP-14_W7.62mm" H 2000 2500 50  0001 C CNN
+F 3 "http://www.ti.com/lit/ds/symlink/lm2902-n.pdf" H 2100 2600 50  0001 C CNN
+	3    2050 2400
 	1    0    0    1
 $EndComp
@@
 L Amplifier_Operational:LM324 U1
 U 1 1 5D5E9E8D
-P 2050 2400
-F 0 "U1" H 2150 2250 50  0000 C CNN
-F 1 "LM324" H 2025 2400 50  0000 C CNN
-F 2 "Package_DIP:DIP-14_W7.62mm" H 2000 2500 50  0001 C CNN
-F 3 "http://www.ti.com/lit/ds/symlink/lm2902-n.pdf" H 2100 2600 50  0001 C CNN
-	1    2050 2400
+P 7350 1825
+F 0 "U1" H 7450 1675 50  0000 C CNN
+F 1 "LM324" H 7325 1825 50  0000 C CNN
+F 2 "Package_DIP:DIP-14_W7.62mm" H 7300 1925 50  0001 C CNN
+F 3 "http://www.ti.com/lit/ds/symlink/lm2902-n.pdf" H 7400 2025 50  0001 C CNN
+	1    7350 1825
 	1    0    0    1
 $EndComp
