File: hardware/vco_mk1/vco_mk1/vco_mk1.kicad_pcb (KiCad board)
At the start: 2 copper layers, 87 parts, among them J1 power supply, J2 control in, J3 signal out, J4 Conn_01x03_Male, J5 BCM847 breakout socket, J6 Conn_01x01_Male, Q1 BCM847, Q2 BC547, Q3 BC547, Q4 2N7000, Q5 BC547, Q6 BC327, U1 LM324, U2 LM324, U3 74HC86

Commit message: grouped all components into logical groups
Parts:
- moved JP1 267.5 mm to (308.6, 47.8), turned to 270 degrees
- moved JP2 265.4 mm to (316.7, 53.1)
- moved JP4 217.8 mm to (250.7, 146.6)
- moved R10 214.0 mm to (306.3, 27.7), turned to 0 degrees
- moved R5 207.7 mm to (265.7, 20.8), turned to 0 degrees
- moved R4 205.9 mm to (265.7, 23.4)
- moved D1 188.7 mm to (304.8, 57.4)
- moved C6 176.3 mm to (281.4, 134.1)
- moved C7 175.9 mm to (276.6, 133.9)
- moved R15 172.0 mm to (306.1, 53.1), turned to 180 degrees
- moved R13 168.7 mm to (305.6, 49.0), turned to 180 degrees
- moved R11 164.8 mm to (307.6, 31.0)
- moved R9 164.1 mm to (302.8, 29.2)
- moved JP5 162.5 mm to (193.3, 128.5)
- moved R14 162.4 mm to (311.7, 49.0)
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Routing:
- net +5V: track 0.00 -> 19.5 mm
- net GNDD: track 0.00 -> 3.63 mm

Commit message: rough layout for U3
Parts:
- moved R52 59.3 mm to (145.5, 26.2), turned to 180 degrees
- moved JP6 27.1 mm to (145.8, 37.8), turned to 270 degrees
- moved R48 15.9 mm to (138.2, 37.3)
- moved R44 15.8 mm to (123.7, 27.2), turned to 270 degrees
- moved R46 13.4 mm to (126.0, 32.3), turned to 90 degrees
- moved R51 13.1 mm to (141.7, 29.0), turned to 180 degrees
- moved R50 7.47 mm to (138.2, 32.0), turned to 90 degrees
- moved Q6 7.27 mm to (141.5, 31.8), turned to 270 degrees
- moved R47 3.23 mm to (138.2, 24.4), turned to 90 degrees
- moved R42 2.03 mm to (126.0, 27.2)
- moved R43 1.02 mm to (123.7, 32.3), turned to 270 degrees
- moved R41 0.51 mm to (125.0, 22.9)
Routing:
- net Net-(R47-Pad1): track 0.00 -> 19.3 mm
- net +5V: track 19.5 -> 35.4 mm
- net Net-(U3-Pad10): track 0.00 -> 14.7 mm
- net VCC: track 0.00 -> 10.5 mm
- net Net-(R42-Pad1): track 0.00 -> 10.2 mm
- net Net-(R41-Pad1): track 0.00 -> 6.73 mm
- net Net-(R43-Pad1): track 0.00 -> 5.52 mm
- net VEE: track 0.00 -> 3.71 mm
- net Net-(Q6-Pad2): track 0.00 -> 3.31 mm
- net Net-(JP6-Pad1): track 0.00 -> 3.11 mm
- net Net-(U3-Pad3): track 0.00 -> 2.54 mm
- net Net-(R48-Pad1): track 0.00 -> 2.39 mm
- net Net-(R50-Pad2): track 0.00 -> 2.29 mm
Other:
- net class Power: clearance 1 -> 0.2; trace_width 0.2 -> 0.4

Commit message: rough layout for U2
Parts:
- moved R35 74.5 mm to (320.5, 132.1), turned to 90 degrees
- moved R40 68.4 mm to (315.7, 140.7), turned to 270 degrees
- moved Q5 67.8 mm to (316.7, 131.6), turned to 270 degrees
- moved R39 65.8 mm to (319.3, 139.7), turned to 180 degrees
- moved R37 55.8 mm to (316.7, 136.7), turned to 180 degrees
- moved R32 54.5 mm to (299.2, 132.3), turned to 90 degrees
- moved R33 52.9 mm to (306.6, 144.5), turned to 0 degrees
- moved R38 51.9 mm to (315.7, 128.0)
- moved C4 50.0 mm to (304.5, 123.4), turned to 180 degrees
- moved R27 49.3 mm to (310.4, 144.5)
- moved R36 46.0 mm to (317.8, 128.0), turned to 270 degrees
- moved U2 44.6 mm to (305.8, 126.5)
- moved C7 44.0 mm to (320.5, 135.9)
- moved Q4 44.0 mm to (293.6, 133.1)
- moved R31 43.9 mm to (303.3, 144.0)
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Routing:
- net VCC: track 10.5 -> 37.1 mm
- net GND: track 10.7 -> 35.8 mm
- net square_ctl: track 0.00 -> 23.2 mm
- net (no net): track 0.00 -> 22.7 mm
- net Net-(R23-Pad1): track 0.00 -> 19.1 mm, vias 0 -> 1
- net Net-(R27-Pad1): track 0.00 -> 18.0 mm
- net VEE: track 3.71 -> 21.5 mm
- net Net-(C5-Pad1): track 0.00 -> 16.3 mm, vias 0 -> 1
- net Net-(J6-Pad1): track 0.00 -> 10.9 mm
- net Net-(C4-Pad2): track 0.00 -> 10.2 mm
- net Net-(R28-Pad2): track 0.00 -> 10.1 mm
- net Net-(Q5-Pad1): track 0.00 -> 9.75 mm
- net Net-(Q4-Pad3): track 0.00 -> 6.01 mm
- net ctl_override: track 0.00 -> 5.64 mm
- net Net-(R28-Pad3): track 0.00 -> 5.03 mm
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
Commit message: rough layout for U1
Parts:
- moved R4 208.6 mm to (62.2, 69.6)
- moved R5 208.6 mm to (62.2, 67.1)
- moved R6 208.6 mm to (62.2, 64.5)
- moved R18 172.0 mm to (74.9, 64.5)
- moved R19 172.0 mm to (74.9, 67.3)
- moved R20 172.0 mm to (74.9, 69.8)
- moved R2 23.4 mm to (278.6, 32.8), turned to 90 degrees
- moved R3 23.1 mm to (273.8, 37.8), turned to 180 degrees
- moved C1 19.3 mm to (259.6, 35.3), turned to 180 degrees
- moved R7 17.0 mm to (258.6, 31.2), turned to 90 degrees
- moved R16 16.3 mm to (260.9, 38.9), turned to 270 degrees
- moved R17 13.1 mm to (258.6, 44.5), turned to 270 degrees
- moved C2 10.0 mm to (273.8, 40.4)
- moved R21 9.57 mm to (282.2, 51.6), turned to 180 degrees
- moved R8 8.49 mm to (260.9, 31.2), turned to 90 degrees
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Routing:
- net GND: track 35.8 -> 54.7 mm
- net VCC: track 37.1 -> 44.2 mm
- net C1: track 13.7 -> 19.7 mm
- net VEE: track 21.5 -> 26.9 mm
- net V_control_raw: track 0.00 -> 4.78 mm
- net Net-(C3-Pad1): track 0.00 -> 4.58 mm
- net Net-(R2-Pad3): track 0.00 -> 3.80 mm
- net Net-(R24-Pad1): track 4.13 -> 7.25 mm
- net (no net): track 22.7 -> 20.0 mm
- net Net-(R8-Pad2): track 0.00 -> 2.29 mm
- net Net-(C5-Pad1): track 16.3 -> 17.8 mm
- net sawtooth: track 2.49 -> 4.07 mm
- net Net-(R36-Pad2): track 4.32 -> 5.60 mm

Commit message: improved double transistor
Parts:
- moved Q2 0.14 mm to (263.8, -4.45)
- moved Q3 0.14 mm to (267.5, -6.99)
- moved Q1 0.06 mm to (265.7, -1.59)
Routing:
- net C2: track 16.9 -> 17.6 mm
- net E: track 18.5 -> 19.1 mm

Commit message: first pass layout clusterfuck
Parts:
- moved C13 182.0 mm to (197.1, 136.4), turned to 90 degrees
- moved C11 180.2 mm to (201.9, 136.4), turned to 270 degrees
- moved C9 168.2 mm to (206.1, 118.0)
- moved C10 164.2 mm to (195.7, 131.6), turned to 90 degrees
- moved C12 162.4 mm to (198.6, 130.9), turned to 270 degrees
- moved J6 161.5 mm to (179.6, 136.4)
- moved R12 161.4 mm to (165.1, 94.5), turned to 270 degrees
- moved J3 159.7 mm to (204.9, 122.3)
- moved R11 156.2 mm to (162.8, 89.7), turned to 90 degrees
- moved R10 154.8 mm to (165.1, 91.2), turned to 90 degrees
- moved JP2 144.9 mm to (178.3, 95.8), turned to 90 degrees
- moved JP1 142.8 mm to (171.4, 87.4)
- moved R13 142.8 mm to (168.4, 88.6)
- moved R14 142.8 mm to (174.5, 88.6)
- moved R15 142.8 mm to (168.9, 92.7)
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Routing:
- net GND: track 54.9 -> 177.0 mm, vias 0 -> 2
- net VEE: track 26.9 -> 141.2 mm, vias 0 -> 1
- net ctl_override: track 5.64 -> 88.1 mm, vias 0 -> 1
- net VCC: track 44.2 -> 125.9 mm, vias 0 -> 1
- net var_vsource: track 0.00 -> 68.4 mm, vias 0 -> 2
- net V_pwm: track 0.00 -> 68.0 mm
- net C2: track 17.6 -> 75.9 mm, vias 0 -> 1
- net V_expo: track 2.01 -> 60.0 mm, vias 0 -> 2
- net triangle: track 3.15 -> 57.5 mm, vias 0 -> 1
- net Net-(R1-Pad2): track 0.00 -> 53.6 mm
- net V_control_raw: track 4.78 -> 58.3 mm
- net sawtooth: track 4.07 -> 49.0 mm, vias 0 -> 2
- net rmpulse: track 0.00 -> 40.1 mm, vias 0 -> 4
- net square_ctl: track 23.2 -> 63.0 mm
- net Net-(R40-Pad2): track 0.00 -> 33.7 mm, vias 0 -> 1
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- added copper zone on B.Cu, net GND
- added copper zone on F.Cu, net GND
Other:
- board outline added: 50 x 80 mm

Commit message: improved grounding a bit
Routing:
- net saw_ctl: track 19.1 -> 20.3 mm
- net GND: vias 2 -> 4
Changed lines of the file:
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@@
     (thickness 1.6)
     (drawings 4)
-    (tracks 811)
+    (tracks 816)
     (zones 0)
     (modules 87)
@@
   (segment (start 165.119999 103.612001) (end 165.119999 96.500001) (width 0.4) (layer B.Cu) (net 2))
   (segment (start 163.83 104.902) (end 165.119999 103.612001) (width 0.4) (layer B.Cu) (net 2))
-  (via (at 197.104 129.032) (size 1) (drill 0.6) (layers F.Cu B.Cu) (net 2))
   (segment (start 200.473001 112.952999) (end 201.676 114.155998) (width 0.4) (layer B.Cu) (net 2))
   (segment (start 199.608999 112.952999) (end 200.473001 112.952999) (width 0.4) (layer B.Cu) (net 2))
@@
   (segment (start 190.389 135.561) (end 192.099 135.561) (width 0.4) (layer F.Cu) (net 2))
   (segment (start 192.099 135.561) (end 192.151 135.509) (width 0.4) (layer F.Cu) (net 2))
+  (via (at 170.688 107.696) (size 1) (drill 0.6) (layers F.Cu B.Cu) (net 2))
+  (via (at 202.057 109.093) (size 1) (drill 0.6) (layers F.Cu B.Cu) (net 2))
+  (via (at 207.899 115.189) (size 1) (drill 0.6) (layers F.Cu B.Cu) (net 2))
   (segment (start 197.835 93.731) (end 200.05 95.946) (width 0.4) (layer F.Cu) (net 3))
   (segment (start 197.835 93.152) (end 197.835 93.731) (width 0.4) (layer F.Cu) (net 3))
@@
   (segment (start 195.888894 106.489602) (end 195.888893 108.067639) (width 0.2) (layer F.Cu) (net 42))
   (segment (start 196.596 106.489602) (end 195.888894 106.489602) (width 0.2) (layer F.Cu) (net 42))
-  (segment (start 205.994 101.346) (end 201.676 105.664) (width 0.2) (layer F.Cu) (net 43))
-  (segment (start 201.676 116.705) (end 200.278 118.103) (width 0.2) (layer F.Cu) (net 43))
-  (segment (start 201.676 105.664) (end 201.676 116.705) (width 0.2) (layer F.Cu) (net 43))
+  (segment (start 200.278 118.103) (end 206.248 112.133) (width 0.2) (layer F.Cu) (net 43))
+  (segment (start 206.248 112.133) (end 206.248 108.458) (width 0.2) (layer F.Cu) (net 43))
+  (segment (start 205.07329 102.26671) (end 205.994 101.346) (width 0.2) (layer F.Cu) (net 43))
+  (segment (start 204.84399 102.49601) (end 205.07329 102.26671) (width 0.2) (layer F.Cu) (net 43))
+  (segment (start 204.84399 107.05399) (end 204.84399 102.49601) (width 0.2) (layer F.Cu) (net 43))
+  (segment (start 206.248 108.458) (end 204.84399 107.05399) (width 0.2) (layer F.Cu) (net 43))
   (segment (start 198.771 96.717) (end 198 95.946) (width 0.2) (layer F.Cu) (net 44))
   (segment (start 198.771 98.74) (end 198.771 96.717) (width 0.2) (layer F.Cu) (net 44))

Commit message: added windfisch
Parts:
- added FISCH: LOGO, footprints:windfisch, F.Cu at (165.2, 66.3)
