File: hardware/vco_mk1/vco_mk1/vco_mk1.kicad_pcb (KiCad board)
At the start: 2 copper layers, 160 x 100 mm, 72 parts, among them J1 power supply, J2 control in, J3 signal out, J4 ringmod in, J5 BCM847 breakout socket, Q1 BCM847, Q2 BC547, Q3 BC547, Q4 2N7000, Q5 BC547, U1 LM324, U2 LM324, U3 74HC86

Commit message: layout wip2
Parts:
- removed Q1: BCM847, Package_TO_SOT_SMD:SOT-363_SC-70-6
- JP2, JP3: moved to B.Cu
- R19, R42: moved to F.Cu
- moved JP2 347.3 mm to (342.0, 105.9), turned to 270 degrees
- moved JP3 345.2 mm to (346.6, 120.2), turned to 180 degrees
- moved J5 330.4 mm to (348.1, 110.7), turned to 180 degrees
- moved Q2 326.8 mm to (346.2, 114.4), turned to 90 degrees
- moved Q3 318.9 mm to (342.4, 111.8), turned to 270 degrees
- moved R15 308.3 mm to (345.5, 109.4), turned to 135 degrees
- moved R19 306.1 mm to (343.6, 96.7), turned to 90 degrees
- moved R2 306.0 mm to (359.3, 113.3)
- moved R10 306.0 mm to (354.7, 111.1)
- moved R13 306.0 mm to (351.7, 121.3)
- moved U1 306.0 mm to (360.8, 106.7)
- moved C2 306.0 mm to (351.9, 101.2)
- moved C3 306.0 mm to (346.9, 104.6)
- moved R1 306.0 mm to (357.5, 95.1)
- moved R12 306.0 mm to (351.7, 119.3)
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Connections:
- J2 pad 11: V_lin_pitchmod_3 -> ctl_override
- J2 pad 12: V_lin_pitchmod_2 -> V_pwm
- J2 pad 13: V_lin_pitchmod_1 -> GND
- J2 pad 2: V_control -> GND
- J2 pad 3: V_control_2 -> V_control
- J2 pad 4: V_control_3 -> V_lin_pitchmod_1
- J2 pad 5: V_control_raw -> V_control_2
- J2 pad 6: ctl_override -> V_lin_pitchmod_2
- J2 pad 7: GND -> V_control_3
- J2 pad 8: GND -> V_lin_pitchmod_3
- J2 pad 9: V_pwm -> V_control_raw
Routing:
- net GND: track 19.2 -> 123.0 mm
- net VCC: track 18.6 -> 100.9 mm
- net VEE: track 31.5 -> 113.1 mm
- net triangle: track 7.58 -> 41.6 mm
- net Net-(R11-Pad2): track 0.00 -> 29.6 mm
- net ctl_override: track 0.00 -> 23.7 mm
- net Net-(R29-Pad1): track 0.00 -> 19.6 mm
- net Net-(JP5-Pad4): track 3.89 -> 19.9 mm
- net V_control_raw: track 2.38 -> 18.1 mm
- net B1: track 2.13 -> 15.8 mm
- net Net-(R32-Pad2): track 0.00 -> 9.57 mm
- net Net-(R6-Pad2): track 2.39 -> 11.7 mm
- net Net-(R26-Pad2): track 0.00 -> 7.87 mm
- net Net-(Q5-Pad2): track 0.00 -> 7.14 mm
- net Net-(C8-Pad2): track 0.00 -> 6.77 mm
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
Commit message: more fiddling
Parts:
- moved J4 265.6 mm to (162.0, 104.1), turned to 180 degrees
- moved U3 260.9 mm to (166.3, 104.4), turned to 270 degrees
- moved C11 255.4 mm to (167.8, 108.4), turned to 180 degrees
- moved R37 252.9 mm to (179.0, 100.1), turned to 0 degrees
- moved R38 250.7 mm to (179.0, 102.1), turned to 0 degrees
- moved Q5 249.3 mm to (160.7, 123.2), turned to 180 degrees
- moved JP5 249.2 mm to (166.5, 116.3), turned to 180 degrees
- moved R31 248.9 mm to (165.0, 118.4), turned to 0 degrees
- moved R40 248.7 mm to (176.4, 106.4), turned to 0 degrees
- moved R33 247.1 mm to (160.4, 126.0), turned to 180 degrees
- moved R39 246.7 mm to (176.4, 108.4), turned to 0 degrees
- moved R32 245.4 mm to (160.4, 127.9), turned to 0 degrees
- moved R34 244.9 mm to (165.5, 122.2), turned to 90 degrees
- moved C7 244.2 mm to (149.0, 135.1), turned to 270 degrees
- moved R41 243.2 mm to (179.5, 108.9), turned to 90 degrees
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Routing:
- net VCC: track 100.9 -> 185.1 mm
- net var_vsource: track 0.00 -> 78.0 mm, vias 0 -> 2
- net V_expo: track 6.28 -> 79.7 mm, vias 0 -> 2
- net VEE: track 113.1 -> 178.3 mm
- net C2: track 15.7 -> 78.2 mm, vias 0 -> 4
- net C1: track 25.4 -> 45.4 mm, vias 0 -> 2
- net Net-(JP5-Pad1): track 0.00 -> 13.0 mm
- net GND: track 123.0 -> 132.9 mm, vias 0 -> 1
- net triangle: track 41.6 -> 48.8 mm
- net Net-(R36-Pad2): track 0.00 -> 3.72 mm
Other:
- board size 160 x 100 mm -> 481.8 x 143.2 mm

Commit message: placement 1/3
Parts:
- added C12: 100n, Capacitor_SMD:C_0805_2012Metric_Pad1.15x1.40mm_HandSolder, F.Cu at (151.0, 53.7)
- added C13: 100n, Capacitor_SMD:C_0805_2012Metric_Pad1.15x1.40mm_HandSolder, F.Cu at (160.6, 31.3)
- added J6: Conn_01x01_Male, Connector_PinHeader_2.54mm:PinHeader_1x01_P2.54mm_Vertical, F.Cu at (179.5, 30.5)
- added JP6: ringmod config, footprints:SolderDipJumper4alt, F.Cu at (108.3, 58.6)
- added Q1: BCM847, Package_TO_SOT_SMD:SOT-363_SC-70-6, F.Cu at (161.2, 137.9)
- added Q6: BC327, Package_TO_SOT_THT:TO-92_Inline, F.Cu at (140.8, 43.7)
- added R43: 10k, Resistor_SMD:R_0805_2012Metric_Pad1.15x1.40mm_HandSolder, F.Cu at (161.2, 47.7)
- added R44: 100k, Resistor_SMD:R_0805_2012Metric_Pad1.15x1.40mm_HandSolder, F.Cu at (155.8, 53.7)
- added R45: 100k, Resistor_SMD:R_0805_2012Metric_Pad1.15x1.40mm_HandSolder, F.Cu at (141.5, 56.6)
- added R46: 100k, Resistor_SMD:R_0805_2012Metric_Pad1.15x1.40mm_HandSolder, F.Cu at (174.8, 35.5)
- added R47: 100k, Resistor_SMD:R_0805_2012Metric_Pad1.15x1.40mm_HandSolder, F.Cu at (150.2, 59.6)
- added R48: 10k, Resistor_SMD:R_0805_2012Metric_Pad1.15x1.40mm_HandSolder, F.Cu at (155.8, 56.7)
- added R49: 10k, Resistor_SMD:R_0805_2012Metric_Pad1.15x1.40mm_HandSolder, F.Cu at (161.2, 50.7)
- added R50: 10k, Resistor_SMD:R_0805_2012Metric_Pad1.15x1.40mm_HandSolder, F.Cu at (171.5, 38.5)
- added R51: 10k, Resistor_SMD:R_0805_2012Metric_Pad1.15x1.40mm_HandSolder, F.Cu at (140.7, 59.5)
- added R52: 1k, Potentiometer_THT:Potentiometer_Runtron_RM-065_Vertical, F.Cu at (146.7, 157.4)
- C1, C2, R14: moved to B.Cu
- C3: value 1n -> 2.2n; moved to B.Cu
- C4: value 100n -> 1n
- C8: value 1n -> 100n
- D1, J2, J5, JP2, JP3, Q2, Q3, Q4, Q5, U1, U2, U3: moved to F.Cu
- J1: footprint Connector_PinHeader_2.54mm:PinHeader_1x03_P2.54mm_Vertical -> Connector_PinHeader_2.54mm:PinHeader_2x03_P2.54mm_Vertical; moved to F.Cu
- J3: footprint Connector_PinHeader_2.54mm:PinHeader_2x06_P2.54mm_Vertical -> Connector_PinHeader_2.54mm:PinHeader_2x07_P2.54mm_Vertical; moved to F.Cu
- J4: value ringmod in -> Conn_01x03_Male; footprint Connector_PinHeader_2.54mm:PinHeader_1x04_P2.54mm_Vertical -> Connector_PinHeader_2.54mm:PinHeader_1x03_P2.54mm_Vertical; moved to F.Cu
- JP5: value ringmod config -> Jumper_2_Open; footprint footprints:SolderDipJumper4alt -> footprints:SolderDipJumper2alt
- R1: value 10k -> 1Meg; footprint Potentiometer_THT:Potentiometer_Bourns_3296W_Vertical -> Resistor_SMD:R_0805_2012Metric_Pad1.15x1.40mm_HandSolder
- R10: footprint Resistor_SMD:R_0805_2012Metric_Pad1.15x1.40mm_HandSolder -> Resistor_THT:R_Axial_DIN0204_L3.6mm_D1.6mm_P2.54mm_Vertical
- R11: footprint Potentiometer_THT:Potentiometer_Bourns_3296W_Vertical -> Resistor_SMD:R_0805_2012Metric_Pad1.15x1.40mm_HandSolder; moved to F.Cu
- R12: value 4.7k -> 2.2k
- R13: value 100k -> 4.7k; moved to B.Cu
- R15, R25: footprint Resistor_SMD:R_0805_2012Metric_Pad1.15x1.40mm_HandSolder -> Potentiometer_THT:Potentiometer_Bourns_3296W_Vertical
- R16: value TODO -> 100k; moved to B.Cu
- R17: value TODO -> 1k
- R19: value 50k -> TODO; footprint Potentiometer_THT:Potentiometer_Runtron_RM-065_Vertical -> Resistor_SMD:R_0805_2012Metric_Pad1.15x1.40mm_HandSolder
- R2: value 147k -> 10k; footprint Resistor_SMD:R_0805_2012Metric_Pad1.15x1.40mm_HandSolder -> Potentiometer_THT:Potentiometer_Bourns_3296W_Vertical
- R20: value 100k -> TODO
- R21: value 47k -> 50k; footprint Resistor_SMD:R_0805_2012Metric_Pad1.15x1.40mm_HandSolder -> Potentiometer_THT:Potentiometer_Runtron_RM-065_Vertical
- R22: value 47k -> 100k
- R23: value 10k -> 47k; footprint Potentiometer_THT:Potentiometer_Bourns_3296W_Vertical -> Resistor_SMD:R_0805_2012Metric_Pad1.15x1.40mm_HandSolder; moved to F.Cu
- R26: value 20k -> 47k; footprint Potentiometer_THT:Potentiometer_Runtron_RM-065_Vertical -> Resistor_SMD:R_0805_2012Metric_Pad1.15x1.40mm_HandSolder; moved to F.Cu
- R28: value 10k -> 20k; footprint Resistor_SMD:R_0805_2012Metric_Pad1.15x1.40mm_HandSolder -> Potentiometer_THT:Potentiometer_Runtron_RM-065_Vertical
- R29: value 1Meg -> 10k; footprint Potentiometer_THT:Potentiometer_Runtron_RM-065_Vertical -> Resistor_SMD:R_0805_2012Metric_Pad1.15x1.40mm_HandSolder; moved to F.Cu
- R3: value 147k -> 1Meg; moved to B.Cu
- R30, R34: value 100k -> none
- R31: value 10k -> 1Meg; footprint Resistor_SMD:R_0805_2012Metric_Pad1.15x1.40mm_HandSolder -> Potentiometer_THT:Potentiometer_Runtron_RM-065_Vertical
- R32, R41: value 100k -> 10k
- R35: value 1k -> 10k
- R36: value 2.2k -> 100k
- R39: value 100k -> 1k
- R40: value 100k -> 2.2k
- R42: value TODO -> 10k; footprint Potentiometer_THT:Potentiometer_Runtron_RM-065_Vertical -> Resistor_SMD:R_0805_2012Metric_Pad1.15x1.40mm_HandSolder
- R5: value 220k -> 147k
- R6: value 12k2 -> 147k
- R7: value 1k -> 220k; footprint Resistor_THT:R_Axial_DIN0204_L3.6mm_D1.6mm_P2.54mm_Vertical -> Resistor_SMD:R_0805_2012Metric_Pad1.15x1.40mm_HandSolder; moved to F.Cu
- R8: value 150 -> 12k2; moved to B.Cu
- R9: value 2.2k -> 150
- moved J3 133.6 mm to (104.5, 18.8), turned to 0 degrees
- moved R28 120.3 mm to (155.2, 18.5)
- moved U2 113.6 mm to (121.8, 18.5), turned to 0 degrees
- moved R26 113.5 mm to (175.4, 26.7), turned to 0 degrees
- moved C5 113.0 mm to (170.7, 23.7), turned to 0 degrees
- moved R25 112.4 mm to (117.5, 39.1), turned to 0 degrees
- moved R19 109.0 mm to (170.1, 29.6), turned to 0 degrees
- moved JP3 108.1 mm to (165.4, 18.8), turned to 0 degrees
- moved Q4 107.8 mm to (171.0, 19.7), turned to 0 degrees
- moved R29 107.3 mm to (170.1, 32.6), turned to 0 degrees
- moved JP4 102.5 mm to (114.2, 51.1), turned to 0 degrees
- moved Q5 98.9 mm to (163.8, 24.3), turned to 0 degrees
- moved R36 98.9 mm to (170.1, 35.5)
- moved R22 96.9 mm to (175.4, 23.7), turned to 0 degrees
- moved R27 92.9 mm to (146.3, 56.7), turned to 0 degrees
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Connections:
- C10 pad 1: GND -> triangle
- C10 pad 2: VCC -> Net-(C10-Pad2)
- C11 pad 1: VEE -> square_ctl
- C11 pad 2: VCC -> Net-(C11-Pad2)
- C4 pad 1: pulse -> triangle
- C5 pad 1: sawtooth -> Net-(C5-Pad1)
- C5 pad 2: Net-(C5-Pad2) -> triangle
- C6 pad 1: triangle -> GND
- C6 pad 2: Net-(C6-Pad2) -> VEE
- C7 pad 1: square_ctl -> GND
- C7 pad 2: Net-(C7-Pad2) -> VCC
- C8 pad 1: triangle -> GNDD
- C8 pad 2: Net-(C8-Pad2) -> +5V
- C9 pad 1: GND -> rmpulse
- C9 pad 2: VEE -> Net-(C9-Pad2)
- J1 pad 2: GND -> +5V
- J1 pad 3: VEE -> GND
- J3 pad 10: Net-(C7-Pad2) -> Net-(C13-Pad2)
- J3 pad 11: GND -> square_ctl
- J3 pad 12: GND -> Net-(C11-Pad2)
- J3 pad 3: pulse -> rmpulse
- J3 pad 4: Net-(C4-Pad2) -> Net-(C9-Pad2)
- J3 pad 5: triangle -> pulse
- J3 pad 6: Net-(C6-Pad2) -> Net-(C12-Pad2)
- J3 pad 7: sawtooth -> triangle
- J3 pad 8: Net-(C5-Pad2) -> Net-(C10-Pad2)
- J3 pad 9: square_ctl -> sawtooth
- JP5 pad 1: Net-(JP5-Pad1) -> triangle
- JP5 pad 2: saw_ctl -> Net-(C5-Pad1)
- R11 pad 1: GND -> Net-(R10-Pad1)
- R11 pad 2: Net-(R11-Pad2) -> Net-(JP1-Pad1)
- R12 pad 1: B1 -> Net-(JP1-Pad1)
- R12 pad 2: Net-(JP1-Pad1) -> GND
- R13 pad 2: Net-(R11-Pad2) -> Net-(JP1-Pad1)
- R14 pad 1: VCC -> B1
- R14 pad 2: C1 -> Net-(R14-Pad2)
- R15 pad 1: E -> GND
- R15 pad 2: Net-(C3-Pad1) -> Net-(R14-Pad2)
- R16 pad 1: V_lin_pitchmod_1 -> VCC
- R16 pad 2: C2 -> C1
- R17 pad 1: V_lin_pitchmod_2 -> E
- R17 pad 2: C2 -> Net-(C3-Pad1)
- R18 pad 1: V_lin_pitchmod_3 -> V_lin_pitchmod_1
- R19 pad 1: V_expo -> V_lin_pitchmod_2
- R2 pad 1: V_control_raw -> Net-(R1-Pad2)
- R2 pad 2: V_control -> Net-(R2-Pad2)
- R20 pad 1: V_expo -> V_lin_pitchmod_3
- R20 pad 2: Net-(C8-Pad2) -> C2
- R21 pad 1: Net-(R21-Pad1) -> V_expo
- R21 pad 2: V_expo -> C2
- R22 pad 1: Net-(R22-Pad1) -> V_expo
- R22 pad 2: Net-(C8-Pad2) -> Net-(C4-Pad2)
- R23 pad 1: Net-(R22-Pad1) -> Net-(R23-Pad1)
- R23 pad 2: Net-(Q4-Pad3) -> V_expo
- R24 pad 1: GND -> Net-(R24-Pad1)
- R24 pad 2: Net-(R21-Pad1) -> Net-(C4-Pad2)
- R25 pad 1: ctl_override -> Net-(R24-Pad1)
- R25 pad 2: square_ctl -> Net-(Q4-Pad3)
- R26 pad 1: Net-(R26-Pad1) -> GND
- R26 pad 2: Net-(R26-Pad2) -> Net-(R23-Pad1)
- R27 pad 1: Net-(R26-Pad1) -> Net-(R27-Pad1)
- R28 pad 1: VEE -> Net-(R27-Pad1)
- R28 pad 2: Net-(R26-Pad3) -> Net-(R28-Pad2)
- R29 pad 1: Net-(R29-Pad1) -> VEE
- R29 pad 2: Net-(R26-Pad2) -> Net-(R28-Pad3)
- R3 pad 1: V_control_raw -> Net-(R2-Pad3)
- R3 pad 2: V_control_2 -> VEE
- R30 pad 1: Net-(R29-Pad1) -> GND
- R30 pad 2: square_ctl -> Net-(R28-Pad2)
- R31 pad 1: Net-(Q5-Pad2) -> Net-(J6-Pad1)
- R31 pad 2: saw_ctl -> Net-(R28-Pad2)
- R32 pad 1: triangle -> ctl_override
- R32 pad 2: Net-(R32-Pad2) -> square_ctl
- R33 pad 1: Net-(Q5-Pad1) -> Net-(J6-Pad1)
- R33 pad 2: triangle -> square_ctl
- R34 pad 1: Net-(R32-Pad2) -> Net-(C5-Pad1)
- R34 pad 2: sawtooth -> GND
- R35 pad 1: GND -> Net-(Q5-Pad2)
- R35 pad 2: pulse -> saw_ctl
- R36 pad 1: pulse -> Net-(C5-Pad1)
- R37 pad 1: Net-(J4-Pad1) -> Net-(Q5-Pad1)
- R37 pad 2: VEE -> Net-(C5-Pad1)
- R38 pad 1: Net-(J4-Pad2) -> Net-(R36-Pad2)
- R38 pad 2: VEE -> sawtooth
- R39 pad 1: Net-(J4-Pad3) -> GND
- R39 pad 2: VEE -> pulse
- R4 pad 2: V_control_3 -> V_control
- R40 pad 1: Net-(J4-Pad4) -> pulse
- R40 pad 2: VEE -> Net-(R40-Pad2)
- R41 pad 1: Net-(JP5-Pad4) -> Net-(R41-Pad1)
- R41 pad 2: VEE -> Net-(J4-Pad1)
- R42 pad 1: VCC -> Net-(R42-Pad1)
- R42 pad 2: V_tune -> Net-(J4-Pad2)
- R5 pad 2: V_tune -> V_control_2
- R6 pad 2: Net-(R6-Pad2) -> V_control_3
- R7 pad 1: Net-(R10-Pad1) -> V_control_raw
- R7 pad 2: Net-(JP1-Pad1) -> V_tune
- R8 pad 1: Net-(R6-Pad2) -> V_control_raw
- R8 pad 2: Net-(R10-Pad1) -> Net-(R8-Pad2)
- R9 pad 1: Net-(JP1-Pad1) -> Net-(R8-Pad2)
- R9 pad 2: GND -> Net-(R10-Pad1)
- U1 pad 1: Net-(R6-Pad2) -> V_expo
- U1 pad 12: Net-(R1-Pad2) -> Net-(R2-Pad2)
- U1 pad 2: V_control_raw -> C2
- U1 pad 8: V_expo -> Net-(R8-Pad2)
- U1 pad 9: C2 -> V_control_raw
- U2 pad 10: V_pwm -> Net-(C5-Pad1)
- U2 pad 13: Net-(R32-Pad2) -> Net-(R36-Pad2)
- U2 pad 2: Net-(C8-Pad2) -> Net-(C4-Pad2)
- U2 pad 3: Net-(R21-Pad1) -> Net-(R23-Pad1)
- U2 pad 5: Net-(R29-Pad1) -> Net-(J6-Pad1)
- U2 pad 8: Net-(R36-Pad2) -> Net-(R40-Pad2)
- U2 pad 9: triangle -> V_pwm
- U3 pad 1: Net-(J4-Pad1) -> Net-(R41-Pad1)
- U3 pad 10: Net-(JP5-Pad4) -> Net-(U3-Pad10)
- U3 pad 11: Net-(U3-Pad11) -> Net-(R50-Pad2)
- U3 pad 12: Net-(J4-Pad3) -> Net-(U3-Pad10)
- U3 pad 13: Net-(J4-Pad4) -> Net-(R47-Pad1)
- U3 pad 14: VCC -> +5V
- U3 pad 2: Net-(J4-Pad2) -> Net-(R42-Pad1)
- U3 pad 5: Net-(U3-Pad11) -> Net-(R43-Pad1)
- U3 pad 6: Net-(U3-Pad6) -> Net-(U3-Pad10)
- U3 pad 7: VEE -> GNDD
- U3 pad 8: Net-(JP5-Pad1) -> rmpulse
- U3 pad 9: Net-(U3-Pad6) -> Net-(R48-Pad1)
Routing:
- net VCC: track 185.1 -> 0.00 mm
- net VEE: track 178.3 -> 0.00 mm
- net GND: track 132.9 -> 10.9 mm
- net V_expo: track 79.7 -> 0.00 mm, vias 2 -> 0
- net var_vsource: track 78.0 -> 0.00 mm, vias 2 -> 0
- net C2: track 78.2 -> 6.53 mm, vias 4 -> 0
- net triangle: track 48.8 -> 0.00 mm
- net C1: track 45.4 -> 9.97 mm, vias 2 -> 0
- net Net-(R11-Pad2): track 29.6 -> 0.00 mm
- net ctl_override: track 23.7 -> 0.00 mm
- net Net-(J4-Pad3): track 20.9 -> 0.00 mm
- net Net-(JP5-Pad4): track 19.9 -> 0.00 mm
- net Net-(R29-Pad1): track 19.6 -> 0.00 mm
- net Net-(J4-Pad1): track 18.4 -> 0.00 mm
- net V_control_raw: track 18.1 -> 0.00 mm
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Other:
- board size 481.8 x 143.2 mm -> 481.8 x 171.7 mm
- net class Default: trace_width 0.25 -> 0.2; via_dia 2.5 -> 1; via_drill 0.9 -> 0.6
- rule trace_min: 0.25 -> 0.2
- rule via_min_drill: 0.9 -> 0.6
- rule via_min_size: 2.5 -> 1

Commit message: placement3/3
Parts:
- removed C10, C11, C12, C13, C9: 100n, Capacitor_SMD:C_0805_2012Metric_Pad1.15x1.40mm_HandSolder
- removed J1: power supply, Connector_PinHeader_2.54mm:PinHeader_2x03_P2.54mm_Vertical
- removed J2: control in, Connector_PinHeader_2.54mm:PinHeader_2x07_P2.54mm_Vertical
- removed J3: signal out, Connector_PinHeader_2.54mm:PinHeader_2x07_P2.54mm_Vertical
- removed R18, R19, R20: TODO, Resistor_SMD:R_0805_2012Metric_Pad1.15x1.40mm_HandSolder
- C4, C5, C6, C7, C8, R27, R29, R30, R32, R33, R34, R38, R47, R49: moved to B.Cu
- moved R28 142.1 mm to (182.5, 157.9), turned to 270 degrees
- moved U2 137.0 mm to (185.4, 139.9)
- moved R29 130.8 mm to (179.6, 163.0)
- moved J6 128.4 mm to (186.1, 158.8)
- moved Q5 127.0 mm to (196.3, 147.1), turned to 270 degrees
- moved R31 126.6 mm to (182.5, 150.6), turned to 270 degrees
- moved R39 126.3 mm to (189.9, 158.0)
- moved C5 122.7 mm to (202.3, 142.2), turned to 180 degrees
- moved R25 121.6 mm to (177.3, 144.9), turned to 270 degrees
- moved R26 120.2 mm to (182.2, 146.7)
- moved U3 119.4 mm to (202.2, 115.6), turned to 270 degrees
- moved R22 119.1 mm to (182.3, 142.6)
- moved Q4 116.5 mm to (184.9, 135.4), turned to 180 degrees
- moved JP6 115.3 mm to (205.7, 120.1), turned to 90 degrees
- moved JP3 115.2 mm to (169.9, 133.9), turned to 180 degrees
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Other:
- board size 481.8 x 171.7 mm -> 498.8 x 171.7 mm

Commit message: routing
Parts:
- added C10: 100n, Capacitor_SMD:C_0805_2012Metric_Pad1.15x1.40mm_HandSolder, F.Cu at (176.1, 131.4)
- added C11: 100n, Capacitor_SMD:C_0805_2012Metric_Pad1.15x1.40mm_HandSolder, F.Cu at (171.1, 131.4)
- added C12: 100n, Capacitor_SMD:C_0805_2012Metric_Pad1.15x1.40mm_HandSolder, B.Cu at (178.7, 131.4)
- added C13: 100n, Capacitor_SMD:C_0805_2012Metric_Pad1.15x1.40mm_HandSolder, F.Cu at (173.6, 131.4)
- added C9: 100n, Capacitor_SMD:C_0805_2012Metric_Pad1.15x1.40mm_HandSolder, F.Cu at (181.2, 131.4)
- added J1: power supply, Connector_PinHeader_2.54mm:PinHeader_2x03_P2.54mm_Vertical, F.Cu at (154.7, 126.6)
- added J2: control in, Connector_PinHeader_2.54mm:PinHeader_2x07_P2.54mm_Vertical, F.Cu at (142.3, 125.7)
- added J3: signal out, Connector_PinHeader_2.54mm:PinHeader_2x07_P2.54mm_Vertical, F.Cu at (183.8, 125.1)
- added R18: TODO, Resistor_SMD:R_0805_2012Metric_Pad1.15x1.40mm_HandSolder, F.Cu at (148.6, 128.4)
- added R19: TODO, Resistor_SMD:R_0805_2012Metric_Pad1.15x1.40mm_HandSolder, F.Cu at (148.6, 130.8)
- added R20: TODO, Resistor_SMD:R_0805_2012Metric_Pad1.15x1.40mm_HandSolder, F.Cu at (148.6, 133.3)
- R22, R23, R24, R26, R35, R39, R40, R44, R45, R46, R48, R50, R51: moved to B.Cu
- moved R40 29.0 mm to (182.5, 131.5), turned to 270 degrees
- moved R39 27.0 mm to (184.7, 131.5), turned to 90 degrees
- moved R5 21.7 mm to (140.6, 145.2), turned to 90 degrees
- moved R4 21.2 mm to (141.5, 148.3), turned to 180 degrees
- moved R43 20.2 mm to (194.4, 126.4)
- moved R46 18.8 mm to (194.4, 126.4), turned to 0 degrees
- moved R6 18.5 mm to (142.6, 145.2), turned to 90 degrees
- moved R42 16.4 mm to (199.8, 126.4), turned to 180 degrees
- moved R45 15.9 mm to (199.8, 126.4)
- moved R44 14.5 mm to (204.5, 126.4), turned to 0 degrees
- moved R51 14.0 mm to (198.2, 141.9), turned to 0 degrees
- moved R41 13.9 mm to (204.5, 126.4)
- moved R49 13.0 mm to (202.2, 134.0)
- moved U3 13.0 mm to (203.5, 128.5)
- moved JP6 13.0 mm to (207.0, 133.1)
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Routing:
- net GND: track 10.9 -> 439.2 mm, vias 1 -> 5
- net VCC: track 0.00 -> 121.6 mm, vias 0 -> 2
- net VEE: track 0.00 -> 106.3 mm, vias 0 -> 4
- net ctl_override: track 0.00 -> 82.2 mm, vias 0 -> 1
- net V_pwm: track 0.00 -> 79.7 mm
- net triangle: track 0.00 -> 72.5 mm, vias 0 -> 1
- net +5V: track 0.00 -> 70.4 mm
- net Net-(R40-Pad2): track 0.00 -> 62.8 mm, vias 0 -> 1
- net square_ctl: track 0.00 -> 57.4 mm
- net GNDD: track 0.00 -> 42.3 mm
- net V_control_raw: track 0.00 -> 41.3 mm
- net C2: track 6.53 -> 45.4 mm
- net sawtooth: track 0.00 -> 35.6 mm
- net var_vsource: track 0.00 -> 30.9 mm
- net Net-(C5-Pad1): track 0.00 -> 25.1 mm
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Other:
- board size 498.8 x 171.7 mm -> 80 x 50 mm

Commit message: slight adjustments
Parts:
- moved JP1 1.27 mm to (148.6, 142.0)
- moved R43 0.91 mm to (193.5, 126.4)
- moved R42 0.88 mm to (200.7, 126.4)
- moved R44 0.25 mm to (204.5, 126.6)
- moved R45 0.25 mm to (199.8, 126.6)
- moved R46 0.25 mm to (194.4, 126.6)
Routing:
- net GND: track 439.2 -> 552.8 mm, vias 5 -> 11
- net B1: track 27.2 -> 28.5 mm
- net Net-(JP1-Pad1): track 9.25 -> 10.5 mm
- added copper zone on B.Cu, net GND
- added copper zone on F.Cu, net GND

Commit message: add windfisch logo
Parts:
- added G***: LOGO, windfisch:windfisch_smaller, F.Cu at (202.3, 157.2)
Other:
- board text added: "(c) 2019 Florian Jung"
- board text added: "VCO development board mk I"
- board text added: "github.com/Windfisch/analog-synth"

Commit message: shrink gndplane, add texts
Parts:
- Q2, Q3: footprint Package_TO_SOT_THT:TO-92_Inline -> footprints:TO-92_Inline_alt
- moved R18 2.29 mm to (150.9, 128.4)
- moved R19 2.29 mm to (150.9, 130.8)
- moved R20 2.29 mm to (150.9, 133.3)
Routing:
- net GND: track 552.8 -> 539.1 mm
- net V_lin_pitchmod_3: track 2.35 -> 4.64 mm
- net V_lin_pitchmod_2: track 2.35 -> 4.64 mm
- net V_lin_pitchmod_1: track 2.41 -> 4.69 mm
Other:
- board text added: "+5V GNDD"
- board text added: "V_control"
- board text added: "Vcc GND Vee"
- board text added: "ctl"
- board text added: "expo"
- board text added: "lin.pitchmod"
- board text added: "mod"
- board text added: "pwm"
- board text added: "raw"
- board text added: "ring mod"
- board text added: "rossum"
- board text added: "schmitt fdbk"
- board text added: "shape trim"
- board text added: "sync"
- board text added: "tune"
