File: hardware/vco_mk1/vco_mk1_windfisch/vco_mk1.sch (KiCad schematic (older format))
At the start: 87 parts, among them J1 power supply, J2 control in, J3 signal out, J4 Conn_01x03_Male, J5 BCM847 breakout socket, J6 Conn_01x01_Male, Q1 BCM847, Q2 BC547, Q3 BC547, Q4 2N7000, Q5 BC547, Q6 BC327, U1 LM324, U2 LM324, U3 74HC86

Commit message: vco_mk1 rev02
Parts:
- renumbered C7 to C6, C6 to C7
Connections:
- net VCC: now also C7.2, U2.4 (V+); no longer C6.2, U2.11 (V-)
- net VEE: now also C6.2, U2.11 (V-); no longer C7.2, U2.4 (V+)
- net V_pwm: now also U2.2 (-); no longer U2.9 (-)
- net sawtooth: now also U2.7; no longer U2.14
- net square_ctl: now also U2.14; no longer U2.7
- net triangle: now also U2.13 (-), U2.8; no longer U2.1, U2.6 (-)
- net at C4.2, R22.2, R24.2: now also U2.9 (-); no longer U2.2 (-)
- net at R23.1, R26.2: now also U2.10 (+); no longer U2.3 (+)
- net at J6.1 (Pin_1), R31.1, R33.1: now also U2.12 (+); no longer U2.5 (+)
- net at C5.1, JP5.2 (B), R34.1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: now also U2.3 (+); no longer U2.10 (+)
- net at R36.2, R38.1: now also U2.6 (-); no longer U2.13 (-)
- net at Q5.1 (C), R37.1: now also U2.5 (+); no longer U2.12 (+)
- net at R40.2, R48.2: now also U2.1; no longer U2.8
Other:
- moved on the sheet: U2A, U2B, U2C, U2D
Changed lines of the file:
@@
 EESchema Schematic File Version 4
 LIBS:vco_mk1-cache
-EELAYER 29 0
+EELAYER 30 0
 EELAYER END
 $Descr A4 11693 8268
@@
 Wire Wire Line
 	2875 6800 2825 6800
-$Comp
-L power:VCC #PWR021
-U 1 1 5CF357C9
-P 3075 7050
-F 0 "#PWR021" H 3075 6900 50  0001 C CNN
-F 1 "VCC" H 3175 7075 50  0000 C CNN
-F 2 "" H 3075 7050 50  0001 C CNN
-F 3 "" H 3075 7050 50  0001 C CNN
-	1    3075 7050
-	-1   0    0    1
-$EndComp
 Wire Wire Line
 	2625 6300 2875 6300
@@
 $Comp
 L Amplifier_Operational:LM324 U2
-U 1 1 5D628926
-P 2225 6300
-F 0 "U2" H 2325 6150 50  0000 C CNN
-F 1 "LM324" H 2200 6300 50  0000 C CNN
-F 2 "Package_DIP:DIP-14_W7.62mm" H 2175 6400 50  0001 C CNN
-F 3 "http://www.ti.com/lit/ds/symlink/lm2902-n.pdf" H 2275 6500 50  0001 C CNN
-	1    2225 6300
-	1    0    0    1
-$EndComp
-$Comp
-L Amplifier_Operational:LM324 U2
 U 2 1 5D628930
-P 3175 6700
-F 0 "U2" H 3275 6550 50  0000 C CNN
-F 1 "LM324" H 3150 6700 50  0000 C CNN
-F 2 "Package_DIP:DIP-14_W7.62mm" H 3125 6800 50  0001 C CNN
-F 3 "http://www.ti.com/lit/ds/symlink/lm2902-n.pdf" H 3225 6900 50  0001 C CNN
-	2    3175 6700
-	1    0    0    1
-$EndComp
-$Comp
-L Amplifier_Operational:LM324 U2
-U 4 1 5D628944
 P 4975 5800
-F 0 "U2" H 5050 5625 50  0000 C CNN
+F 0 "U2" H 5075 5650 50  0000 C CNN
 F 1 "LM324" H 4950 5800 50  0000 C CNN
 F 2 "Package_DIP:DIP-14_W7.62mm" H 4925 5900 50  0001 C CNN
 F 3 "http://www.ti.com/lit/ds/symlink/lm2902-n.pdf" H 5025 6000 50  0001 C CNN
-	4    4975 5800
+	2    4975 5800
 	1    0    0    1
 $EndComp
@@
 $EndComp
 Connection ~ 3475 6700
-$Comp
-L power:VEE #PWR020
-U 1 1 5CF354CF
-P 3075 6350
-F 0 "#PWR020" H 3075 6200 50  0001 C CNN
-F 1 "VEE" H 2975 6475 50  0000 C CNN
-F 2 "" H 3075 6350 50  0001 C CNN
-F 3 "" H 3075 6350 50  0001 C CNN
-	1    3075 6350
-	1    0    0    -1
-$EndComp
 Wire Wire Line
 	5275 5800 5375 5800
@@
 	3075 7050 3075 7025
 $Comp
-L Device:C_Small C7
+L Device:C_Small C6
 U 1 1 5D5CE3BE
 P 3225 7025
-F 0 "C7" V 3175 7125 50  0000 C CNN
+F 0 "C6" V 3175 7125 50  0000 C CNN
 F 1 "100n" V 3100 7025 50  0000 C CNN
 F 2 "Capacitor_SMD:C_0805_2012Metric_Pad1.15x1.40mm_HandSolder" H 3225 7025 50  0001 C CNN
@@
 	3075 7025 3075 7000
 $Comp
-L Device:C_Small C6
+L Device:C_Small C7
 U 1 1 5D5E8697
 P 3225 6375
-F 0 "C6" V 3175 6450 50  0000 C CNN
+F 0 "C7" V 3175 6450 50  0000 C CNN
 F 1 "100n" V 3100 6375 50  0000 C CNN
 F 2 "Capacitor_SMD:C_0805_2012Metric_Pad1.15x1.40mm_HandSolder" H 3225 6375 50  0001 C CNN
@@
 L Amplifier_Operational:LM324 U2
 U 3 1 5D62893A
-P 4975 4975
-F 0 "U2" H 5075 4825 50  0000 C CNN
-F 1 "LM324" H 4950 4975 50  0000 C CNN
-F 2 "Package_DIP:DIP-14_W7.62mm" H 4925 5075 50  0001 C CNN
-F 3 "http://www.ti.com/lit/ds/symlink/lm2902-n.pdf" H 5025 5175 50  0001 C CNN
-	3    4975 4975
+P 2225 6300
+F 0 "U2" H 2325 6150 50  0000 C CNN
+F 1 "LM324" H 2200 6300 50  0000 C CNN
+F 2 "Package_DIP:DIP-14_W7.62mm" H 2175 6400 50  0001 C CNN
+F 3 "http://www.ti.com/lit/ds/symlink/lm2902-n.pdf" H 2275 6500 50  0001 C CNN
+	3    2225 6300
 	1    0    0    1
 $EndComp
@@
 Wire Wire Line
 	5675 4975 6350 4975
+$Comp
+L power:VEE #PWR020
+U 1 1 5CF354CF
+P 3075 7050
+F 0 "#PWR020" H 3075 6900 50  0001 C CNN
+F 1 "VEE" H 3175 7075 50  0000 C CNN
+F 2 "" H 3075 7050 50  0001 C CNN
+F 3 "" H 3075 7050 50  0001 C CNN
+	1    3075 7050
+	-1   0    0    1
+$EndComp
+$Comp
+L power:VCC #PWR021
+U 1 1 5CF357C9
+P 3075 6350
+F 0 "#PWR021" H 3075 6200 50  0001 C CNN
+F 1 "VCC" H 2975 6475 50  0000 C CNN
+F 2 "" H 3075 6350 50  0001 C CNN
+F 3 "" H 3075 6350 50  0001 C CNN
+	1    3075 6350
+	1    0    0    -1
+$EndComp
+$Comp
+L Amplifier_Operational:LM324 U2
+U 1 1 5D628926
+P 4975 4975
+F 0 "U2" H 5075 4825 50  0000 C CNN
+F 1 "LM324" H 4950 4975 50  0000 C CNN
+F 2 "Package_DIP:DIP-14_W7.62mm" H 4925 5075 50  0001 C CNN
+F 3 "http://www.ti.com/lit/ds/symlink/lm2902-n.pdf" H 5025 5175 50  0001 C CNN
+	1    4975 4975
+	1    0    0    1
+$EndComp
+$Comp
+L Amplifier_Operational:LM324 U2
+U 4 1 5D628944
+P 3175 6700
+F 0 "U2" H 3250 6525 50  0000 C CNN
+F 1 "LM324" H 3150 6700 50  0000 C CNN
+F 2 "Package_DIP:DIP-14_W7.62mm" H 3125 6800 50  0001 C CNN
+F 3 "http://www.ti.com/lit/ds/symlink/lm2902-n.pdf" H 3225 6900 50  0001 C CNN
+	4    3175 6700
+	1    0    0    1
+$EndComp
 $EndSCHEMATC
