File: hardware/vco_mk1/vco_mk1_windfisch/vco_mk1.kicad_pcb (KiCad board)
At the start: 2 copper layers, 71.6 x 44.7 mm, 88 parts, among them J1 power supply, J2 control in, J3 signal out, J4 Conn_01x03_Male, J5 BCM847 breakout socket, J6 Conn_01x01_Male, Q1 BCM847, Q2 BC547, Q3 BC547, Q4 2N7000, Q5 BC547, Q6 BC327, U1 LM324, U2 LM324, U3 74HC86

Commit message: vco_mk1 rev02
Parts:
- moved U2 17.0 mm to (193.1, 157.9), turned to 180 degrees
Connections:
- U2 pad 1: triangle -> Net-(R40-Pad2)
- U2 pad 10: Net-(C5-Pad1) -> Net-(R23-Pad1)
- U2 pad 11: VCC -> VEE
- U2 pad 12: Net-(Q5-Pad1) -> Net-(J6-Pad1)
- U2 pad 13: Net-(R36-Pad2) -> triangle
- U2 pad 14: sawtooth -> square_ctl
- U2 pad 2: Net-(C4-Pad2) -> V_pwm
- U2 pad 3: Net-(R23-Pad1) -> Net-(C5-Pad1)
- U2 pad 4: VEE -> VCC
- U2 pad 5: Net-(J6-Pad1) -> Net-(Q5-Pad1)
- U2 pad 6: triangle -> Net-(R36-Pad2)
- U2 pad 7: square_ctl -> sawtooth
- U2 pad 8: Net-(R40-Pad2) -> triangle
- U2 pad 9: V_pwm -> Net-(C4-Pad2)
Other:
- board text added: "(rev02)"
Changed lines of the file:
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@@
-(kicad_pcb (version 20171130) (host pcbnew 5.1.2)
+(kicad_pcb (version 20171130) (host pcbnew 5.1.4)
   (general
     (thickness 1.6)
-    (drawings 80)
+    (drawings 81)
     (tracks 700)
     (zones 0)
@@
   )
   (module Package_DIP:DIP-14_W7.62mm (layer F.Cu)
-    (at 185.4962 142.6464)
+    (at 193.1162 157.8864 180)
     (descr "14-lead though-hole mounted DIP package, row spacing 7.62 mm (300 mils)")
     (tags "THT DIP DIL PDIP 2.54mm 7.62mm 300mil")
-    (fp_text reference U2 (at 7.5438 17.7546) (layer F.SilkS)
+    (fp_text reference U2 (at 0.0762 -2.6416) (layer F.SilkS)
       (effects (font (size 1 1) (thickness 0.2)))
     )
@@
       (effects (font (size 1 1) (thickness 0.2)))
     )
+    (fp_arc (start 3.81 -1.33) (end 2.81 -1.33) (angle -180) (layer F.SilkS) (width 0.12))
+    (fp_line (start 1.635 -1.27) (end 6.985 -1.27) (layer F.Fab) (width 0.1))
+    (fp_line (start 6.985 -1.27) (end 6.985 16.51) (layer F.Fab) (width 0.1))
+    (fp_line (start 6.985 16.51) (end 0.635 16.51) (layer F.Fab) (width 0.1))
+    (fp_line (start 0.635 16.51) (end 0.635 -0.27) (layer F.Fab) (width 0.1))
+    (fp_line (start 0.635 -0.27) (end 1.635 -1.27) (layer F.Fab) (width 0.1))
+    (fp_line (start 2.81 -1.33) (end 1.16 -1.33) (layer F.SilkS) (width 0.12))
+    (fp_line (start 1.16 -1.33) (end 1.16 16.57) (layer F.SilkS) (width 0.12))
+    (fp_line (start 1.16 16.57) (end 6.46 16.57) (layer F.SilkS) (width 0.12))
+    (fp_line (start 6.46 16.57) (end 6.46 -1.33) (layer F.SilkS) (width 0.12))
+    (fp_line (start 6.46 -1.33) (end 4.81 -1.33) (layer F.SilkS) (width 0.12))
+    (fp_line (start -1.1 -1.55) (end -1.1 16.8) (layer F.CrtYd) (width 0.05))
+    (fp_line (start -1.1 16.8) (end 8.7 16.8) (layer F.CrtYd) (width 0.05))
+    (fp_line (start 8.7 16.8) (end 8.7 -1.55) (layer F.CrtYd) (width 0.05))
+    (fp_line (start 8.7 -1.55) (end -1.1 -1.55) (layer F.CrtYd) (width 0.05))
     (fp_text user %R (at 3.81 7.62) (layer F.Fab)
       (effects (font (size 1 1) (thickness 0.2)))
     )
-    (fp_line (start 8.7 -1.55) (end -1.1 -1.55) (layer F.CrtYd) (width 0.05))
-    (fp_line (start 8.7 16.8) (end 8.7 -1.55) (layer F.CrtYd) (width 0.05))
-    (fp_line (start -1.1 16.8) (end 8.7 16.8) (layer F.CrtYd) (width 0.05))
-    (fp_line (start -1.1 -1.55) (end -1.1 16.8) (layer F.CrtYd) (width 0.05))
-    (fp_line (start 6.46 -1.33) (end 4.81 -1.33) (layer F.SilkS) (width 0.12))
-    (fp_line (start 6.46 16.57) (end 6.46 -1.33) (layer F.SilkS) (width 0.12))
-    (fp_line (start 1.16 16.57) (end 6.46 16.57) (layer F.SilkS) (width 0.12))
-    (fp_line (start 1.16 -1.33) (end 1.16 16.57) (layer F.SilkS) (width 0.12))
-    (fp_line (start 2.81 -1.33) (end 1.16 -1.33) (layer F.SilkS) (width 0.12))
-    (fp_line (start 0.635 -0.27) (end 1.635 -1.27) (layer F.Fab) (width 0.1))
-    (fp_line (start 0.635 16.51) (end 0.635 -0.27) (layer F.Fab) (width 0.1))
-    (fp_line (start 6.985 16.51) (end 0.635 16.51) (layer F.Fab) (width 0.1))
-    (fp_line (start 6.985 -1.27) (end 6.985 16.51) (layer F.Fab) (width 0.1))
-    (fp_line (start 1.635 -1.27) (end 6.985 -1.27) (layer F.Fab) (width 0.1))
-    (fp_arc (start 3.81 -1.33) (end 2.81 -1.33) (angle -180) (layer F.SilkS) (width 0.12))
-    (pad 14 thru_hole oval (at 7.62 0) (size 1.6 1.6) (drill 0.8) (layers *.Cu *.Mask)
-      (net 7 sawtooth))
-    (pad 7 thru_hole oval (at 0 15.24) (size 1.6 1.6) (drill 0.8) (layers *.Cu *.Mask)
-      (net 9 square_ctl))
-    (pad 13 thru_hole oval (at 7.62 2.54) (size 1.6 1.6) (drill 0.8) (layers *.Cu *.Mask)
-      (net 37 "Net-(R36-Pad2)"))
-    (pad 6 thru_hole oval (at 0 12.7) (size 1.6 1.6) (drill 0.8) (layers *.Cu *.Mask)
+    (pad 1 thru_hole rect (at 0 0 180) (size 1.6 1.6) (drill 0.8) (layers *.Cu *.Mask)
+      (net 63 "Net-(R40-Pad2)"))
+    (pad 8 thru_hole oval (at 7.62 15.24 180) (size 1.6 1.6) (drill 0.8) (layers *.Cu *.Mask)
       (net 8 triangle))
-    (pad 12 thru_hole oval (at 7.62 5.08) (size 1.6 1.6) (drill 0.8) (layers *.Cu *.Mask)
-      (net 29 "Net-(Q5-Pad1)"))
-    (pad 5 thru_hole oval (at 0 10.16) (size 1.6 1.6) (drill 0.8) (layers *.Cu *.Mask)
-      (net 50 "Net-(J6-Pad1)"))
-    (pad 11 thru_hole oval (at 7.62 7.62) (size 1.6 1.6) (drill 0.8) (layers *.Cu *.Mask)
-      (net 1 VCC))
-    (pad 4 thru_hole oval (at 0 7.62) (size 1.6 1.6) (drill 0.8) (layers *.Cu *.Mask)
-      (net 2 VEE))
-    (pad 10 thru_hole oval (at 7.62 10.16) (size 1.6 1.6) (drill 0.8) (layers *.Cu *.Mask)
-      (net 41 "Net-(C5-Pad1)"))
-    (pad 3 thru_hole oval (at 0 5.08) (size 1.6 1.6) (drill 0.8) (layers *.Cu *.Mask)
-      (net 58 "Net-(R23-Pad1)"))
-    (pad 9 thru_hole oval (at 7.62 12.7) (size 1.6 1.6) (drill 0.8) (layers *.Cu *.Mask)
+    (pad 2 thru_hole oval (at 0 2.54 180) (size 1.6 1.6) (drill 0.8) (layers *.Cu *.Mask)
       (net 16 V_pwm))
-    (pad 2 thru_hole oval (at 0 2.54) (size 1.6 1.6) (drill 0.8) (layers *.Cu *.Mask)
+    (pad 9 thru_hole oval (at 7.62 12.7 180) (size 1.6 1.6) (drill 0.8) (layers *.Cu *.Mask)
       (net 5 "Net-(C4-Pad2)"))
-    (pad 8 thru_hole oval (at 7.62 15.24) (size 1.6 1.6) (drill 0.8) (layers *.Cu *.Mask)
-      (net 63 "Net-(R40-Pad2)"))
-    (pad 1 thru_hole rect (at 0 0) (size 1.6 1.6) (drill 0.8) (layers *.Cu *.Mask)
+    (pad 3 thru_hole oval (at 0 5.08 180) (size 1.6 1.6) (drill 0.8) (layers *.Cu *.Mask)
+      (net 41 "Net-(C5-Pad1)"))
+    (pad 10 thru_hole oval (at 7.62 10.16 180) (size 1.6 1.6) (drill 0.8) (layers *.Cu *.Mask)
+      (net 58 "Net-(R23-Pad1)"))
+    (pad 4 thru_hole oval (at 0 7.62 180) (size 1.6 1.6) (drill 0.8) (layers *.Cu *.Mask)
+      (net 1 VCC))
+    (pad 11 thru_hole oval (at 7.62 7.62 180) (size 1.6 1.6) (drill 0.8) (layers *.Cu *.Mask)
+      (net 2 VEE))
+    (pad 5 thru_hole oval (at 0 10.16 180) (size 1.6 1.6) (drill 0.8) (layers *.Cu *.Mask)
+      (net 29 "Net-(Q5-Pad1)"))
+    (pad 12 thru_hole oval (at 7.62 5.08 180) (size 1.6 1.6) (drill 0.8) (layers *.Cu *.Mask)
+      (net 50 "Net-(J6-Pad1)"))
+    (pad 6 thru_hole oval (at 0 12.7 180) (size 1.6 1.6) (drill 0.8) (layers *.Cu *.Mask)
+      (net 37 "Net-(R36-Pad2)"))
+    (pad 13 thru_hole oval (at 7.62 2.54 180) (size 1.6 1.6) (drill 0.8) (layers *.Cu *.Mask)
       (net 8 triangle))
+    (pad 7 thru_hole oval (at 0 15.24 180) (size 1.6 1.6) (drill 0.8) (layers *.Cu *.Mask)
+      (net 7 sawtooth))
+    (pad 14 thru_hole oval (at 7.62 0 180) (size 1.6 1.6) (drill 0.8) (layers *.Cu *.Mask)
+      (net 9 square_ctl))
     (model ${KISYS3DMOD}/Package_DIP.3dshapes/DIP-14_W7.62mm.wrl
       (at (xyz 0 0 0))
@@
     )
   )
+  (gr_text "(rev02)" (at 170.688 164.211) (layer F.SilkS)
+    (effects (font (size 1 1) (thickness 0.2)))
+  )
   (gr_text JLCJLCJLCJLC (at 167.894 161.29) (layer B.SilkS)
     (effects (font (size 0.9 0.9) (thickness 0.16)) (justify mirror))
@@
     (effects (font (size 1 1) (thickness 0.2)))
   )
-  (gr_text "VCO development\nboard mk I" (at 163.83 162.814) (layer F.SilkS)
+  (gr_text "VCO development\nboard mk I      " (at 163.83 162.814) (layer F.SilkS)
     (effects (font (size 1.5 1.5) (thickness 0.2)))
   )
@@
   (segment (start 146.431 139.975) (end 145.696999 139.240999) (width 0.2) (layer B.Cu) (net 16))
   (segment (start 145.696999 139.240999) (end 144.847 138.391) (width 0.2) (layer B.Cu) (net 16))
+  (segment (start 145.6055 144.2085) (end 146.431 143.383) (width 0.2) (layer B.Cu) (net 16))
+  (segment (start 145.415 144.399) (end 145.6055 144.2085) (width 0.2) (layer B.Cu) (net 16))
   (segment (start 145.141989 144.672011) (end 145.6055 144.2085) (width 0.2) (layer B.Cu) (net 16))
   (segment (start 145.141989 159.900991) (end 145.141989 144.672011) (width 0.2) (layer B.Cu) (net 16))
+  (segment (start 194.945 157.1752) (end 194.945 158.197602) (width 0.2) (layer B.Cu) (net 16))
   (segment (start 149.258208 164.01721) (end 145.141989 159.900991) (width 0.2) (layer B.Cu) (net 16))
+  (segment (start 194.945 158.197602) (end 189.125392 164.01721) (width 0.2) (layer B.Cu) (net 16))
   (segment (start 193.1162 155.3464) (end 194.945 157.1752) (width 0.2) (layer B.Cu) (net 16))
-  (segment (start 145.6055 144.2085) (end 146.431 143.383) (width 0.2) (layer B.Cu) (net 16))
-  (segment (start 188.613392 164.01721) (end 149.258208 164.01721) (width 0.2) (layer B.Cu) (net 16))
-  (segment (start 145.415 144.399) (end 145.6055 144.2085) (width 0.2) (layer B.Cu) (net 16))
-  (segment (start 194.945 157.1752) (end 194.945 157.685602) (width 0.2) (layer B.Cu) (net 16))
-  (segment (start 194.945 157.685602) (end 188.613392 164.01721) (width 0.2) (layer B.Cu) (net 16))
+  (segment (start 189.125392 164.01721) (end 149.258208 164.01721) (width 0.2) (layer B.Cu) (net 16))
   (via (at 191.262 143.002) (size 1) (drill 0.6) (layers F.Cu B.Cu) (net 17))
   (segment (start 189.6872 142.8914) (end 191.1514 142.8914) (width 0.2) (layer B.Cu) (net 17))
