File: hardware/vco_mk1/vco_mk1_spitfire/vco_mk1.kicad_pcb (KiCad board)
At the start: 2 copper layers, 50 x 80 mm, 91 parts, among them J1 power supply, J2 control in, J3 signal out, J4 Conn_01x03_Male, J5 BCM847 breakout socket, J6 Conn_01x01_Male, Q1 BCM847, Q2 BC547, Q3 BC547, Q4 2N7000, Q5 BC547, Q6 BC327, U1 LM324, U2 LM324, U3 74HC86

Commit message: added README and updated file structure to new naming conventions
Parts:
- removed the G*** at (0.00, 0.00)

Commit message: vco_mk1 rev02
Parts:
- moved U2 17.0 mm to (191.9, 128.8), turned to 180 degrees
Connections:
- U2 pad 1: triangle -> Net-(R40-Pad2)
- U2 pad 10: Net-(C5-Pad1) -> Net-(R23-Pad1)
- U2 pad 11: VCC -> VEE
- U2 pad 12: Net-(Q5-Pad1) -> Net-(J6-Pad1)
- U2 pad 13: Net-(R36-Pad2) -> triangle
- U2 pad 14: sawtooth -> square_ctl
- U2 pad 2: Net-(C4-Pad2) -> V_pwm
- U2 pad 3: Net-(R23-Pad1) -> Net-(C5-Pad1)
- U2 pad 4: VEE -> VCC
- U2 pad 5: Net-(J6-Pad1) -> Net-(Q5-Pad1)
- U2 pad 6: triangle -> Net-(R36-Pad2)
- U2 pad 7: square_ctl -> sawtooth
- U2 pad 8: Net-(R40-Pad2) -> triangle
- U2 pad 9: V_pwm -> Net-(C4-Pad2)
Other:
- board text added: "(rev02)"
