File: measure_vco/schem/measure_vco.sch (KiCad schematic (older format))
At the start: 32 parts, among them Q1 2N7000, Q3 BC546, Q4 BC546, U1 LM324, U2 LM324, U3 LM324, U6 LM324, U7 LM324, U8 LM324

Commit message: test tones for adjusting R10
Parts:
- gave numbers to parts that had none: 4
Changed lines of the file:
@@
 EESchema Schematic File Version 4
+LIBS:measure_vco-cache
 EELAYER 29 0
 EELAYER END
@@
 unused
 $Comp
-L Device:R_POT RV?
+L Device:R_POT R10
 U 1 1 5D1F262E
 P 10350 4050
-F 0 "RV?" H 10280 4096 50  0000 R CNN
+F 0 "R10" H 10280 4096 50  0000 R CNN
 F 1 "1k" H 10280 4005 50  0000 R CNN
 F 2 "" H 10350 4050 50  0001 C CNN
@@
 $EndComp
 $Comp
-L power:VEE #PWR?
+L power:VEE #PWR027
 U 1 1 5D1F30D6
 P 10350 4200
-F 0 "#PWR?" H 10350 4050 50  0001 C CNN
+F 0 "#PWR027" H 10350 4050 50  0001 C CNN
 F 1 "VEE" H 10368 4373 50  0000 C CNN
 F 2 "" H 10350 4200 50  0001 C CNN
@@
 $EndComp
 $Comp
-L power:VCC #PWR?
+L power:VCC #PWR014
 U 1 1 5D1F38FD
 P 10350 3900
-F 0 "#PWR?" H 10350 3750 50  0001 C CNN
+F 0 "#PWR014" H 10350 3750 50  0001 C CNN
 F 1 "VCC" H 10367 4073 50  0000 C CNN
 F 2 "" H 10350 3900 50  0001 C CNN
@@
 middle\npositon\nis fine
 $Comp
-L Analog_DAC:MCP4822 U?
+L Analog_DAC:MCP4822 U4
 U 1 1 5D1F7952
 P 9200 3800
-F 0 "U?" H 8800 4250 50  0000 C CNN
+F 0 "U4" H 8800 4250 50  0000 C CNN
 F 1 "MCP4822" H 8900 4150 50  0000 C CNN
 F 2 "" H 10000 3500 50  0001 C CNN
@@
 	8100 4300 9200 4300
 $Comp
-L power:GNDREF #PWR?
+L power:GNDREF #PWR013
 U 1 1 5D1FFD8B
 P 9200 4400
-F 0 "#PWR?" H 9200 4150 50  0001 C CNN
+F 0 "#PWR013" H 9200 4150 50  0001 C CNN
 F 1 "GNDREF" H 9205 4227 50  0000 C CNN
 F 2 "" H 9200 4400 50  0001 C CNN
@@
 Connection ~ 9200 4300
 $Comp
-L power:VCC #PWR?
+L power:VCC #PWR012
 U 1 1 5D20405E
 P 9200 3400
-F 0 "#PWR?" H 9200 3250 50  0001 C CNN
+F 0 "#PWR012" H 9200 3250 50  0001 C CNN
 F 1 "VCC" H 9217 3573 50  0000 C CNN
 F 2 "" H 9200 3400 50  0001 C CNN
@@
 NoConn ~ 9700 4000
 $Comp
-L Diode:1N5817 D?
+L Diode:1N5817 D1
 U 1 1 5D20D972
 P 9150 5650
-F 0 "D?" V 9104 5729 50  0000 L CNN
+F 0 "D1" V 9104 5729 50  0000 L CNN
 F 1 "1N5817" V 9195 5729 50  0000 L CNN
 F 2 "Diode_THT:D_DO-41_SOD81_P10.16mm_Horizontal" H 9150 5475 50  0001 C CNN
@@
 $EndComp
 $Comp
-L Device:R R?
+L Device:R R8
 U 1 1 5D20E97C
 P 9150 5250
-F 0 "R?" H 9220 5296 50  0000 L CNN
+F 0 "R8" H 9220 5296 50  0000 L CNN
 F 1 "10k" V 9150 5200 50  0000 L CNN
 F 2 "" V 9080 5250 50  0001 C CNN
@@
 $EndComp
 $Comp
-L power:GNDREF #PWR?
+L power:GNDREF #PWR011
 U 1 1 5D20F2EC
 P 9150 5800
-F 0 "#PWR?" H 9150 5550 50  0001 C CNN
+F 0 "#PWR011" H 9150 5550 50  0001 C CNN
 F 1 "GNDREF" H 9155 5627 50  0000 C CNN
 F 2 "" H 9150 5800 50  0001 C CNN

Commit message: measure_vco schematic: reality update
Parts:
- removed R14, R15: 100k, symbol Device:R_Small
- added D1: 3V3, symbol Device:D_Zener
- added R8: 100k, symbol Device:R
- Q3, Q4: value BC546 -> 1/2 BCM847
- renumbered D1 to D2, R8 to R11
Connections:
- net GNDREF: now also D1.2 (A), R8.2
- net STM32_PE7: now also D1.1 (K)
- net at R9.1, U3.1 (+): now also R8.1
Other:
- note added: "Because R8 is connected to GNDREF, the triangle would be\ncentered around GNDREF, but only if the output of the\ncomparator U3 would swing between Vcc and Vee.\nHowever, U3 swings between less-than-Vcc and\nexactly Vee, so the triangle isn't centered."
- note added: "or use\n2x BC547"
- note added: "square_ctl swings between Vee and Vcc - 1.5V (circa).\nGNDREF is at (Vcc+Vee)/2, i.e. PE7 sees at least 3V for\nVcc-Vee = 9V.\nThe diodes protect the MCU pin from overvoltage (D1)\nand undervoltage (D2): The schottky diode D2 clamps\naway negative voltages (to approx. -200mV), while the\nzener diode D1 limits. That's within the MCU specs.\nthe voltage to 3.3V"
- note removed: "If R8 was connected to GNDREF, the triangle would be\ncentered around GNDREF, but only if the output of the\ncomparator U3 would swing between Vcc and Vee.\nHowever, U3 swings between less-than-Vcc and\nexactly Vee, so the triangle isn't centered.\nR14 and R15 comprise a poti to compensate for that."
- note removed: "or use\nBCM847"
- note removed: "square_ctl swings between Vee and Vcc - 1.5V (circa).\nGNDREF is at (Vcc+Vee)/2, i.e. PE7 sees 3V for\nVcc-Vee = 9V.\nThe diode clamps away negative voltages."
- moved on the sheet: D2, R10, R11, U4

Commit message: schematic: add thermal and rossum compensation
Parts:
- added D3: D, symbol Device:D
- added R12: 150, symbol Device:R
- added R13: 1k, symbol Device:Thermistor_NTC
- added R14, R27: 1k, symbol Device:R
- added R15: 2.2k, symbol Device:R
- added R22: 4.7k, symbol Device:R
- added R23: 100k, symbol Device:R
- added R24, R26: 1k, symbol Device:R_POT_TRIM
- added R25: 220, symbol Device:R
- added U5: LM317L_TO92, Package_TO_SOT_THT:TO-92_Inline, symbol Regulator_Linear:LM317L_TO92
- R19: value 534k -> 147k
- R20: value 10k -> 12k2
- R8: value 100k -> 50k
Connections:
- net GNDREF: now also R15.2, R24.1
- net VCC: now also R25.1, U5.2 (VO)
- net at R20.2, U8.3: now also R12.1; no longer Q3.2 (B)
- net at C2.1, R17.2, U6.3: now also D3.1 (K)
- net 0 renamed -VDC
- net -VDC: now also R27.2
- new net: Q3.2 (B), R22.1, R23.1
- new net: R12.2, R13.1, R14.1
- new net: R13.2, R14.2, R15.1, R22.2
- new net: R23.2, R24.2
- new net: D3.2 (A), R24.3
- new net: R25.2, R26.1, U5.1 (ADJ)
- new net: R26.2, R26.3, R27.1
- new net +VDC: U5.3 (VI)
Other:
- note added: "364 Ohm for 9V\n892 Ohm for 12V"
- note added: "Changing the R8/R9 ratio affects the maximum frequency\nand the triangle's amplitude. R8 = 16k has proved to work,\nproviding very high maximum frequencies.\nR8 = 5k and R9 = 10k works fine, too."
- note added: "R3 * C1 should be 100µs, this affects the frequency range\nR3 : R5 must be 2:1, this affects the triangle shape\nR4 : R6 must be 1:1, this affects the triangle shape\nR8 : R9 should be 1:2, this affects the triangle amplitude and\nfrequency range. If R9 is too large, this may cause distortion"
- note added: "Rossum\ncompensation"
- note added: "Symmetric power supply"
- note added: "To power supply.\nE.g. a 12V LiPo\nor a lab PSU"
- note added: "ca 18mV/oct"
- note added: "ca 19mV/Oct"
- note added: "ca 24mV/oct"
- note added: "ca 290mV/oct"
- note added: "for Q4, the following holds true:\nI_C = const * exp(V_B / VT) with VT=26mV\n(thermal voltage of a transistor)\nnow this means that Vout will double\nevery (log(2) * 26mV) = 18mV.\n\nNote that VT is temperature dependent.\nWhen the temperature rises, VT rises and so\nthe input voltage must rise too. The thermal\ncompensation consisting of TODO does that.\n\nAdditionally, Q3 and Q4 have a bulk res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"
- note added: "replace this GNDREF by a\nvoltage source ca. 1mV-\n1.5mV below GNDREF for\nbest results."
- note added: "thermal\ncompensation"
- note removed: "10k / 534k = 0.0187\ni.e. for 1V on V_control, the output\nwill change by 18.7mV."
- note removed: "R3 * C1 should be 100µs, this affects the frequency range\nR3 : R5 must be 2:1, this affects the triangle shape\nR4 : R6 must be 1:1, this affects the triangle shape\nR8 : R9 should be 1:2, this affects the triangle amplitude and\nfrequency range. If R9 is too large, this may cause distortion\nR11 : R12 should be 1:1, this affects sawtooth amplitude"
- note removed: "for Q4, the following holds true:\nI_C = const * exp(V_B / VT) with VT=26mV\n(thermal voltage of a transistor)\nnow this means that Vout will double\nevery (log(2) * 26mV) = 18mV."
- moved on the sheet: C2, Q3, Q4, R1, R10, R16, R17, R18, R2, U1, U4, U6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

Commit message: add buffer to measure_vco schematic
Parts:
- added U?: LM324, symbol pspice:OPAMP
Connections:
- net -VDC: now also U?.5 (V-); no longer U7.5 (V-)
- net VCC: now also U?.4 (V+); no longer U7.4 (V+)
- net V_expo: now also U?.1 (+), U?.3; no longer R18.1, U7.3
- new net: R18.1, U7.3, U?.2 (-)
Other:
- note added: "This buffer is not\nneccessary, but it\nwas on my bread-\nboard. So for the\nsake of documen-\ntation...\nActually, tuning\naccuracy might\nbe a bit better\nwithout."
Changed lines of the file:
@@
 Wire Wire Line
 	7700 1700 7550 1700
-Text GLabel 7700 1700 2    50   Input ~ 0
+Text GLabel 8150 2425 1    50   Input ~ 0
 V_expo
 Connection ~ 6700 1600
@@
 L power:VCC #PWR023
 U 1 1 5CFF2C24
-P 7050 2000
-F 0 "#PWR023" H 7050 1850 50  0001 C CNN
-F 1 "VCC" H 7068 2173 50  0000 C CNN
-F 2 "" H 7050 2000 50  0001 C CNN
-F 3 "" H 7050 2000 50  0001 C CNN
-	1    7050 2000
-	-1   0    0    1
+P 7900 2100
+F 0 "#PWR023" H 7900 1950 50  0001 C CNN
+F 1 "VCC" H 7918 2273 50  0000 C CNN
+F 2 "" H 7900 2100 50  0001 C CNN
+F 3 "" H 7900 2100 50  0001 C CNN
+	1    7900 2100
+	1    0    0    1
 $EndComp
 $Comp
@@
 L power:VEE #PWR022
 U 1 1 5CFF1E9C
-P 7050 1400
-F 0 "#PWR022" H 7050 1250 50  0001 C CNN
-F 1 "VEE" H 7067 1573 50  0000 C CNN
-F 2 "" H 7050 1400 50  0001 C CNN
-F 3 "" H 7050 1400 50  0001 C CNN
-	1    7050 1400
-	1    0    0    -1
+P 7900 1500
+F 0 "#PWR022" H 7900 1350 50  0001 C CNN
+F 1 "VEE" H 7917 1673 50  0000 C CNN
+F 2 "" H 7900 1500 50  0001 C CNN
+F 3 "" H 7900 1500 50  0001 C CNN
+	1    7900 1500
+	-1   0    0    -1
 $EndComp
 $Comp
@@
 Text Notes 475  1750 0    50   ~ 0
 ca 290mV/oct
+$Comp
+L pspice:OPAMP U?
+U 1 1 5D421CD1
+P 8000 1800
+F 0 "U?" H 8150 1700 50  0000 L CNN
+F 1 "LM324" H 8100 1600 50  0000 L CNN
+F 2 "" H 8000 1800 50  0001 C CNN
+F 3 "~" H 8000 1800 50  0001 C CNN
+F 4 "X" H 8000 1800 50  0001 C CNN "Spice_Primitive"
+F 5 "LM324" H 8000 1800 50  0001 C CNN "Spice_Model"
+F 6 "Y" H 8000 1800 50  0001 C CNN "Spice_Netlist_Enabled"
+F 7 "LM324.ti.lib" H 8000 1800 50  0001 C CNN "Spice_Lib_File"
+F 8 "1,2,4,5,3" H 8000 1800 50  0001 C CNN "Spice_Node_Sequence"
+	1    8000 1800
+	1    0    0    1
+$EndComp
+Wire Wire Line
+	8300 1800 8300 2425
+Wire Wire Line
+	8300 2425 7700 2425
+Wire Wire Line
+	7700 2425 7700 1900
+Text Notes 7675 3250 0    50   ~ 0
+This buffer is not\nneccessary, but it\nwas on my bread-\nboard. So for the\nsake of documen-\ntation...\nActually, tuning\naccuracy might\nbe a bit better\nwithout.
+Wire Notes Line
+	7650 3275 8400 3275
+Wire Notes Line
+	8400 3275 8400 1225
+Wire Notes Line
+	8400 1225 7650 1225
+Wire Notes Line
+	7650 1225 7650 3275
 $EndSCHEMATC

Commit message: update measure_vco schematics
Parts:
- removed C1: 1n, symbol pspice:C
- removed C2: 1n, symbol Device:C
- removed D3: D, symbol Device:D
- removed Q1: 2N7000, Package_TO_SOT_THT:TO-92_Inline, symbol Transistor_FET:2N7000
- removed Q3, Q4: 1/2 BCM847, symbol pspice:QNPN
- removed R12: 150, symbol Device:R
- removed R13: 1k, symbol Device:Thermistor_NTC
- removed R14, R17: 1k, symbol Device:R
- removed R15: 2.2k, symbol Device:R
- removed R16, R23, R3, R9: 100k, symbol Device:R
- removed R18, R7: 10k, symbol Device:R
- removed R19: 147k, symbol Device:R
- removed R20: 12k2, symbol Device:R
- removed R21: 220k, symbol Device:R
- removed R22: 4.7k, symbol Device:R
- removed R24: 1k, symbol Device:R_POT_TRIM
- removed R4, R5, R6: 47k, symbol Device:R
- removed R8: 50k, symbol Device:R
- removed U2, U3, U6, U7, U8, U?: LM324, symbol pspice:OPAMP
- added Q?: BC547, Package_TO_SOT_THT:TO-92_Inline, symbol Transistor_BJT:BC547
- added R?: 10k, symbol Device:R
- added R?: 1k, symbol Device:R
- added R?: 100k, symbol Device:R
- added RV?: 1k, symbol Device:R_POT
Connections:
- net -VDC: now also R?.1
- net GNDREF: now also RV?.3
- net VCC: now also Q?.1 (C)
- net V_control: now also R?.1; no longer U4.8 (VA)
- net square_ctl: now also R?.2; no longer R11.1
- new net: RV?.1, U4.8 (VA)
- new net: Q?.3 (E), R11.1, R?.2
- new net: Q?.2 (B), R?.1
- new net: R?.2, RV?.2
Other:
- note added: "poti at ca 40%"
- note added: "transistor buffer.\nsquare_ctl is very sensitive,\nloading it will affect the\nfrequency and pulse width\nof the oscillator"
- note removed: "Because R8 is connected to GNDREF, the triangle would be\ncentered around GNDREF, but only if the output of the\ncomparator U3 would swing between Vcc and Vee.\nHowever, U3 swings between less-than-Vcc and\nexactly Vee, so the triangle isn't centered."
- note removed: "Changing the R8/R9 ratio affects the maximum frequency\nand the triangle's amplitude. R8 = 16k has proved to work,\nproviding very high maximum frequencies.\nR8 = 5k and R9 = 10k works fine, too."
- note removed: "R16 determines the I_C current through\nQ4 when Q4's base is at GNDREF.\nTogether with V_tune, it determines the pitch.\nChoose R16 and V_tune such, that U8's output needs\nto be at around GNDREF for "sane" pitches."
- note removed: "R3 * C1 should be 100µs, this affects the frequency range\nR3 : R5 must be 2:1, this affects the triangle shape\nR4 : R6 must be 1:1, this affects the triangle shape\nR8 : R9 should be 1:2, this affects the triangle amplitude and\nfrequency range. If R9 is too large, this may cause distortion"
- note removed: "Rossum\ncompensation"
- note removed: "This buffer is not\nneccessary, but it\nwas on my bread-\nboard. So for the\nsake of documen-\ntation...\nActually, tuning\naccuracy might\nbe a bit better\nwithout."
- note removed: "ca 18mV/oct"
- note removed: "ca 19mV/Oct"
- note removed: "ca 24mV/oct"
- note removed: "ca 290mV/oct"
- note removed: "for Q4, the following holds true:\nI_C = const * exp(V_B / VT) with VT=26mV\n(thermal voltage of a transistor)\nnow this means that Vout will double\nevery (log(2) * 26mV) = 18mV.\n\nNote that VT is temperature dependent.\nWhen the temperature rises, VT rises and so\nthe input voltage must rise too. The thermal\ncompensation consisting of TODO does that.\n\nAdditionally, Q3 and Q4 have a bulk res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"
- note removed: "or use\n2x BC547"
- note removed: "replace this GNDREF by a\nvoltage source ca. 1mV-\n1.5mV below GNDREF for\nbest results."
- note removed: "thermal\ncompensation"
- note removed: "unused"
- moved on the sheet: D1, D2, R11, U4
