File: hardware/vca/vca.sch (KiCad schematic (older format))
At the start: 20 parts

Commit message: changed vca
Parts:
- added C?: 470u, symbol Device:C
- added R? (x2): 100k, symbol Device:R
- added R?: 1k, symbol Device:R_Variable
- added R? (x2): 1k, symbol Device:R
Connections:
- net GNDREF: now also U?.3 (+), R?.1; no longer RV?.1
- net signal_in: now also C?.2; no longer Q?.2 (B)
- net v_control: now also R?.2; no longer R?.1, U?.1, U?.2 (-)
- net at RV?.2: now also R?.1; no longer U?.3 (+)
- new net: R?.1, RV?.1, U?.1
- new net: R?.1, R?.2, U?.2 (-)
- new net: Q?.2 (B), R?.2, R?.2
- new net: R?.1, R?.1
- new net: C?.1, R?.2
Other:
- note added: "input preattenuation.\ncontrols distortion"
- note added: "v_control ranges between\n0=GND and +Vcc and is\nconverted to -Vee to 0 here\n"
- moved on the sheet: RV?, U?A
Changed lines of the file:
@@
 L Amplifier_Operational:TL074 U?
 U 1 1 5D8E8672
-P 5250 2000
-F 0 "U?" H 5275 2175 50  0000 C CNN
-F 1 "TL074" H 5275 2000 50  0000 C CNN
-F 2 "" H 5200 2100 50  0001 C CNN
-F 3 "http://www.ti.com/lit/ds/symlink/tl071.pdf" H 5300 2200 50  0001 C CNN
-	1    5250 2000
+P 5225 1725
+F 0 "U?" H 5250 1900 50  0000 C CNN
+F 1 "TL074" H 5250 1725 50  0000 C CNN
+F 2 "" H 5175 1825 50  0001 C CNN
+F 3 "http://www.ti.com/lit/ds/symlink/tl071.pdf" H 5275 1925 50  0001 C CNN
+	1    5225 1725
 	1    0    0    -1
 $EndComp
@@
 L Amplifier_Operational:TL074 U?
 U 5 1 5D8EBDB3
-P 5250 2000
-F 0 "U?" H 5208 2046 50  0001 L CNN
-F 1 "TL074" H 5208 2000 50  0001 L CNN
-F 2 "" H 5200 2100 50  0001 C CNN
-F 3 "http://www.ti.com/lit/ds/symlink/tl071.pdf" H 5300 2200 50  0001 C CNN
-	5    5250 2000
+P 5225 1725
+F 0 "U?" H 5183 1771 50  0001 L CNN
+F 1 "TL074" H 5183 1725 50  0001 L CNN
+F 2 "" H 5175 1825 50  0001 C CNN
+F 3 "http://www.ti.com/lit/ds/symlink/tl071.pdf" H 5275 1925 50  0001 C CNN
+	5    5225 1725
 	1    0    0    -1
 $EndComp
@@
 L Device:R_POT RV?
 U 1 1 5D8F28FE
-P 4700 1900
-F 0 "RV?" H 4630 1946 50  0000 R CNN
-F 1 "50k" V 4700 1975 50  0000 R CNN
-F 2 "" H 4700 1900 50  0001 C CNN
-F 3 "~" H 4700 1900 50  0001 C CNN
-	1    4700 1900
+P 5775 2000
+F 0 "RV?" H 5705 2046 50  0000 R CNN
+F 1 "50k" V 5775 2075 50  0000 R CNN
+F 2 "" H 5775 2000 50  0001 C CNN
+F 3 "~" H 5775 2000 50  0001 C CNN
+	1    5775 2000
 	1    0    0    -1
 $EndComp
@@
 L power:VEE #PWR?
 U 1 1 5D8F3591
-P 4700 2050
-F 0 "#PWR?" H 4700 1900 50  0001 C CNN
-F 1 "VEE" H 4718 2223 50  0000 C CNN
-F 2 "" H 4700 2050 50  0001 C CNN
-F 3 "" H 4700 2050 50  0001 C CNN
-	1    4700 2050
+P 5775 2150
+F 0 "#PWR?" H 5775 2000 50  0001 C CNN
+F 1 "VEE" H 5793 2323 50  0000 C CNN
+F 2 "" H 5775 2150 50  0001 C CNN
+F 3 "" H 5775 2150 50  0001 C CNN
+	1    5775 2150
 	-1   0    0    1
 $EndComp
@@
 L power:GNDREF #PWR?
 U 1 1 5D8F40C2
-P 4550 1650
-F 0 "#PWR?" H 4550 1400 50  0001 C CNN
-F 1 "GNDREF" H 4555 1477 50  0001 C CNN
-F 2 "" H 4550 1650 50  0001 C CNN
-F 3 "" H 4550 1650 50  0001 C CNN
-	1    4550 1650
-	1    0    0    -1
-$EndComp
-Wire Wire Line
-	4550 1650 4700 1650
-Wire Wire Line
-	4700 1650 4700 1750
+P 4925 1625
+F 0 "#PWR?" H 4925 1375 50  0001 C CNN
+F 1 "GNDREF" H 4930 1452 50  0001 C CNN
+F 2 "" H 4925 1625 50  0001 C CNN
+F 3 "" H 4925 1625 50  0001 C CNN
+	1    4925 1625
+	1    0    0    -1
+$EndComp
 $Comp
 L power:VEE #PWR?
 U 1 1 5D902B53
-P 5150 2300
-F 0 "#PWR?" H 5150 2150 50  0001 C CNN
-F 1 "VEE" H 5168 2473 50  0000 C CNN
-F 2 "" H 5150 2300 50  0001 C CNN
-F 3 "" H 5150 2300 50  0001 C CNN
-	1    5150 2300
+P 5125 2025
+F 0 "#PWR?" H 5125 1875 50  0001 C CNN
+F 1 "VEE" H 5143 2198 50  0000 C CNN
+F 2 "" H 5125 2025 50  0001 C CNN
+F 3 "" H 5125 2025 50  0001 C CNN
+	1    5125 2025
 	-1   0    0    1
 $EndComp
@@
 L power:VCC #PWR?
 U 1 1 5D9039B8
-P 5150 1700
-F 0 "#PWR?" H 5150 1550 50  0001 C CNN
-F 1 "VCC" H 5167 1873 50  0000 C CNN
-F 2 "" H 5150 1700 50  0001 C CNN
-F 3 "" H 5150 1700 50  0001 C CNN
-	1    5150 1700
-	1    0    0    -1
-$EndComp
-Wire Wire Line
-	4950 2100 4950 2525
-Wire Wire Line
-	4950 2525 5550 2525
-Wire Wire Line
-	5550 2525 5550 2000
-Wire Wire Line
-	4850 1900 4950 1900
+P 5125 1425
+F 0 "#PWR?" H 5125 1275 50  0001 C CNN
+F 1 "VCC" H 5142 1598 50  0000 C CNN
+F 2 "" H 5125 1425 50  0001 C CNN
+F 3 "" H 5125 1425 50  0001 C CNN
+	1    5125 1425
+	1    0    0    -1
+$EndComp
 $Comp
 L Device:R R?
@@
 Text Notes 6750 1575 2    50   ~ 0
 differential pair\n(current controlled\namplification)
-Wire Wire Line
-	6325 2000 5550 2000
-Connection ~ 5550 2000
-Text GLabel 5925 2000 3    50   Input ~ 0
+Text GLabel 4625 1825 0    50   Input ~ 0
 v_control
-Text GLabel 6500 1800 0    50   Input ~ 0
+Text GLabel 5475 600  0    50   Input ~ 0
 signal_in
 Text GLabel 8725 1450 2    50   Input ~ 0
 signal_out
+Wire Wire Line
+	6325 2000 5925 2000
+Wire Wire Line
+	5525 1725 5775 1725
+Wire Wire Line
+	5775 1725 5775 1850
+$Comp
+L Device:R R?
+U 1 1 5DA36ABE
+P 5150 2350
+F 0 "R?" V 5050 2325 50  0000 L CNN
+F 1 "100k" V 5150 2250 50  0000 L CNN
+F 2 "" V 5080 2350 50  0001 C CNN
+F 3 "~" H 5150 2350 50  0001 C CNN
+	1    5150 2350
+	0    1    -1   0
+$EndComp
+Wire Wire Line
+	5525 1725 5525 2350
+Wire Wire Line
+	5525 2350 5300 2350
+Connection ~ 5525 1725
+Wire Wire Line
+	5000 2350 4925 2350
+Wire Wire Line
+	4925 2350 4925 1825
+$Comp
+L Device:R R?
+U 1 1 5DA3A90A
+P 4775 1825
+F 0 "R?" V 4675 1800 50  0000 L CNN
+F 1 "100k" V 4775 1725 50  0000 L CNN
+F 2 "" V 4705 1825 50  0001 C CNN
+F 3 "~" H 4775 1825 50  0001 C CNN
+	1    4775 1825
+	0    1    -1   0
+$EndComp
+Connection ~ 4925 1825
+Text Notes 4525 2750 0    50   ~ 0
+v_control ranges between\n0=GND and +Vcc and is\nconverted to -Vee to 0 here\n
+$Comp
+L Device:R_Variable R?
+U 1 1 5DA5A9B7
+P 5775 1050
+F 0 "R?" H 5900 1075 50  0000 L CNN
+F 1 "1k" H 5825 1000 50  0000 L CNN
+F 2 "" V 5705 1050 50  0001 C CNN
+F 3 "~" H 5775 1050 50  0001 C CNN
+	1    5775 1050
+	1    0    0    -1
+$EndComp
+$Comp
+L Device:R R?
+U 1 1 5DA5E13B
+P 5775 750
+F 0 "R?" H 5850 700 50  0000 L CNN
+F 1 "1k" V 5775 700 50  0000 L CNN
+F 2 "" V 5705 750 50  0001 C CNN
+F 3 "~" H 5775 750 50  0001 C CNN
+	1    5775 750
+	1    0    0    1
+$EndComp
+$Comp
+L Device:R R?
+U 1 1 5DA5ECCF
+P 5775 1350
+F 0 "R?" H 5850 1300 50  0000 L CNN
+F 1 "1k" V 5775 1300 50  0000 L CNN
+F 2 "" V 5705 1350 50  0001 C CNN
+F 3 "~" H 5775 1350 50  0001 C CNN
+	1    5775 1350
+	1    0    0    1
+$EndComp
+$Comp
+L Device:C C?
+U 1 1 5DA64FC2
+P 5625 600
+F 0 "C?" V 5373 600 50  0000 C CNN
+F 1 "470u" V 5464 600 50  0000 C CNN
+F 2 "" H 5663 450 50  0001 C CNN
+F 3 "~" H 5625 600 50  0001 C CNN
+	1    5625 600
+	0    1    1    0
+$EndComp
+$Comp
+L power:GNDREF #PWR?
+U 1 1 5DA6EBCF
+P 5775 1500
+F 0 "#PWR?" H 5775 1250 50  0001 C CNN
+F 1 "GNDREF" H 5780 1327 50  0001 C CNN
+F 2 "" H 5775 1500 50  0001 C CNN
+F 3 "" H 5775 1500 50  0001 C CNN
+	1    5775 1500
+	1    0    0    -1
+$EndComp
+Wire Wire Line
+	5775 1200 5975 1200
+Connection ~ 5775 1200
+Wire Wire Line
+	6500 1800 5975 1800
+Wire Wire Line
+	5975 1800 5975 1200
+Text Notes 4925 900  0    50   ~ 0
+input preattenuation.\ncontrols distortion
 $EndSCHEMATC

Commit message: schematic for the new firmware setup
Parts:
- added C?: 470u, symbol Device:C
- added Q? (x4): BC327, Package_TO_SOT_THT:TO-92_Inline, symbol Transistor_BJT:BC327
- added R? (x4): 10k, symbol Device:R
- added R?: 1k, symbol Device:R_Variable
- added R? (x2): 1k, symbol Device:R
Connections:
- wire segments 33 -> 44
Changed lines of the file:
@@
 EESchema Schematic File Version 4
+LIBS:vca-cache
 EELAYER 30 0
 EELAYER END
@@
 Text Notes 4925 900  0    50   ~ 0
 input preattenuation.\ncontrols distortion
+$Comp
+L Transistor_BJT:BC327 Q?
+U 1 1 5D927D0A
+P 9400 3625
+F 0 "Q?" H 9300 3775 50  0000 L CNN
+F 1 "BC327" H 9075 3550 50  0000 L CNN
+F 2 "Package_TO_SOT_THT:TO-92_Inline" H 9600 3550 50  0001 L CIN
+F 3 "http://www.onsemi.com/pub_link/Collateral/BC327-D.PDF" H 9400 3625 50  0001 L CNN
+	1    9400 3625
+	1    0    0    1
+$EndComp
+$Comp
+L Transistor_BJT:BC327 Q?
+U 1 1 5D936D87
+P 9000 3625
+F 0 "Q?" H 8875 3775 50  0000 L CNN
+F 1 "BC327" H 9191 3580 50  0001 L CNN
+F 2 "Package_TO_SOT_THT:TO-92_Inline" H 9200 3550 50  0001 L CIN
+F 3 "http://www.onsemi.com/pub_link/Collateral/BC327-D.PDF" H 9000 3625 50  0001 L CNN
+	1    9000 3625
+	-1   0    0    1
+$EndComp
+$Comp
+L power:VCC #PWR?
+U 1 1 5D942900
+P 9200 3425
+F 0 "#PWR?" H 9200 3275 50  0001 C CNN
+F 1 "VCC" H 9217 3598 50  0000 C CNN
+F 2 "" H 9200 3425 50  0001 C CNN
+F 3 "" H 9200 3425 50  0001 C CNN
+	1    9200 3425
+	1    0    0    -1
+$EndComp
+Wire Wire Line
+	9500 3425 9200 3425
+Connection ~ 9200 3425
+Wire Wire Line
+	9200 3425 8900 3425
+Wire Wire Line
+	9200 3625 9200 3825
+Connection ~ 9200 3625
+Wire Wire Line
+	9200 3825 8900 3825
+$Comp
+L Device:R R?
+U 1 1 5D94CF4E
+P 8900 3975
+F 0 "R?" H 8970 4021 50  0000 L CNN
+F 1 "10k" V 8900 3900 50  0000 L CNN
+F 2 "" V 8830 3975 50  0001 C CNN
+F 3 "~" H 8900 3975 50  0001 C CNN
+	1    8900 3975
+	1    0    0    -1
+$EndComp
+Connection ~ 8900 3825
+Connection ~ 9500 4125
+$Comp
+L Device:R R?
+U 1 1 5D95F81E
+P 9500 3975
+F 0 "R?" H 9570 4021 50  0000 L CNN
+F 1 "10k" V 9500 3900 50  0000 L CNN
+F 2 "" V 9430 3975 50  0001 C CNN
+F 3 "~" H 9500 3975 50  0001 C CNN
+	1    9500 3975
+	1    0    0    1
+$EndComp
+Wire Wire Line
+	9375 4125 9500 4125
+Wire Wire Line
+	9500 4125 9625 4125
+$Comp
+L power:GNDREF #PWR?
+U 1 1 5D95F82A
+P 9925 4325
+F 0 "#PWR?" H 9925 4075 50  0001 C CNN
+F 1 "GNDREF" H 9930 4152 50  0001 C CNN
+F 2 "" H 9925 4325 50  0001 C CNN
+F 3 "" H 9925 4325 50  0001 C CNN
+	1    9925 4325
+	-1   0    0    -1
+$EndComp
+$Comp
+L Transistor_BJT:BC327 Q?
+U 1 1 5D96447B
+P 9725 4325
+F 0 "Q?" H 9600 4475 50  0000 L CNN
+F 1 "BC327" H 9916 4280 50  0001 L CNN
+F 2 "Package_TO_SOT_THT:TO-92_Inline" H 9925 4250 50  0001 L CIN
+F 3 "http://www.onsemi.com/pub_link/Collateral/BC327-D.PDF" H 9725 4325 50  0001 L CNN
+	1    9725 4325
+	-1   0    0    1
+$EndComp
+$Comp
+L Transistor_BJT:BC327 Q?
+U 1 1 5D969E4D
+P 9275 4325
+F 0 "Q?" H 9150 4475 50  0000 L CNN
+F 1 "BC327" V 9500 4200 50  0000 L CNN
+F 2 "Package_TO_SOT_THT:TO-92_Inline" H 9475 4250 50  0001 L CIN
+F 3 "http://www.onsemi.com/pub_link/Collateral/BC327-D.PDF" H 9275 4325 50  0001 L CNN
+	1    9275 4325
+	1    0    0    1
+$EndComp
+$Comp
+L Device:R R?
+U 1 1 5D97C329
+P 9375 4675
+F 0 "R?" H 9445 4721 50  0000 L CNN
+F 1 "10k" V 9375 4600 50  0000 L CNN
+F 2 "" V 9305 4675 50  0001 C CNN
+F 3 "~" H 9375 4675 50  0001 C CNN
+	1    9375 4675
+	1    0    0    1
+$EndComp
+$Comp
+L Device:R R?
+U 1 1 5D97C9D7
+P 9625 4675
+F 0 "R?" H 9695 4721 50  0000 L CNN
+F 1 "10k" V 9625 4600 50  0000 L CNN
+F 2 "" V 9555 4675 50  0001 C CNN
+F 3 "~" H 9625 4675 50  0001 C CNN
+	1    9625 4675
+	1    0    0    1
+$EndComp
+$Comp
+L power:VEE #PWR?
+U 1 1 5D9809F3
+P 9625 4825
+F 0 "#PWR?" H 9625 4675 50  0001 C CNN
+F 1 "VEE" H 9643 4998 50  0000 C CNN
+F 2 "" H 9625 4825 50  0001 C CNN
+F 3 "" H 9625 4825 50  0001 C CNN
+	1    9625 4825
+	-1   0    0    1
+$EndComp
+$Comp
+L power:VEE #PWR?
+U 1 1 5D9813BC
+P 9375 4825
+F 0 "#PWR?" H 9375 4675 50  0001 C CNN
+F 1 "VEE" H 9393 4998 50  0000 C CNN
+F 2 "" H 9375 4825 50  0001 C CNN
+F 3 "" H 9375 4825 50  0001 C CNN
+	1    9375 4825
+	-1   0    0    1
+$EndComp
+Text GLabel 8100 3725 0    50   Input ~ 0
+signal_in
+$Comp
+L Device:R_Variable R?
+U 1 1 5D9A8C32
+P 8400 4175
+F 0 "R?" H 8525 4200 50  0000 L CNN
+F 1 "1k" H 8450 4125 50  0000 L CNN
+F 2 "" V 8330 4175 50  0001 C CNN
+F 3 "~" H 8400 4175 50  0001 C CNN
+	1    8400 4175
+	1    0    0    -1
+$EndComp
+$Comp
+L Device:R R?
+U 1 1 5D9A8C3C
+P 8400 3875
+F 0 "R?" H 8475 3825 50  0000 L CNN
+F 1 "1k" V 8400 3825 50  0000 L CNN
+F 2 "" V 8330 3875 50  0001 C CNN
+F 3 "~" H 8400 3875 50  0001 C CNN
+	1    8400 3875
+	1    0    0    1
+$EndComp
+$Comp
+L Device:R R?
+U 1 1 5D9A8C46
+P 8400 4475
+F 0 "R?" H 8475 4425 50  0000 L CNN
+F 1 "1k" V 8400 4425 50  0000 L CNN
+F 2 "" V 8330 4475 50  0001 C CNN
+F 3 "~" H 8400 4475 50  0001 C CNN
+	1    8400 4475
+	1    0    0    1
+$EndComp
+$Comp
+L Device:C C?
+U 1 1 5D9A8C50
+P 8250 3725
+F 0 "C?" V 7998 3725 50  0000 C CNN
+F 1 "470u" V 8089 3725 50  0000 C CNN
+F 2 "" H 8288 3575 50  0001 C CNN
+F 3 "~" H 8250 3725 50  0001 C CNN
+	1    8250 3725
+	0    1    1    0
+$EndComp
+Connection ~ 8400 4325
+Text Notes 7550 4025 0    50   ~ 0
+input preattenuation.\ncontrols distortion
+$Comp
+L power:GNDREF #PWR?
+U 1 1 5D9C7217
+P 8400 4625
+F 0 "#PWR?" H 8400 4375 50  0001 C CNN
+F 1 "GNDREF" H 8405 4452 50  0001 C CNN
+F 2 "" H 8400 4625 50  0001 C CNN
+F 3 "" H 8400 4625 50  0001 C CNN
+	1    8400 4625
+	1    0    0    -1
+$EndComp
+Wire Wire Line
+	8400 4325 9075 4325
+Wire Wire Line
+	8900 4125 8900 4175
+Wire Wire Line
+	8900 4175 8700 4175
+Wire Wire Line
+	8700 4175 8700 3200
+Wire Wire Line
+	8700 3200 8350 3200
 $EndSCHEMATC
