File: hardware/voice_board/voice_board.sch (KiCad schematic (older format))
At the start: 90 parts

Commit message: boards++
Parts:
- removed R?: 1k, symbol Device:R
- removed R?: 100k, symbol Device:R
- removed RV?: 1k, symbol Device:R_POT
- added C? (x2): 1u, symbol Device:C
- added J?: Conn_01x02_Male, symbol Connector:Conn_01x02_Male
- added J?: Conn_02x02_Odd_Even, symbol Connector_Generic:Conn_02x02_Odd_Even
- added R?: 100k, symbol Device:R
- added RV? (x2): 1k, symbol Device:R_POT
- R?: value 110k -> 100k
Connections:
- net +3V3: now also J?.1 (Pin_1); no longer J?.2 (Pin_2)
- net GND: now also C?.2, C?.2, RV?.3, RV?.3
- net PB12: now also J?.2 (Pin_2)
- net PB13: now also J?.4 (Pin_4)
- net PB15: now also J?.3 (Pin_3)
- net at U?.6 (VB): now also C?.1, RV?.1
- net at U?.8 (VA): now also C?.1, RV?.1
- net vca_ctl_raw: now reaches R?.1, R?.2, U?.2 (-)
- net vca_ctl_raw: now also R?.2
- net vca_ctl renamed vca_ctl2
- new net: J?.2 (Pin_2), RV?.2
- new net: J?.1 (Pin_1), RV?.2
- new net vca_ctl1: R?.1
- no-connect marks 0 -> 1
Other:
- note added: "TODO: replace that 50k poti\nwith input adjusts at vca_ctl"
- note removed: "TODO"
- note removed: "or 100k? TODO:\ntune so that the\nopamp does not\nclip the envelope"
- moved on the sheet: R?

Commit message: proper VCF ctl input stage
Parts:
- removed R?: 1k, symbol Device:R
- removed RV?: 1k, symbol Device:R_POT
- added R? (x3): 100k, symbol Device:R
- added R?: 200k, symbol Device:RTRIM
- added R?: 10k, symbol Device:R
- added R?: 10k, symbol Device:R_Variable
- added U?: TL074, symbol Amplifier_Operational:TL074
Connections:
- net GND: now also U?.3 (+)
- net VCC: now also R?.1
- net VEE: now also R?.2
- net vcf_audio_in: now also R?.2; no longer R?.1
- net at C?.2, R?.2: now also R?.1; no longer R?.2
- net at R?.2: now also Q?.1 (C); no longer Q?.1 (C)
- net at Q?.2 (B), Q?.2 (B): now also Q?.1 (C), R?.2, R?.2; no longer Q?.1 (C)
- new net: R?.1, R?.2, U?.1
- new net vcf_ctl1: R?.1
- new net vcf_ctl2: R?.1
- new net vcf_ctl_raw: R?.1, R?.1, R?.2, R?.2, U?.2 (-)
Other:
- note added: "TODO: expo converter for the VCF input"
- note added: "offset compensation: the OpAmp would\nneed to output exactly Vcc - 0.7V (i.e., the voltage\nat the transistor's base) in order to fully close the\nVCF. However, the OpAmp is limited to approx. Vcc-1.5V,\nso we inject some current through this trimming poti.\nWhen the OpAmp is at its Vmax, tune this poti such that\nthe VCF is just fully closed.\n"
- note added: "set such, that with zero control input, the\noutput of the op amp is just at maximum\n(i.e., Vcc minus like 1 V or so)"
- note added: "set to 100k"
- note added: "set to 7.26k"
- note added: "should be 2x 47k maybe"
- note removed: "TODO: input stage similar to VCA"
- note removed: "TODO: multiple inputs, one raw"
- moved on the sheet: Q?, R?

Commit message: general purpose filters, VCA input stage
Parts:
- removed Q? (x2): BC327, Package_TO_SOT_THT:TO-92_Inline, symbol Transistor_BJT:BC327
- removed R?: 110k, symbol Device:R
- removed R?: 100k, symbol Device:R_Variable
- removed R? (x5): 100k, symbol Device:R
- removed RV?: 50k, symbol Device:R_POT
- removed U?: TL074, symbol Amplifier_Operational:TL074
- added C? (x3): any, symbol Device:C
- added J?: Conn_02x03_Odd_Even, symbol Connector_Generic:Conn_02x03_Odd_Even
- added Q? (x2): BC557, Package_TO_SOT_THT:TO-92_Inline, symbol Transistor_BJT:BC557
- added R? (x4): 100k, symbol Device:R
- added R?: 100k, symbol Device:R_Variable
- added R?: 200k, symbol Device:RTRIM
- added R? (x3): any, symbol Device:R_Variable
- added U?: TL074, symbol Amplifier_Operational:TL074
Connections:
- net GND: now also C?.2, C?.2, C?.2, U?.3 (+)
- net VCC: now also Q?.3 (E), Q?.3 (E), R?.1
- net VEE: now also R?.2
- net vca_ctl1: now also R?.1
- net vca_ctl2: now also R?.1
- net vca_ctl_raw: now also R?.1, R?.1, R?.2, R?.2, U?.2 (-)
- net at R?.2: now also Q?.1 (C)
- new net: Q?.1 (C), Q?.2 (B), Q?.2 (B), R?.2, R?.2
- new net: R?.1, R?.2, U?.1
- new net: C?.1, J?.2 (Pin_2), R?.1
- new net: J?.1 (Pin_1), R?.2
- new net: C?.1, J?.4 (Pin_4), R?.1
- new net: J?.3 (Pin_3), R?.2
- new net: C?.1, J?.6 (Pin_6), R?.1
- new net: J?.5 (Pin_5), R?.2
Other:
- note added: "TODO: more square_ctl_buf outputs.\nor add the clamping circuitry here"
- note added: "TODO: or just put a resistor here\nor a proper poti for opening the filter."
- note added: "general\npurpose\nlow pass\nfilters"
- note removed: "TODO: two low pass filters\nfor general purpose (portamento?)"

Commit message: some todos
Other:
- note added: "TODO: some input preattenuators for all control inputs"
- note added: "TODO\n- input preattenuators\n- input pre-bias\n- expo for filter\n- what to do about the clamping?\n- connectors"
Changed lines of the file:
@@
 Wire Notes Line
 	6325 4650 6325 6150
+Text Notes 475  300  0    50   ~ 0
+TODO: some input preattenuators for all control inputs
+Text Notes 450  -575 0    50   ~ 0
+TODO\n- input preattenuators\n- input pre-bias\n- expo for filter\n- what to do about the clamping?\n- connectors
 $EndSCHEMATC

Commit message: add pre-bias poti for the VCF
Parts:
- removed R?: 200k, symbol Device:RTRIM
- added R?: 47k, symbol Device:R
- added RV?: 100k, symbol Device:R_POT
Connections:
- net VCC: now also RV?.1
- net VEE: now also RV?.3
- net vcf_ctl_raw: now also R?.2
- new net: R?.1, RV?.2
Other:
- note added: "TODO\n- input preattenuators\n- expo for filter\n- what to do about the clamping?\n- connectors"
- note added: "or connect (-) with ~~100k to VEE\n(like the VCA)"
- note removed: "TODO: or just put a resistor here\nor a proper poti for opening the filter."
- note removed: "TODO: raw in"
- note removed: "TODO: replace that 50k poti\nwith input adjusts at vca_ctl"
- note removed: "TODO\n- input preattenuators\n- input pre-bias\n- expo for filter\n- what to do about the clamping?\n- connectors"
Changed lines of the file:
@@
 	0    -1   1    0
 $EndComp
-Text Notes 5450 3775 0    50   ~ 0
-TODO: raw in
 Text Notes 4975 3025 0    50   ~ 0
 mixer
@@
 Wire Notes Line
 	450  725  4450 725
-Text Notes 500  675  0    50   ~ 0
-TODO: replace that 50k poti\nwith input adjusts at  vca_ctl
 $Comp
 L Device:R R?
@@
 Text Notes 6425 700  0    50   ~ 0
 TODO: expo converter for the VCF input
-Text Notes 6425 1825 0    50   ~ 0
-set such, that with zero control input, the\noutput of the op amp is just at maximum\n(i.e., Vcc minus like 1 V or so)
-Connection ~ 8150 1325
-$Comp
-L Device:RTRIM R?
-U 1 1 5E3D0F12
-P 8000 1325
-F 0 "R?" V 7900 1200 50  0000 C CNN
-F 1 "200k" V 7900 1375 50  0000 C CNN
-F 2 "" V 7930 1325 50  0001 C CNN
-F 3 "~" H 8000 1325 50  0001 C CNN
-	1    8000 1325
-	0    1    -1   0
-$EndComp
-Wire Wire Line
-	7800 1325 7850 1325
-Wire Wire Line
-	7800 1375 7800 1325
 $Comp
 L power:VEE #PWR?
 U 1 1 5E3C6C3C
-P 7800 1375
-F 0 "#PWR?" H 7800 1225 50  0001 C CNN
-F 1 "VEE" H 7818 1548 50  0000 C CNN
-F 2 "" H 7800 1375 50  0001 C CNN
-F 3 "" H 7800 1375 50  0001 C CNN
-	1    7800 1375
+P 7500 1650
+F 0 "#PWR?" H 7500 1500 50  0001 C CNN
+F 1 "VEE" H 7625 1750 50  0000 C CNN
+F 2 "" H 7500 1650 50  0001 C CNN
+F 3 "" H 7500 1650 50  0001 C CNN
+	1    7500 1650
 	-1   0    0    1
 $EndComp
-Text Notes 7325 1375 0    50   ~ 0
-set to 100k
 Connection ~ 8150 1000
 $Comp
@@
 Text Notes 2350 5825 0    50   ~ 0
 TODO: more square_ctl_buf outputs.\nor add the clamping circuitry here
-Text Notes 6225 1525 0    50   ~ 0
-TODO: or just put a resistor here\nor a proper poti for opening the filter.
 $Comp
 L Transistor_BJT:BC557 Q?
@@
 Text Notes 3625 1025 3    50   ~ 0
 set to ~~47k
-Text Notes -500 1450 0    50   ~ 0
-TODO: or just put a resistor here\nor a proper poti for opening the filter.
 Text GLabel 1175 800  0    50   Input ~ 0
 vca_ctl_raw
@@
 TODO: some input preattenuators for all control inputs
 Text Notes 450  -575 0    50   ~ 0
-TODO\n- input preattenuators\n- input pre-bias\n- expo for filter\n- what to do about the clamping?\n- connectors
+TODO\n- input preattenuators\n- expo for filter\n- what to do about the clamping?\n- connectors
+Text Notes 7350 1950 0    50   ~ 0
+or connect (-) with ~~100k to VEE\n(like the VCA)
+$Comp
+L Device:R_POT RV?
+U 1 1 5DCFDA87
+P 7500 1500
+F 0 "RV?" H 7625 1625 50  0000 C CNN
+F 1 "100k" V 7500 1500 50  0000 C CNN
+F 2 "" H 7500 1500 50  0001 C CNN
+F 3 "~" H 7500 1500 50  0001 C CNN
+	1    7500 1500
+	1    0    0    -1
+$EndComp
+$Comp
+L Device:R R?
+U 1 1 5DD3D8B2
+P 8000 1325
+F 0 "R?" V 7950 1425 50  0000 L CNN
+F 1 "47k" V 8000 1250 50  0000 L CNN
+F 2 "" V 7930 1325 50  0001 C CNN
+F 3 "~" H 8000 1325 50  0001 C CNN
+	1    8000 1325
+	0    -1   1    0
+$EndComp
+Connection ~ 8150 1325
+$Comp
+L power:VCC #PWR?
+U 1 1 5DD4583C
+P 7500 1350
+F 0 "#PWR?" H 7500 1200 50  0001 C CNN
+F 1 "VCC" H 7375 1425 50  0000 C CNN
+F 2 "" H 7500 1350 50  0001 C CNN
+F 3 "" H 7500 1350 50  0001 C CNN
+	1    7500 1350
+	1    0    0    -1
+$EndComp
+Wire Wire Line
+	7850 1325 7775 1325
+Wire Wire Line
+	7775 1325 7775 1500
+Wire Wire Line
+	7775 1500 7650 1500
 $EndSCHEMATC

Commit message: add input preattenuation
Parts:
- added R? (x4): 10k, symbol Device:R_POT
Connections:
- net GND: now also R?.3, R?.3, R?.3, R?.3
- net vca_ctl1: now also R?.2
- net vca_ctl2: now also R?.2
- net vcf_ctl1: now also R?.2
- net vcf_ctl2: now also R?.2
Other:
- note added: "TODO\n- expo for filter\n- what to do about the clamping?\n- connectors"
- note removed: "TODO: some input preattenuators for all control inputs"
- note removed: "TODO\n- input preattenuators\n- expo for filter\n- what to do about the clamping?\n- connectors"
Changed lines of the file:
@@
 	0    -1   1    0
 $EndComp
-Text GLabel 1050 1050 0    50   Input ~ 0
-vca_ctl2
 $Comp
 L Amplifier_Operational:TL074 U?
@@
 Wire Notes Line
 	6325 4650 6325 6150
-Text Notes 475  300  0    50   ~ 0
-TODO: some input preattenuators for all control inputs
 Text Notes 450  -575 0    50   ~ 0
-TODO\n- input preattenuators\n- expo for filter\n- what to do about the clamping?\n- connectors
+TODO\n- expo for filter\n- what to do about the clamping?\n- connectors
 Text Notes 7350 1950 0    50   ~ 0
 or connect (-) with ~~100k to VEE\n(like the VCA)
@@
 Wire Wire Line
 	7775 1500 7650 1500
+Text GLabel 5575 1775 2    50   Input ~ 0
+vcf_ctl2
+$Comp
+L Device:R_POT R?
+U 1 1 5DDA947B
+P 5575 1925
+F 0 "R?" V 5475 1950 50  0000 C CNN
+F 1 "10k" V 5575 1925 50  0000 C CNN
+F 2 "" H 5575 1925 50  0001 C CNN
+F 3 "~" H 5575 1925 50  0001 C CNN
+	1    5575 1925
+	0    -1   -1   0
+$EndComp
+$Comp
+L power:GND #PWR?
+U 1 1 5DDF0531
+P 5725 1925
+F 0 "#PWR?" H 5725 1675 50  0001 C CNN
+F 1 "GND" H 5730 1752 50  0001 C CNN
+F 2 "" H 5725 1925 50  0001 C CNN
+F 3 "" H 5725 1925 50  0001 C CNN
+	1    5725 1925
+	1    0    0    -1
+$EndComp
+Text GLabel 5575 1425 2    50   Input ~ 0
+vcf_ctl1
+$Comp
+L Device:R_POT R?
+U 1 1 5DDF0D1B
+P 5575 1575
+F 0 "R?" V 5475 1600 50  0000 C CNN
+F 1 "10k" V 5575 1575 50  0000 C CNN
+F 2 "" H 5575 1575 50  0001 C CNN
+F 3 "~" H 5575 1575 50  0001 C CNN
+	1    5575 1575
+	0    -1   -1   0
+$EndComp
+$Comp
+L power:GND #PWR?
+U 1 1 5DDF0D25
+P 5725 1575
+F 0 "#PWR?" H 5725 1325 50  0001 C CNN
+F 1 "GND" H 5730 1402 50  0001 C CNN
+F 2 "" H 5725 1575 50  0001 C CNN
+F 3 "" H 5725 1575 50  0001 C CNN
+	1    5725 1575
+	1    0    0    -1
+$EndComp
+Text GLabel 5575 1075 2    50   Input ~ 0
+vca_ctl2
+$Comp
+L Device:R_POT R?
+U 1 1 5DE0C3D1
+P 5575 1225
+F 0 "R?" V 5475 1250 50  0000 C CNN
+F 1 "10k" V 5575 1225 50  0000 C CNN
+F 2 "" H 5575 1225 50  0001 C CNN
+F 3 "~" H 5575 1225 50  0001 C CNN
+	1    5575 1225
+	0    -1   -1   0
+$EndComp
+$Comp
+L power:GND #PWR?
+U 1 1 5DE0C3D7
+P 5725 1225
+F 0 "#PWR?" H 5725 975 50  0001 C CNN
+F 1 "GND" H 5730 1052 50  0001 C CNN
+F 2 "" H 5725 1225 50  0001 C CNN
+F 3 "" H 5725 1225 50  0001 C CNN
+	1    5725 1225
+	1    0    0    -1
+$EndComp
+Text GLabel 5575 725  2    50   Input ~ 0
+vca_ctl1
+$Comp
+L Device:R_POT R?
+U 1 1 5DE0C3DE
+P 5575 875
+F 0 "R?" V 5475 900 50  0000 C CNN
+F 1 "10k" V 5575 875 50  0000 C CNN
+F 2 "" H 5575 875 50  0001 C CNN
+F 3 "~" H 5575 875 50  0001 C CNN
+	1    5575 875
+	0    -1   -1   0
+$EndComp
+$Comp
+L power:GND #PWR?
+U 1 1 5DE0C3E4
+P 5725 875
+F 0 "#PWR?" H 5725 625 50  0001 C CNN
+F 1 "GND" H 5730 702 50  0001 C CNN
+F 2 "" H 5725 875 50  0001 C CNN
+F 3 "" H 5725 875 50  0001 C CNN
+	1    5725 875
+	1    0    0    -1
+$EndComp
+Text GLabel 1050 1050 0    50   Input ~ 0
+vca_ctl2
 $EndSCHEMATC

Commit message: put measurement clamping circuitry on the voice board
Parts:
- removed C?: 1n, symbol Device:C
- removed J?: Conn_02x03_Odd_Even, symbol Connector_Generic:Conn_02x03_Odd_Even
- removed JP?: Jumper_2_Bridged, symbol Jumper:Jumper_2_Bridged
- removed Q?: BC547, Package_TO_SOT_THT:TO-92_Inline, symbol Transistor_BJT:BC547
- removed Q?: 2N7000, Package_TO_SOT_THT:TO-92_Inline, symbol Transistor_FET:2N7000
- removed R? (x2): 1k, symbol Device:R
- removed R?: 10k, symbol Device:R
- added C?: 1n, symbol Device:C
- added D? (x2): 3V3, symbol Device:D_Zener
- added D? (x2): 1N5817, Diode_THT:D_DO-41_SOD81_P10.16mm_Horizontal, symbol Diode:1N5817
- added J?: Conn_02x06_Odd_Even, symbol Connector_Generic:Conn_02x06_Odd_Even
- added JP?: Jumper_2_Bridged, symbol Jumper:Jumper_2_Bridged
- added Q?: BC547, Package_TO_SOT_THT:TO-92_Inline, symbol Transistor_BJT:BC547
- added Q?: 2N7000, Package_TO_SOT_THT:TO-92_Inline, symbol Transistor_FET:2N7000
- added R? (x3): 10k, symbol Device:R
- added R? (x2): 1k, symbol Device:R
Connections:
- net GND: now also D?.2 (A), D?.2 (A), D?.2 (A), D?.2 (A)
- net VCC: now also Q?.1 (C)
- net VEE: now also Q?.1 (S), R?.1, R?.1
- net square_ctl1: now also J?.1 (Pin_1)
- net square_ctl2: now also J?.2 (Pin_2), R?.2
- net square_ctl_buf1: now also J?.3 (Pin_3), J?.5 (Pin_5), J?.7 (Pin_7), R?.2
- net square_ctl_buf2: now also J?.4 (Pin_4), J?.6 (Pin_6), J?.8 (Pin_8), JP?.1 (A), Q?.3 (E), R?.2, R?.2
- net sync_out1: now also J?.11 (Pin_11)
- net sync_out2: now also J?.12 (Pin_12), Q?.3 (D)
- new net: Q?.2 (B), R?.1
- new net: C?.2, JP?.2 (B)
- new net: C?.1, Q?.2 (G), R?.2
- new net clamped1: D?.1 (K), D?.1 (K), J?.9 (Pin_9), R?.1
- new net clamped2: D?.1 (K), D?.1 (K), J?.10 (Pin_10), R?.1
Other:
- note added: "TODO\n- expo for filter\n- connectors"
- note added: "clamp\nfor the\nSTM32\nmeasure-\nment pin"
- note added: "square_ctl swings between Vee and Vcc - 1.5V (circa).\nGNDREF is at (Vcc+Vee)/2, i.e. PE7 sees at least 3V for\nVcc-Vee = 9V.\nThe diodes protect the MCU pin from overvoltage (D1)\nand undervoltage (D2): The schottky diode D2 clamps\naway negative voltages (to approx. -200mV), while the\nzener diode D1 limits the voltage to 3.3V. That's within\nthe MCU specs."
- note removed: "TODO: expo converter for the VCF input"
- note removed: "TODO: more square_ctl_buf outputs.\nor add the clamping circuitry here"
- note removed: "TODO: vca_ctl and vcf_ctl connectors,\n mixer, vca, vcf inputs and outputs"
- note removed: "TODO\n- expo for filter\n- what to do about the clamping?\n- connectors"
- moved on the sheet: C?, JP?, Q?, R?

Commit message: rename RV->R
Parts:
- gave numbers to parts that had none: 1
Changed lines of the file:
@@
 $EndComp
 $Comp
-L Device:R_POT RV?
+L Device:R_POT R?
 U 1 1 5DC6E5D7
 P 2875 6650
-F 0 "RV?" H 2805 6696 50  0000 R CNN
+F 0 "R?" H 2805 6696 50  0000 R CNN
 F 1 "1k" V 2875 6700 50  0000 R CNN
 F 2 "" H 2875 6650 50  0001 C CNN
@@
 LFO
 $Comp
-L Device:R_POT RV?
+L Device:R_POT R?
 U 1 1 5DC95C10
 P 2125 7350
-F 0 "RV?" H 2055 7396 50  0000 R CNN
+F 0 "R?" H 2055 7396 50  0000 R CNN
 F 1 "1k" V 2125 7400 50  0000 R CNN
 F 2 "" H 2125 7350 50  0001 C CNN
@@
 vco1_in
 $Comp
-L Device:R_POT RV?
+L Device:R_POT R?
 U 1 1 5DEF116D
 P 5350 2825
-F 0 "RV?" V 5235 2825 50  0000 C CNN
+F 0 "R?" V 5235 2825 50  0000 C CNN
 F 1 "10k" V 5350 2825 50  0000 C CNN
 F 2 "" H 5350 2825 50  0001 C CNN
@@
 vco2_in
 $Comp
-L Device:R_POT RV?
+L Device:R_POT R?
 U 1 1 5DEFFDC3
 P 5350 3525
-F 0 "RV?" V 5235 3525 50  0000 C CNN
+F 0 "R?" V 5235 3525 50  0000 C CNN
 F 1 "10k" V 5350 3525 50  0000 C CNN
 F 2 "" H 5350 3525 50  0001 C CNN
@@
 	5800 6900 5800 7275
 $Comp
-L Device:R_POT RV?
+L Device:R_POT R?
 U 1 1 5E12A7CE
 P 6100 7350
-F 0 "RV?" H 6031 7396 50  0000 R CNN
+F 0 "R?" H 6031 7396 50  0000 R CNN
 F 1 "1k" V 6100 7400 50  0000 R CNN
 F 2 "" H 6100 7350 50  0001 C CNN
@@
 $EndComp
 $Comp
-L Device:R_POT RV?
+L Device:R_POT R?
 U 1 1 5E1317B6
 P 6375 7050
-F 0 "RV?" H 6306 7096 50  0000 R CNN
+F 0 "R?" H 6306 7096 50  0000 R CNN
 F 1 "1k" V 6375 7100 50  0000 R CNN
 F 2 "" H 6375 7050 50  0001 C CNN
@@
 or connect (-) with ~~100k to VEE\n(like the VCA)
 $Comp
-L Device:R_POT RV?
+L Device:R_POT R?
 U 1 1 5DCFDA87
 P 7500 1500
-F 0 "RV?" H 7625 1625 50  0000 C CNN
+F 0 "R?" H 7625 1625 50  0000 C CNN
 F 1 "100k" V 7500 1500 50  0000 C CNN
 F 2 "" H 7500 1500 50  0001 C CNN
