File: hardware/voice_board/voice_board.sch (KiCad schematic (older format))
At the start: 131 parts, among them J1 Conn_02x06_Odd_Even, J10 Conn_01x02_Male, J2 Conn_02x02_Odd_Even, J3 Conn_02x02_Odd_Even, J4 Conn_01x02_Male, J5 Conn_02x03_Odd_Even, J6 Conn_02x02_Odd_Even, J7 Conn_02x02_Odd_Even, J8 Conn_02x02_Odd_Even, J9 Conn_02x02_Odd_Even, Q1 BC327, Q10 BC557, Q11 BC557, Q12 BC557, Q13 BC557, Q14 BC557, Q15 BC557, Q16 BC557, Q17 BC547, Q18 BC547, Q19 2N7000, Q2 BC557, Q20 2N7000, Q21 BC547, Q22 BC547, Q3 BC327, Q4 BC557, Q5 BC557, Q6 BC557, Q7 BC557, Q8 BC557, Q9 BC557, U1 TL074, U2 MCP4822, U3 LM324

Commit message: use film caps for the filter
Parts:
- C3, C4, C5, C6: footprint Capacitor_SMD:C_0805_2012Metric_Pad1.15x1.40mm_HandSolder -> footprints:C_rect_smd_combo
Changed lines of the file:
@@
 F 0 "C3" V 8875 2800 50  0000 C CNN
 F 1 "47n" V 8950 2825 50  0000 C CNN
-F 2 "Capacitor_SMD:C_0805_2012Metric_Pad1.15x1.40mm_HandSolder" H 8963 2425 50  0001 C CNN
+F 2 "footprints:C_rect_smd_combo" H 8963 2425 50  0001 C CNN
 F 3 "~" H 8925 2575 50  0001 C CNN
 	1    8925 2575
@@
 F 0 "C4" V 8875 3425 50  0000 C CNN
 F 1 "47n" V 8950 3450 50  0000 C CNN
-F 2 "Capacitor_SMD:C_0805_2012Metric_Pad1.15x1.40mm_HandSolder" H 8963 3050 50  0001 C CNN
+F 2 "footprints:C_rect_smd_combo" H 8963 3050 50  0001 C CNN
 F 3 "~" H 8925 3200 50  0001 C CNN
 	1    8925 3200
@@
 F 0 "C5" V 8875 4050 50  0000 C CNN
 F 1 "47n" V 8950 4075 50  0000 C CNN
-F 2 "Capacitor_SMD:C_0805_2012Metric_Pad1.15x1.40mm_HandSolder" H 8963 3675 50  0001 C CNN
+F 2 "footprints:C_rect_smd_combo" H 8963 3675 50  0001 C CNN
 F 3 "~" H 8925 3825 50  0001 C CNN
 	1    8925 3825
@@
 F 0 "C6" V 8875 4350 50  0000 C CNN
 F 1 "47n" V 8975 4325 50  0000 C CNN
-F 2 "Capacitor_SMD:C_0805_2012Metric_Pad1.15x1.40mm_HandSolder" H 8963 4425 50  0001 C CNN
+F 2 "footprints:C_rect_smd_combo" H 8963 4425 50  0001 C CNN
 F 3 "~" H 8925 4575 50  0001 C CNN
 	1    8925 4575

Commit message: final version of voice board mk I
Parts:
- removed C12: 100n, Capacitor_SMD:C_0805_2012Metric_Pad1.15x1.40mm_HandSolder, symbol Device:C
- removed R52, R55: 1k, Potentiometer_THT:Potentiometer_Runtron_RM-065_Vertical, symbol Device:R_POT
- removed R56: 10k, Resistor_SMD:R_0805_2012Metric_Pad1.15x1.40mm_HandSolder, symbol Device:R
Other:
- note removed: "Low-pass filter for fast\nattacking envelopes.\nTime constant T =\n10kOhm * 100nF = \n1ms. This removes\npops, but is still ballsy."
- note removed: "TODO\n- some potis\n- prototyping area"
Changed lines of the file:
@@
 Comment4 ""
 $EndDescr
-Text GLabel 2500 -1050 0    50   Input ~ 0
-Envelope
 Connection ~ 2350 1550
 $Comp
@@
 	1    0    0    -1
 $EndComp
-$Comp
-L Device:R_POT R55
-U 1 1 5DC6E5D7
-P 2650 -900
-F 0 "R55" H 2580 -854 50  0000 R CNN
-F 1 "1k" V 2650 -850 50  0000 R CNN
-F 2 "Potentiometer_THT:Potentiometer_Runtron_RM-065_Vertical" H 2650 -900 50  0001 C CNN
-F 3 "~" H 2650 -900 50  0001 C CNN
-	1    2650 -900
-	1    0    0    -1
-$EndComp
-$Comp
-L power:GND #PWR045
-U 1 1 5DC78980
-P 2650 -750
-F 0 "#PWR045" H 2650 -1000 50  0001 C CNN
-F 1 "GND" H 2655 -923 50  0000 C CNN
-F 2 "" H 2650 -750 50  0001 C CNN
-F 3 "" H 2650 -750 50  0001 C CNN
-	1    2650 -750
-	1    0    0    -1
-$EndComp
-$Comp
-L Device:R R56
-U 1 1 5DC7A310
-P 2950 -900
-F 0 "R56" V 2850 -925 50  0000 L CNN
-F 1 "10k" V 2950 -975 50  0000 L CNN
-F 2 "Resistor_SMD:R_0805_2012Metric_Pad1.15x1.40mm_HandSolder" V 2880 -900 50  0001 C CNN
-F 3 "~" H 2950 -900 50  0001 C CNN
-	1    2950 -900
-	0    -1   1    0
-$EndComp
-$Comp
-L Device:C C12
-U 1 1 5DC7AF18
-P 3100 -750
-F 0 "C12" H 3215 -704 50  0000 L CNN
-F 1 "100n" H 3215 -795 50  0000 L CNN
-F 2 "Capacitor_SMD:C_0805_2012Metric_Pad1.15x1.40mm_HandSolder" H 3138 -900 50  0001 C CNN
-F 3 "~" H 3100 -750 50  0001 C CNN
-	1    3100 -750
-	1    0    0    -1
-$EndComp
-$Comp
-L power:GND #PWR046
-U 1 1 5DC7B326
-P 3100 -600
-F 0 "#PWR046" H 3100 -850 50  0001 C CNN
-F 1 "GND" H 3105 -773 50  0000 C CNN
-F 2 "" H 3100 -600 50  0001 C CNN
-F 3 "" H 3100 -600 50  0001 C CNN
-	1    3100 -600
-	1    0    0    -1
-$EndComp
-Text Notes 2450 125  0    50   ~ 0
-Low-pass filter for fast\nattacking envelopes.\nTime constant T =\n10kOhm * 100nF = \n1ms. This removes\npops, but is still ballsy.
-Wire Wire Line
-	2500 -1050 2650 -1050
-Text GLabel 1450 -425 0    50   Input ~ 0
-LFO
-$Comp
-L Device:R_POT R52
-U 1 1 5DC95C10
-P 1550 -275
-F 0 "R52" H 1480 -229 50  0000 R CNN
-F 1 "1k" V 1550 -225 50  0000 R CNN
-F 2 "Potentiometer_THT:Potentiometer_Runtron_RM-065_Vertical" H 1550 -275 50  0001 C CNN
-F 3 "~" H 1550 -275 50  0001 C CNN
-	1    1550 -275
-	1    0    0    -1
-$EndComp
-Wire Wire Line
-	1550 -425 1450 -425
-$Comp
-L power:GND #PWR041
-U 1 1 5DC985D7
-P 1550 -125
-F 0 "#PWR041" H 1550 -375 50  0001 C CNN
-F 1 "GND" H 1555 -298 50  0000 C CNN
-F 2 "" H 1550 -125 50  0001 C CNN
-F 3 "" H 1550 -125 50  0001 C CNN
-	1    1550 -125
-	1    0    0    -1
-$EndComp
-Text GLabel 1700 -275 2    50   Input ~ 0
-PWM
 Text GLabel 3775 5050 2    50   Input ~ 0
 VCA_ctl
-Wire Wire Line
-	3200 -900 3100 -900
-Connection ~ 3100 -900
 Wire Wire Line
 	1725 1775 1425 1775
@@
 Wire Notes Line
 	4900 6275 4900 7775
-Text Notes 1275 -875 0    50   ~ 0
-TODO\n- some potis\n- prototyping area
 Text Notes 7400 1700 0    50   ~ 0
 or connect (-) with ~~100k to VEE\n(like the VCA)

Commit message: voice board: towards production
Other:
- note removed: "TODO: support film caps"
Changed lines of the file:
@@
 U 1 1 5DDF220D
 P 8325 2325
-F 0 "R27" V 8325 2050 50  0000 L CNN
+F 0 "R27" V 8325 2025 50  0000 L CNN
 F 1 "470" V 8325 2250 50  0000 L CNN
 F 2 "Resistor_SMD:R_0805_2012Metric_Pad1.15x1.40mm_HandSolder" V 8255 2325 50  0001 C CNN
@@
 Text Notes 6500 5775 0    50   ~ 0
 TODO: keep or remove ground connection
-Text Notes 9025 875  0    50   ~ 0
-TODO: support film caps
 $Comp
 L Device:R R15

Commit message: Fix swapped resistors in voice board's sync circuit
Fixes #18
Parts:
- R48, R49: value 10k -> 1k
- R50, R51: value 1k -> 10k
Changed lines of the file:
@@
 EESchema Schematic File Version 4
-LIBS:voice_board-cache
 EELAYER 30 0
 EELAYER END
@@
 encoding utf-8
 Sheet 1 1
-Title ""
+Title "voice board"
 Date ""
-Rev ""
-Comp ""
+Rev "02"
+Comp "Windfisch"
 Comment1 ""
 Comment2 ""
@@
 	1    0    0    -1
 $EndComp
-Text GLabel 3775 5050 2    50   Input ~ 0
-VCA_ctl
 Wire Wire Line
 	1725 1775 1425 1775
@@
 P 3100 3700
 F 0 "R50" H 2975 3750 50  0000 C CNN
-F 1 "1k" V 3100 3700 50  0000 C CNN
+F 1 "10k" V 3100 3700 50  0000 C CNN
 F 2 "Resistor_SMD:R_0805_2012Metric_Pad1.15x1.40mm_HandSolder" V 3030 3700 50  0001 C CNN
 F 3 "~" H 3100 3700 50  0001 C CNN
@@
 P 2300 3700
 F 0 "R48" H 2400 3600 50  0000 C CNN
-F 1 "10k" V 2300 3700 50  0000 C CNN
+F 1 "1k" V 2300 3700 50  0000 C CNN
 F 2 "Resistor_SMD:R_0805_2012Metric_Pad1.15x1.40mm_HandSolder" V 2230 3700 50  0001 C CNN
 F 3 "~" H 2300 3700 50  0001 C CNN
@@
 P 3100 4850
 F 0 "R51" H 2975 4900 50  0000 C CNN
-F 1 "1k" V 3100 4850 50  0000 C CNN
+F 1 "10k" V 3100 4850 50  0000 C CNN
 F 2 "Resistor_SMD:R_0805_2012Metric_Pad1.15x1.40mm_HandSolder" V 3030 4850 50  0001 C CNN
 F 3 "~" H 3100 4850 50  0001 C CNN
@@
 P 2300 4850
 F 0 "R49" H 2400 4750 50  0000 C CNN
-F 1 "10k" V 2300 4850 50  0000 C CNN
+F 1 "1k" V 2300 4850 50  0000 C CNN
 F 2 "Resistor_SMD:R_0805_2012Metric_Pad1.15x1.40mm_HandSolder" V 2230 4850 50  0001 C CNN
 F 3 "~" H 2300 4850 50  0001 C CNN

Commit message: voice board: remove DAC potis, tie down dangling op amp
Parts:
- removed R53, R54: 1k, Potentiometer_THT:Potentiometer_Runtron_RM-065_Vertical, symbol Device:R_POT
- added unit 4 of U3
Connections:
- net GND: now also U3.12 (+)
- net at C10.1, U2.6 (VB): now also J4.2 (Pin_2)
- net at C11.1, U2.8 (VA): now also J4.1 (Pin_1)
- new net: U3.13 (-), U3.14
Other:
- note removed: "TODO: keep or remove ground connection"
- moved on the sheet: J4
Changed lines of the file:
@@
 Wire Wire Line
 	5900 5225 5900 5600
-$Comp
-L Device:R_POT R53
-U 1 1 5E12A7CE
-P 6200 5675
-F 0 "R53" H 6150 5750 50  0000 R CNN
-F 1 "1k" V 6200 5725 50  0000 R CNN
-F 2 "Potentiometer_THT:Potentiometer_Runtron_RM-065_Vertical" H 6200 5675 50  0001 C CNN
-F 3 "~" H 6200 5675 50  0001 C CNN
-	1    6200 5675
-	1    0    0    -1
-$EndComp
-$Comp
-L Device:R_POT R54
-U 1 1 5E1317B6
-P 6475 5375
-F 0 "R54" H 6425 5450 50  0000 R CNN
-F 1 "1k" V 6475 5425 50  0000 R CNN
-F 2 "Potentiometer_THT:Potentiometer_Runtron_RM-065_Vertical" H 6475 5375 50  0001 C CNN
-F 3 "~" H 6475 5375 50  0001 C CNN
-	1    6475 5375
-	1    0    0    -1
-$EndComp
-Wire Wire Line
-	5675 5525 6200 5525
 Connection ~ 5675 5525
-Wire Wire Line
-	5900 5225 6475 5225
 Connection ~ 5900 5225
-Wire Wire Line
-	6475 5525 6475 5825
-$Comp
-L power:GND #PWR043
-U 1 1 5E14B5EA
-P 6200 5825
-F 0 "#PWR043" H 6200 5575 50  0001 C CNN
-F 1 "GND" H 6205 5652 50  0000 C CNN
-F 2 "" H 6200 5825 50  0001 C CNN
-F 3 "" H 6200 5825 50  0001 C CNN
-	1    6200 5825
-	1    0    0    -1
-$EndComp
-$Comp
-L power:GND #PWR044
-U 1 1 5E14B87F
-P 6475 5825
-F 0 "#PWR044" H 6475 5575 50  0001 C CNN
-F 1 "GND" H 6480 5652 50  0000 C CNN
-F 2 "" H 6475 5825 50  0001 C CNN
-F 3 "" H 6475 5825 50  0001 C CNN
-	1    6475 5825
-	1    0    0    -1
-$EndComp
-Wire Wire Line
-	6625 5375 6725 5375
-Wire Wire Line
-	6825 5675 6825 5375
-Wire Wire Line
-	6350 5675 6825 5675
 $Comp
 L Connector_Generic:Conn_02x02_Odd_Even J2
@@
 L Connector:Conn_01x02_Male J4
 U 1 1 5E1550B9
-P 6725 5175
-F 0 "J4" V 6625 5175 50  0000 R CNN
-F 1 "Conn_01x02_Male" V 6878 5219 50  0001 L CNN
-F 2 "Connector_PinHeader_2.54mm:PinHeader_1x02_P2.54mm_Vertical" H 6725 5175 50  0001 C CNN
-F 3 "~" H 6725 5175 50  0001 C CNN
-	1    6725 5175
+P 6725 5025
+F 0 "J4" V 6625 5025 50  0000 R CNN
+F 1 "Conn_01x02_Male" V 6878 5069 50  0001 L CNN
+F 2 "Connector_PinHeader_2.54mm:PinHeader_1x02_P2.54mm_Vertical" H 6725 5025 50  0001 C CNN
+F 3 "~" H 6725 5025 50  0001 C CNN
+	1    6725 5025
 	0    -1   1    0
 $EndComp
@@
 	0    1    1    0
 $EndComp
-Text Notes 6500 5775 0    50   ~ 0
-TODO: keep or remove ground connection
 $Comp
 L Device:R R15
@@
 	-1   0    0    -1
 $EndComp
+$Comp
+L Amplifier_Operational:LM324 U3
+U 4 1 600A4073
+P 7475 6175
+F 0 "U3" H 7550 6350 50  0000 C CNN
+F 1 "LM324" H 7450 6175 50  0000 C CNN
+F 2 "Package_DIP:DIP-14_W7.62mm" H 7425 6275 50  0001 C CNN
+F 3 "http://www.ti.com/lit/ds/symlink/lm2902-n.pdf" H 7525 6375 50  0001 C CNN
+	4    7475 6175
+	1    0    0    1
+$EndComp
+$Comp
+L power:GND #PWR?
+U 1 1 600A9C22
+P 7175 6275
+F 0 "#PWR?" H 7175 6025 50  0001 C CNN
+F 1 "GND" H 7180 6102 50  0000 C CNN
+F 2 "" H 7175 6275 50  0001 C CNN
+F 3 "" H 7175 6275 50  0001 C CNN
+	1    7175 6275
+	1    0    0    -1
+$EndComp
+Wire Wire Line
+	7175 6075 7150 6075
+Wire Wire Line
+	7150 6075 7150 5900
+Wire Wire Line
+	7150 5900 7825 5900
+Wire Wire Line
+	7825 5900 7825 6175
+Wire Wire Line
+	7825 6175 7775 6175
+Wire Wire Line
+	5675 5525 6825 5525
+Wire Wire Line
+	5900 5225 6725 5225
+Wire Wire Line
+	6825 5225 6825 5525
 $EndSCHEMATC

Commit message: updated resistor values to match current situation
Parts:
- R12, R13: value 20k -> 22k
- R36, R37: value 10k -> 1k
- R42, R43: value 1Meg -> 100k
- R68: value 2.5k -> 2.4k
Changed lines of the file:
@@
 P 2950 2225
 F 0 "R13" V 2850 2200 50  0000 L CNN
-F 1 "20k" V 2950 2150 50  0000 L CNN
+F 1 "22k" V 2950 2150 50  0000 L CNN
 F 2 "Resistor_SMD:R_0805_2012Metric_Pad1.15x1.40mm_HandSolder" V 2880 2225 50  0001 C CNN
 F 3 "~" H 2950 2225 50  0001 C CNN
@@
 P 2950 2025
 F 0 "R12" V 3050 2000 50  0000 L CNN
-F 1 "20k" V 2950 1950 50  0000 L CNN
+F 1 "22k" V 2950 1950 50  0000 L CNN
 F 2 "Resistor_SMD:R_0805_2012Metric_Pad1.15x1.40mm_HandSolder" V 2880 2025 50  0001 C CNN
 F 3 "~" H 2950 2025 50  0001 C CNN
@@
 P 9675 4575
 F 0 "R37" V 9575 4550 50  0000 L CNN
-F 1 "10k" V 9675 4500 50  0000 L CNN
+F 1 "1k" V 9675 4525 50  0000 L CNN
 F 2 "Resistor_SMD:R_0805_2012Metric_Pad1.15x1.40mm_HandSolder" V 9605 4575 50  0001 C CNN
 F 3 "~" H 9675 4575 50  0001 C CNN
@@
 P 9675 4375
 F 0 "R36" V 9775 4350 50  0000 L CNN
-F 1 "10k" V 9675 4300 50  0000 L CNN
+F 1 "1k" V 9675 4325 50  0000 L CNN
 F 2 "Resistor_SMD:R_0805_2012Metric_Pad1.15x1.40mm_HandSolder" V 9605 4375 50  0001 C CNN
 F 3 "~" H 9675 4375 50  0001 C CNN
@@
 P 10250 4150
 F 0 "R43" V 10350 4075 50  0000 L CNN
-F 1 "1Meg" V 10250 4050 50  0000 L CNN
+F 1 "100k" V 10250 4050 50  0000 L CNN
 F 2 "Resistor_SMD:R_0805_2012Metric_Pad1.15x1.40mm_HandSolder" V 10180 4150 50  0001 C CNN
 F 3 "~" H 10250 4150 50  0001 C CNN
@@
 P 9900 4825
 F 0 "R42" H 9975 4800 50  0000 L CNN
-F 1 "1Meg" V 9900 4725 50  0000 L CNN
+F 1 "100k" V 9900 4725 50  0000 L CNN
 F 2 "Resistor_SMD:R_0805_2012Metric_Pad1.15x1.40mm_HandSolder" V 9830 4825 50  0001 C CNN
 F 3 "~" H 9900 4825 50  0001 C CNN
@@
 P 1575 6500
 F 0 "R68" V 1525 6600 50  0000 L CNN
-F 1 "2.5k" V 1575 6425 50  0000 L CNN
+F 1 "2.4k" V 1575 6425 50  0000 L CNN
 F 2 "Resistor_SMD:R_0805_2012Metric_Pad1.15x1.40mm_HandSolder" V 1505 6500 50  0001 C CNN
 F 3 "~" H 1575 6500 50  0001 C CNN

Commit message: add capacitors in an attempt to fix the buzzing
Parts:
- added C? (x3): 4.7n, symbol Device:C_Small
- added C?: C_Small, symbol Device:C_Small
- added C?: 27p, symbol Device:C_Small
Connections:
- net GND: now also C?.2, C?.2, C?.2
- net vcf_audio_out: now also C?.1
- net at C2.1, Q5.2 (B), R27.1: now also C?.1
- net at C7.2, Q11.2 (B), R35.2: now also C?.1
- net at R37.1, R42.1, U1.12 (+): now also C?.1
- net at R36.1, R43.2, U1.13 (-): now also C?.2, C?.2
- net at Q11.3 (E), Q5.3 (E), R34.1: now also C?.1
Changed lines of the file:
@@
 	8475 3075 8475 2850
-Wire Wire Line
-	9375 2325 9375 2225
 Wire Wire Line
 	8475 2325 8475 2225
@@
 $EndComp
 $Comp
-L Transistor_BJT:BC557 Q11
-U 1 1 5E3B0CD3
-P 9175 2225
-F 0 "Q11" H 9000 2350 50  0000 L CNN
-F 1 "BC557" H 9366 2180 50  0001 L CNN
-F 2 "Package_TO_SOT_THT:TO-92_Inline" H 9375 2150 50  0001 L CIN
-F 3 "http://www.fairchildsemi.com/ds/BC/BC557.pdf" H 9175 2225 50  0001 L CNN
-	1    9175 2225
-	-1   0    0    1
-$EndComp
-$Comp
 L Transistor_BJT:BC557 Q10
 U 1 1 5E3BC860
@@
 Wire Wire Line
 	8475 4825 8475 4725
-Connection ~ 9375 2225
-Wire Wire Line
-	9375 2225 9375 2125
 $Comp
 L Device:R_Variable R40
@@
 U 1 1 5DF2729E
 P 10250 4150
-F 0 "R43" V 10350 4075 50  0000 L CNN
+F 0 "R43" V 10150 4075 50  0000 L CNN
 F 1 "100k" V 10250 4050 50  0000 L CNN
 F 2 "Resistor_SMD:R_0805_2012Metric_Pad1.15x1.40mm_HandSolder" V 10180 4150 50  0001 C CNN
@@
 	9375 4375 9525 4375
 Wire Wire Line
-	10575 4150 10575 3825
+	10575 4150 10575 4050
 Wire Wire Line
 	10575 3825 9900 3825
@@
 Wire Wire Line
 	6825 5225 6825 5525
+$Comp
+L Device:C_Small C?
+U 1 1 601F797F
+P 9275 1975
+F 0 "C?" H 9367 2021 50  0001 L CNN
+F 1 "4.7n" V 9375 1900 50  0000 L CNN
+F 2 "" H 9275 1975 50  0001 C CNN
+F 3 "~" H 9275 1975 50  0001 C CNN
+	1    9275 1975
+	0    1    1    0
+$EndComp
+Wire Wire Line
+	9375 2225 9375 2125
+Wire Wire Line
+	9375 2325 9375 2225
+Connection ~ 9375 2225
+$Comp
+L Transistor_BJT:BC557 Q11
+U 1 1 5E3B0CD3
+P 9175 2225
+F 0 "Q11" H 9000 2350 50  0000 L CNN
+F 1 "BC557" H 9366 2180 50  0001 L CNN
+F 2 "Package_TO_SOT_THT:TO-92_Inline" H 9375 2150 50  0001 L CIN
+F 3 "http://www.fairchildsemi.com/ds/BC/BC557.pdf" H 9175 2225 50  0001 L CNN
+	1    9175 2225
+	-1   0    0    1
+$EndComp
+Wire Wire Line
+	9375 1975 9375 2125
+Connection ~ 9375 2125
+$Comp
+L power:GND #PWR?
+U 1 1 6022405F
+P 9175 1975
+F 0 "#PWR?" H 9175 1725 50  0001 C CNN
+F 1 "GND" H 9180 1802 50  0001 C CNN
+F 2 "" H 9175 1975 50  0001 C CNN
+F 3 "" H 9175 1975 50  0001 C CNN
+	1    9175 1975
+	-1   0    0    -1
+$EndComp
+$Comp
+L Device:C_Small C?
+U 1 1 60224C0A
+P 8675 1975
+F 0 "C?" H 8767 2021 50  0001 L CNN
+F 1 "4.7n" V 8575 1850 50  0000 L CNN
+F 2 "" H 8675 1975 50  0001 C CNN
+F 3 "~" H 8675 1975 50  0001 C CNN
+	1    8675 1975
+	0    1    1    0
+$EndComp
+Wire Wire Line
+	8775 2025 8775 1975
+Connection ~ 8775 2025
+$Comp
+L power:GND #PWR?
+U 1 1 60236998
+P 8575 1975
+F 0 "#PWR?" H 8575 1725 50  0001 C CNN
+F 1 "GND" H 8580 1802 50  0001 C CNN
+F 2 "" H 8575 1975 50  0001 C CNN
+F 3 "" H 8575 1975 50  0001 C CNN
+	1    8575 1975
+	-1   0    0    -1
+$EndComp
+$Comp
+L Device:C_Small C?
+U 1 1 6023C519
+P 8475 2025
+F 0 "C?" H 8567 2071 50  0001 L CNN
+F 1 "4.7n" H 8500 1950 50  0001 L CNN
+F 2 "" H 8475 2025 50  0001 C CNN
+F 3 "~" H 8475 2025 50  0001 C CNN
+	1    8475 2025
+	-1   0    0    1
+$EndComp
+Connection ~ 8475 2125
+Wire Wire Line
+	8575 1975 8575 1925
+Wire Wire Line
+	8575 1925 8475 1925
+Connection ~ 8575 1975
+$Comp
+L Device:C_Small C?
+U 1 1 60250ED8
+P 10050 4050
+F 0 "C?" V 9925 4050 50  0001 C CNN
+F 1 "C_Small" V 10000 4250 50  0001 C CNN
+F 2 "" H 10050 4050 50  0001 C CNN
+F 3 "~" H 10050 4050 50  0001 C CNN
+	1    10050 4050
+	0    1    1    0
+$EndComp
+Wire Wire Line
+	9900 4150 9900 4050
+Wire Wire Line
+	9900 4050 9950 4050
+Connection ~ 9900 4150
+Wire Wire Line
+	10150 4050 10575 4050
+Connection ~ 10575 4050
+Wire Wire Line
+	10575 4050 10575 3825
+$Comp
+L Device:C_Small C?
+U 1 1 60295CCD
+P 9900 4475
+F 0 "C?" V 9775 4475 50  0001 C CNN
+F 1 "27p" H 10050 4475 50  0000 C CNN
+F 2 "" H 9900 4475 50  0001 C CNN
+F 3 "~" H 9900 4475 50  0001 C CNN
+	1    9900 4475
+	-1   0    0    1
+$EndComp
 $EndSCHEMATC

Commit message: voiceboard patch3; still wip
Parts:
- removed C? (x3): 4.7n, symbol Device:C_Small
- removed C?: C_Small, symbol Device:C_Small
- removed C?: 27p, symbol Device:C_Small
- added R? (x3): 1k, Resistor_SMD:R_0805_2012Metric_Pad1.15x1.40mm_HandSolder, symbol Device:R
- added R? (x3): 20k, Resistor_SMD:R_0805_2012Metric_Pad1.15x1.40mm_HandSolder, symbol Device:R
- added U? (x4): TL074, Package_DIP:DIP-14_W7.62mm, symbol Amplifier_Operational:TL074
- R36, R37: value 1k -> (none)
Connections:
- net GND: now also R?.2, U?.12 (+)
- net vcf_audio_out: now also R?.1, U?.14; no longer R43.1, U1.14
- net at C6.1, Q8.1 (C), Q9.3 (E): now also U?.12 (+); no longer R36.2
- net at C6.2, Q14.1 (C), Q15.3 (E): now also U?.12 (+); no longer R37.2
- net at R42.1, U1.12 (+): no longer R37.1
- net at R43.2, U1.13 (-): no longer R36.1
- new net: R43.1, U1.14
- new net: R?.2, U?.13 (-), U?.14 (x2)
- new net: R?.1, R?.1, U?.12 (+)
- new net: R?.1, R?.2, U?.13 (-) (x2)
- new net: R?.1, R?.2, U?.14
- no-connect marks 1 -> 6
Other:
- note added: "TODO: amplify at this point \nalready? (needs correct reference\nvoltage, i diode drop above Q9's base).\nOr capacitor?"
