File: hardware/voice_board/voice_board.kicad_pcb (KiCad board)
At the start: 2 copper layers, 114 parts, among them J1 Conn_02x06_Odd_Even, J2 Conn_02x02_Odd_Even, J3 Conn_02x02_Odd_Even, J4 Conn_01x02_Male, J5 Conn_02x03_Odd_Even, Q1 BC327, Q10 BC557, Q11 BC557, Q12 BC557, Q13 BC557, Q14 BC557, Q15 BC557, Q16 BC557, Q17 BC547, Q18 BC547, Q19 2N7000, Q2 BC557, Q20 2N7000, Q3 BC327, Q4 BC557, Q5 BC557, Q6 BC557, Q7 BC557, Q8 BC557, Q9 BC557, U1 TL074, U2 MCP4822

Commit message: voice board: vcf
Parts:
- Q10, Q11, Q12, Q13, Q14, Q15, Q16, Q5, Q6, Q7, Q8, Q9, R18, R19, R39, R40: moved to B.Cu
- R35: footprint Potentiometer_THT:Potentiometer_Runtron_RM-065_Vertical -> Resistor_SMD:R_0805_2012Metric_Pad1.15x1.40mm_HandSolder
- moved C7 205.4 mm to (240.3, 53.7), turned to 180 degrees
- moved Q14 184.6 mm to (233.8, 71.8), turned to 90 degrees
- moved Q12 183.3 mm to (233.8, 60.6), turned to 90 degrees
- moved Q15 182.0 mm to (233.8, 77.3), turned to 90 degrees
- moved Q9 180.3 mm to (229.0, 77.3), turned to 90 degrees
- moved C2 176.2 mm to (207.8, 28.7), turned to 180 degrees
- moved R40 172.8 mm to (242.7, 59.8), turned to 180 degrees
- moved Q8 170.3 mm to (229.0, 71.8), turned to 90 degrees
- moved R19 170.3 mm to (230.1, 31.8), turned to 180 degrees
- moved Q10 169.6 mm to (233.8, 49.4), turned to 90 degrees
- moved Q13 169.5 mm to (233.8, 66.2), turned to 90 degrees
- moved R18 166.6 mm to (237.4, 31.8), turned to 180 degrees
- moved Q11 166.1 mm to (233.8, 55.0), turned to 90 degrees
- moved C5 166.0 mm to (231.3, 67.7), turned to 180 degrees
- moved Q7 165.8 mm to (229.0, 66.2), turned to 90 degrees
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Routing:
- net VEE: track 4.83 -> 45.8 mm
- net Net-(R40-Pad2): track 0.00 -> 33.5 mm
- net Net-(Q10-Pad2): track 0.00 -> 21.5 mm
- net Net-(C6-Pad2): track 0.00 -> 20.4 mm
- net VCC: track 12.5 -> 30.2 mm
- net Net-(R37-Pad1): track 0.00 -> 16.1 mm
- net vcf_ctl_raw: track 0.00 -> 15.3 mm
- net vcf_ctl1: track 0.00 -> 12.9 mm
- net Net-(Q15-Pad2): track 0.00 -> 10.9 mm
- net Net-(Q13-Pad2): track 0.00 -> 10.5 mm
- net Net-(Q14-Pad2): track 0.00 -> 10.3 mm
- net GND: track 30.8 -> 40.9 mm
- net Net-(R36-Pad1): track 0.00 -> 9.53 mm
- net vcf_audio_out: track 0.00 -> 9.32 mm
- net (no net): track 8.28 -> 17.0 mm
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
Commit message: mixer and lowpass filters
Parts:
- added J6: Conn_02x02_Odd_Even, Connector_PinHeader_2.54mm:PinHeader_2x02_P2.54mm_Vertical, B.Cu at (41.1, 109.7)
- J5, R21, R57, R58, R59, R63, R64, R65: moved to B.Cu
- moved J5 203.9 mm to (82.0, 159.5), turned to 90 degrees
- moved R64 188.8 mm to (77.0, 167.6)
- moved C14 184.0 mm to (79.0, 166.6), turned to 90 degrees
- moved R65 177.8 mm to (84.1, 167.6)
- moved R63 175.1 mm to (69.8, 167.6)
- moved C15 168.4 mm to (71.9, 166.6), turned to 90 degrees
- moved C13 165.1 mm to (86.1, 166.6), turned to 90 degrees
- moved R58 155.7 mm to (53.8, 110.5)
- moved JP3 153.1 mm to (186.9, 41.1)
- moved R57 146.1 mm to (46.7, 110.5)
- moved J3 139.0 mm to (105.5, 110.0)
- moved R61 137.3 mm to (58.7, 105.2), turned to 90 degrees
- moved R21 128.2 mm to (199.6, 37.6)
- moved R62 127.1 mm to (65.8, 105.2), turned to 90 degrees
- moved R59 124.7 mm to (61.0, 110.5)
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Connections:
- R22 pad 1: (no net) -> GND
- R57 pad 1: (no net) -> vco1_in
- R58 pad 1: (no net) -> vco2_in
- R59 pad 1: (no net) -> vco3_in
Routing:
- net VCC: track 30.2 -> 62.7 mm
- net vco3_in: track 0.00 -> 32.0 mm
- net GND: track 40.9 -> 71.2 mm
- net Net-(C14-Pad1): track 0.00 -> 24.6 mm
- net mixer_out: track 0.00 -> 23.4 mm
- net vco2_in: track 0.00 -> 19.4 mm
- net Net-(C15-Pad1): track 0.00 -> 16.4 mm
- net Net-(C13-Pad1): track 0.00 -> 16.0 mm
- net vco1_in: track 0.00 -> 6.89 mm
- net Net-(J5-Pad5): track 0.00 -> 5.91 mm
- net Net-(J5-Pad1): track 0.00 -> 5.83 mm
- net Net-(J5-Pad3): track 0.00 -> 3.14 mm
- net Net-(R57-Pad2): track 0.00 -> 2.61 mm
- net Net-(R59-Pad2): track 0.00 -> 2.61 mm
- net Net-(R58-Pad2): track 0.00 -> 2.61 mm

Commit message: finished layout for all individual sections
Parts:
- added C16: 10n, Capacitor_SMD:C_0805_2012Metric_Pad1.15x1.40mm_HandSolder, F.Cu at (47.2, -20.6)
- added C17: 1u, Capacitor_SMD:C_0805_2012Metric_Pad1.15x1.40mm_HandSolder, F.Cu at (47.2, -24.6)
- D1, D2, D3, D4, J1, J2, J4, JP1, JP2, Q17, Q18, Q19, Q20, R53, R54, U2: moved to B.Cu
- moved D4 111.6 mm to (99.3, 50.5), turned to 180 degrees
- moved D1 103.6 mm to (108.2, 47.5)
- moved J1 98.7 mm to (105.2, 39.1), turned to 180 degrees
- moved D3 98.1 mm to (108.5, 50.5)
- moved R55 91.5 mm to (42.2, 65.0)
- moved D2 87.1 mm to (99.6, 47.5), turned to 180 degrees
- moved JP1 80.5 mm to (116.3, 39.9), turned to 270 degrees
- moved Q20 80.0 mm to (89.2, 45.7), turned to 90 degrees
- moved Q19 76.9 mm to (118.4, 45.7), turned to 90 degrees
- moved JP2 75.6 mm to (91.4, 39.9), turned to 90 degrees
- moved Q17 74.4 mm to (111.3, 39.6), turned to 270 degrees
- moved R45 71.6 mm to (99.6, 40.1), turned to 90 degrees
- moved R46 68.4 mm to (111.5, 47.0), turned to 180 degrees
- moved R49 63.6 mm to (98.8, 45.0), turned to 180 degrees
- moved C8 63.3 mm to (114.3, 42.9), turned to 180 degrees
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Routing:
- net VEE: track 45.8 -> 88.7 mm
- net GND: track 71.2 -> 111.2 mm
- net square_ctl_buf2: track 0.00 -> 22.4 mm
- net square_ctl_buf1: track 0.00 -> 22.4 mm
- net sync_out2: track 0.00 -> 21.8 mm
- net sync_out1: track 0.00 -> 21.0 mm
- net VCC: track 62.7 -> 79.8 mm
- net +3V3: track 0.00 -> 12.9 mm
- net clamped2: track 0.00 -> 9.10 mm
- net clamped1: track 0.00 -> 9.10 mm
- net PB15: track 0.00 -> 7.70 mm
- net Net-(C8-Pad2): track 0.00 -> 7.45 mm
- net Net-(C9-Pad2): track 0.00 -> 7.32 mm
- net Net-(C10-Pad1): track 0.00 -> 6.76 mm
- net Net-(C11-Pad1): track 0.00 -> 5.22 mm
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Other:
- board text added: "3x low pass filter"

Commit message: small todos
Parts:
- moved R56 10.2 mm to (93.0, -18.0)
Routing:
- net GND: track 111.2 -> 114.2 mm
- net (no net): track 17.5 -> 17.0 mm
Changed lines of the file:
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@@
     (thickness 1.6)
     (drawings 1)
-    (tracks 499)
+    (tracks 502)
     (zones 0)
     (modules 117)
@@
   )
   (module Resistor_SMD:R_0805_2012Metric_Pad1.15x1.40mm_HandSolder (layer F.Cu)
-    (at 101.4435 -12.4455)
+    (at 92.964 -18.034)
     (descr "Resistor SMD 0805 (2012 Metric), square (rectangular) end terminal, IPC_7351 nominal with elongated pad for handsoldering. (Body size source: https://docs.google.com/spreadsheets/d/1BsfQQcO9C6DZCsRaXUlFlo91Tg2WpOkGARC1WS5S8t0/edit?usp=sharing), generated with kicad-footprint-generator")
     (tags "resistor handsolder")
@@
   (segment (start 230.124 32.775) (end 230.199001 32.850001) (width 0.25) (layer F.Cu) (net 0))
   (segment (start 230.124 31.75) (end 230.124 32.775) (width 0.25) (layer F.Cu) (net 0))
-  (segment (start 224.282 48.514) (end 223.774 48.514) (width 0.25) (layer F.Cu) (net 0))
   (segment (start 196.106 61.468) (end 196.596 61.468) (width 0.25) (layer F.Cu) (net 1))
   (segment (start 194.056 63.518) (end 196.106 61.468) (width 0.25) (layer F.Cu) (net 1))
@@
   (segment (start 211.235001 44.691001) (end 212.01 45.466) (width 0.25) (layer F.Cu) (net 19))
   (segment (start 210.909999 44.365999) (end 211.235001 44.691001) (width 0.25) (layer F.Cu) (net 19))
-  (segment (start 205.744001 44.365999) (end 210.909999 44.365999) (width 0.25) (layer F.Cu) (net 19))
   (segment (start 204.644 45.466) (end 205.744001 44.365999) (width 0.25) (layer F.Cu) (net 19))
   (segment (start 214.5485 60.8785) (end 215.138 60.8785) (width 0.25) (layer F.Cu) (net 19))
@@
   (segment (start 115.824 47.752) (end 115.824 47.498) (width 0.25) (layer F.Cu) (net 19))
   (segment (start 118.618 50.546) (end 115.824 47.752) (width 0.25) (layer F.Cu) (net 19))
+  (segment (start 206.417999 42.179001) (end 206.417999 44.365999) (width 0.25) (layer F.Cu) (net 19))
+  (segment (start 206.502 41.42) (end 206.502 42.095) (width 0.25) (layer F.Cu) (net 19))
+  (segment (start 205.744001 44.365999) (end 206.417999 44.365999) (width 0.25) (layer F.Cu) (net 19))
+  (segment (start 206.502 42.095) (end 206.417999 42.179001) (width 0.25) (layer F.Cu) (net 19))
+  (segment (start 206.417999 44.365999) (end 210.909999 44.365999) (width 0.25) (layer F.Cu) (net 19))
   (segment (start 43.6505 -17.8175) (end 43.942 -17.526) (width 0.25) (layer F.Cu) (net 20))
   (segment (start 41.8345 -17.8175) (end 43.6505 -17.8175) (width 0.25) (layer F.Cu) (net 20))
@@
   (segment (start 229.252002 36.75) (end 228.152001 37.850001) (width 0.25) (layer F.Cu) (net 69))
   (segment (start 234.863 36.75) (end 229.252002 36.75) (width 0.25) (layer F.Cu) (net 69))
-  (segment (start 225.672 34.798) (end 227.624 36.75) (width 0.25) (layer F.Cu) (net 70))
   (segment (start 222.894 34.798) (end 225.672 34.798) (width 0.25) (layer F.Cu) (net 70))
+  (segment (start 225.672 34.798) (end 227.624 36.75) (width 0.25) (layer F.Cu) (net 70))
   (segment (start 218.988 33.862) (end 219.748 33.862) (width 0.25) (layer F.Cu) (net 71))
   (segment (start 220.28082 31.74099) (end 219.762999 32.258811) (width 0.25) (layer F.Cu) (net 71))

Commit message: fix voice board: layout
Parts:
- moved R15 0.32 mm to (215.1, 62.2)
- moved R42 0.24 mm to (218.6, 62.2)
Connections:
- U1 pad 11: (no net) -> VEE
- U1 pad 4: (no net) -> VCC
Routing:
- net VEE: track 88.7 -> 107.2 mm
- net VCC: track 79.8 -> 84.5 mm
- net Net-(R13-Pad1): track 11.8 -> 16.3 mm
- net GND: track 114.2 -> 115.6 mm
Changed lines of the file:
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@@
     (thickness 1.6)
     (drawings 1)
-    (tracks 502)
+    (tracks 515)
     (zones 0)
     (modules 117)
@@
     (pad 5 thru_hole oval (at 0 10.16) (size 1.6 1.6) (drill 0.8) (layers *.Cu *.Mask)
       (net 67 "Net-(R13-Pad1)"))
-    (pad 11 thru_hole oval (at 7.62 7.62) (size 1.6 1.6) (drill 0.8) (layers *.Cu *.Mask))
-    (pad 4 thru_hole oval (at 0 7.62) (size 1.6 1.6) (drill 0.8) (layers *.Cu *.Mask))
+    (pad 11 thru_hole oval (at 7.62 7.62) (size 1.6 1.6) (drill 0.8) (layers *.Cu *.Mask)
+      (net 38 VEE))
+    (pad 4 thru_hole oval (at 0 7.62) (size 1.6 1.6) (drill 0.8) (layers *.Cu *.Mask)
+      (net 39 VCC))
     (pad 10 thru_hole oval (at 7.62 10.16) (size 1.6 1.6) (drill 0.8) (layers *.Cu *.Mask)
       (net 76 "Net-(R37-Pad1)"))
@@
   )
   (module Resistor_SMD:R_0805_2012Metric_Pad1.15x1.40mm_HandSolder (layer F.Cu)
-    (at 218.567 61.976 90)
+    (at 218.567 62.221 90)
     (descr "Resistor SMD 0805 (2012 Metric), square (rectangular) end terminal, IPC_7351 nominal with elongated pad for handsoldering. (Body size source: https://docs.google.com/spreadsheets/d/1BsfQQcO9C6DZCsRaXUlFlo91Tg2WpOkGARC1WS5S8t0/edit?usp=sharing), generated with kicad-footprint-generator")
     (tags "resistor handsolder")
@@
   )
   (module Resistor_SMD:R_0805_2012Metric_Pad1.15x1.40mm_HandSolder (layer F.Cu)
-    (at 215.138 61.9035 90)
+    (at 215.138 62.221 90)
     (descr "Resistor SMD 0805 (2012 Metric), square (rectangular) end terminal, IPC_7351 nominal with elongated pad for handsoldering. (Body size source: https://docs.google.com/spreadsheets/d/1BsfQQcO9C6DZCsRaXUlFlo91Tg2WpOkGARC1WS5S8t0/edit?usp=sharing), generated with kicad-footprint-generator")
     (tags "resistor handsolder")
@@
   (segment (start 212.9155 59.2455) (end 214.5485 60.8785) (width 0.25) (layer F.Cu) (net 19))
   (segment (start 218.9025 60.8785) (end 220.5355 59.2455) (width 0.25) (layer F.Cu) (net 19))
-  (segment (start 215.138 60.8785) (end 218.9025 60.8785) (width 0.25) (layer F.Cu) (net 19))
-  (segment (start 207.3275 64.8335) (end 212.9155 59.2455) (width 0.25) (layer F.Cu) (net 19))
-  (segment (start 204.597 64.8335) (end 207.3275 64.8335) (width 0.25) (layer F.Cu) (net 19))
   (segment (start 203.3995 64.8335) (end 204.597 64.8335) (width 0.25) (layer F.Cu) (net 19))
   (segment (start 202.184 66.049) (end 203.3995 64.8335) (width 0.25) (layer F.Cu) (net 19))
@@
   (segment (start 206.502 42.095) (end 206.417999 42.179001) (width 0.25) (layer F.Cu) (net 19))
   (segment (start 206.417999 44.365999) (end 210.909999 44.365999) (width 0.25) (layer F.Cu) (net 19))
+  (segment (start 215.138 60.8785) (end 216.9975 60.8785) (width 0.25) (layer F.Cu) (net 19))
+  (segment (start 216.9975 60.8785) (end 218.9025 60.8785) (width 0.25) (layer F.Cu) (net 19))
+  (segment (start 213.342 62.992) (end 215.138 61.196) (width 0.25) (layer F.Cu) (net 19))
+  (segment (start 204.597 64.8335) (end 210.742498 64.8335) (width 0.25) (layer F.Cu) (net 19))
+  (segment (start 212.583998 62.992) (end 213.342 62.992) (width 0.25) (layer F.Cu) (net 19))
+  (segment (start 210.742498 64.8335) (end 212.583998 62.992) (width 0.25) (layer F.Cu) (net 19))
   (segment (start 43.6505 -17.8175) (end 43.942 -17.526) (width 0.25) (layer F.Cu) (net 20))
   (segment (start 41.8345 -17.8175) (end 43.6505 -17.8175) (width 0.25) (layer F.Cu) (net 20))
@@
   (segment (start 205.220372 70.545872) (end 204.597 69.9225) (width 0.25) (layer F.Cu) (net 38))
   (segment (start 212.156128 77.481628) (end 205.220372 70.545872) (width 0.25) (layer F.Cu) (net 38))
-  (segment (start 226.325628 77.481628) (end 212.156128 77.481628) (width 0.25) (layer F.Cu) (net 38))
   (segment (start 226.949 78.105) (end 226.325628 77.481628) (width 0.25) (layer F.Cu) (net 38))
   (segment (start 219.162 41.536) (end 216.488 38.862) (width 0.25) (layer F.Cu) (net 38))
@@
   (segment (start 109.339413 53.086) (end 98.432587 53.086) (width 0.25) (layer F.Cu) (net 38))
   (segment (start 113.594499 48.062499) (end 113.594499 48.830914) (width 0.25) (layer F.Cu) (net 38))
+  (segment (start 217.99481 62.23) (end 216.904372 63.320438) (width 0.25) (layer F.Cu) (net 38))
+  (segment (start 220.091 62.23) (end 217.99481 62.23) (width 0.25) (layer F.Cu) (net 38))
+  (segment (start 220.5355 61.7855) (end 220.091 62.23) (width 0.25) (layer F.Cu) (net 38))
+  (segment (start 216.904372 63.320438) (end 216.904372 77.481628) (width 0.25) (layer F.Cu) (net 38))
+  (segment (start 216.904372 77.481628) (end 212.156128 77.481628) (width 0.25) (layer F.Cu) (net 38))
+  (segment (start 226.325628 77.481628) (end 216.904372 77.481628) (width 0.25) (layer F.Cu) (net 38))
   (segment (start 199.8345 52.451) (end 199.8345 57.2135) (width 0.25) (layer F.Cu) (net 39))
   (segment (start 204.851 59.4995) (end 204.216 60.1345) (width 0.25) (layer F.Cu) (net 39))
@@
   (segment (start 205.876 59.4995) (end 204.851 59.4995) (width 0.25) (layer F.Cu) (net 39))
   (segment (start 207.544999 57.830501) (end 205.876 59.4995) (width 0.25) (layer F.Cu) (net 39))
-  (segment (start 215.029689 57.830501) (end 207.544999 57.830501) (width 0.25) (layer F.Cu) (net 39))
   (segment (start 216.35902 56.50117) (end 215.029689 57.830501) (width 0.25) (layer F.Cu) (net 39))
   (segment (start 216.35902 53.19161) (end 216.35902 56.50117) (width 0.25) (layer F.Cu) (net 39))
@@
   (segment (start 111.252 38.849) (end 110.249 37.846) (width 0.25) (layer F.Cu) (net 39))
   (segment (start 109.728 37.846) (end 97.523 37.846) (width 0.25) (layer F.Cu) (net 39))
+  (segment (start 211.282499 60.152499) (end 211.282499 57.830501) (width 0.25) (layer F.Cu) (net 39))
+  (segment (start 212.9155 61.7855) (end 211.282499 60.152499) (width 0.25) (layer F.Cu) (net 39))
+  (segment (start 215.029689 57.830501) (end 211.282499 57.830501) (width 0.25) (layer F.Cu) (net 39))
+  (segment (start 211.282499 57.830501) (end 207.544999 57.830501) (width 0.25) (layer F.Cu) (net 39))
   (segment (start 33.06 -17.994) (end 33.862 -17.994) (width 0.25) (layer F.Cu) (net 40))
   (segment (start 30.734 -20.32) (end 33.06 -17.994) (width 0.25) (layer F.Cu) (net 40))
@@
   (segment (start 214.3125 62.9285) (end 212.9155 64.3255) (width 0.25) (layer F.Cu) (net 67))
   (segment (start 215.138 62.9285) (end 214.3125 62.9285) (width 0.25) (layer F.Cu) (net 67))
-  (segment (start 211.78413 64.3255) (end 212.9155 64.3255) (width 0.25) (layer F.Cu) (net 67))
-  (segment (start 210.81931 64.3255) (end 211.78413 64.3255) (width 0.25) (layer F.Cu) (net 67))
-  (segment (start 208.14199 68.94099) (end 208.14199 67.00282) (width 0.25) (layer F.Cu) (net 67))
-  (segment (start 208.14199 67.00282) (end 210.81931 64.3255) (width 0.25) (layer F.Cu) (net 67))
-  (segment (start 208.9875 69.7865) (end 208.14199 68.94099) (width 0.25) (layer F.Cu) (net 67))
+  (segment (start 209.610872 69.163128) (end 208.9875 69.7865) (width 0.25) (layer F.Cu) (net 67))
+  (segment (start 210.493501 68.280499) (end 209.610872 69.163128) (width 0.25) (layer F.Cu) (net 67))
+  (segment (start 214.04687 64.3255) (end 216.09951 66.37814) (width 0.25) (layer F.Cu) (net 67))
+  (segment (start 215.806171 68.280499) (end 210.493501 68.280499) (width 0.25) (layer F.Cu) (net 67))
+  (segment (start 216.09951 67.98716) (end 215.806171 68.280499) (width 0.25) (layer F.Cu) (net 67))
+  (segment (start 216.09951 66.37814) (end 216.09951 67.98716) (width 0.25) (layer F.Cu) (net 67))
+  (segment (start 212.9155 64.3255) (end 214.04687 64.3255) (width 0.25) (layer F.Cu) (net 67))
   (segment (start 213.097 69.224) (end 212.9155 69.4055) (width 0.25) (layer F.Cu) (net 68))
   (segment (start 215.0745 69.224) (end 213.097 69.224) (width 0.25) (layer F.Cu) (net 68))

Commit message: minor fixes
Parts:
- added J7: Conn_02x02_Odd_Even, Connector_PinHeader_2.54mm:PinHeader_2x02_P2.54mm_Vertical, B.Cu at (242.6, 110.5)
- added Q21: BC547, Package_TO_SOT_THT:TO-92_Inline, B.Cu at (240.3, 133.6)
- added Q22: BC547, Package_TO_SOT_THT:TO-92_Inline, B.Cu at (235.5, 133.6)
- added R66: 100k, Resistor_SMD:R_0805_2012Metric_Pad1.15x1.40mm_HandSolder, F.Cu at (234.7, 108.5)
- added R67: 200k, Potentiometer_THT:Potentiometer_Bourns_3296W_Vertical, B.Cu at (238.0, 110.5)
- added R68: 2.5k, Resistor_SMD:R_0805_2012Metric_Pad1.15x1.40mm_HandSolder, F.Cu at (236.0, 129.0)
- added R69: 1Meg, Resistor_SMD:R_0805_2012Metric_Pad1.15x1.40mm_HandSolder, F.Cu at (243.6, 126.2)
- added R70: 1k, Resistor_SMD:R_0805_2012Metric_Pad1.15x1.40mm_HandSolder, F.Cu at (243.3, 132.1)
- added R71: 10k, Potentiometer_THT:Potentiometer_Bourns_3296W_Vertical, B.Cu at (245.4, 115.1)
- added R72: 10k, Potentiometer_THT:Potentiometer_Runtron_RM-065_Vertical, B.Cu at (229.1, 111.5)
- added U3: LM324, Package_DIP:DIP-14_W7.62mm, B.Cu at (233.7, 130.3)
- moved C12 98.8 mm to (51.8, 68.2)
- moved R56 98.8 mm to (51.6, 71.6)
- moved J6 76.5 mm to (65.0, 182.4)
- moved R60 76.5 mm to (75.4, 177.8)
- moved R61 76.5 mm to (82.5, 177.8)
- moved R62 76.5 mm to (89.7, 177.8)
- moved R57 76.5 mm to (70.6, 183.1)
- moved R58 76.5 mm to (77.7, 183.1)
- moved R59 76.5 mm to (84.8, 183.1)
Routing:
- net expo_raw: track 0.00 -> 36.1 mm
- net Net-(Q22-Pad1): track 0.00 -> 29.3 mm
- net Net-(Q21-Pad2): track 0.00 -> 27.9 mm
- net VCC: track 84.5 -> 112.2 mm
- net GND: track 115.6 -> 142.7 mm
- net VEE: track 107.2 -> 122.9 mm
- net expo_out: track 0.00 -> 12.0 mm
- net Net-(Q21-Pad3): track 0.00 -> 9.71 mm
- net Net-(Q21-Pad1): track 0.00 -> 8.85 mm
- net expo_in: track 0.00 -> 4.57 mm
- net Net-(R66-Pad1): track 0.00 -> 2.88 mm
- net Net-(R70-Pad2): track 0.00 -> 2.34 mm
Other:
- board text added: "PerfBoard"

Commit message: clean up schematic
Parts:
- added J8: Conn_02x03_Odd_Even, Connector_PinHeader_2.54mm:PinHeader_2x03_P2.54mm_Vertical, F.Cu at (124.7, -7.11)
- added J9: Conn_02x02_Odd_Even, Connector_PinHeader_2.54mm:PinHeader_2x02_P2.54mm_Vertical, F.Cu at (131.9, -7.11)
- JP1, JP2: footprint Connector_PinHeader_2.54mm:PinHeader_1x02_P2.54mm_Vertical -> footprints:SolderDipJumper2alt
- JP3: value Jumper_3_Bridged12 -> Conn_01x04_Male; footprint Connector_PinHeader_2.54mm:PinHeader_1x03_P2.54mm_Vertical -> Connector_PinHeader_2.54mm:PinHeader_1x04_P2.54mm_Vertical
- moved JP3 82.5 mm to (120.1, -7.11)
- moved JP1 1.27 mm to (117.6, 39.9), turned to 0 degrees
- moved JP2 1.27 mm to (90.2, 39.9), turned to 180 degrees
- moved R24 0.51 mm to (222.4, 34.8)
- moved R25 0.51 mm to (222.4, 32.8)
- moved R23 0.51 mm to (222.4, 36.8)
Connections:
- net VCA_ctl renamed Net-(C12-Pad1)
- net vca_audio_out renamed Net-(R17-Pad1)
- R1 pad 1: (no net) -> Net-(J8-Pad5)
- R18 pad 1: (no net) -> Net-(J9-Pad1)
- R19 pad 1: (no net) -> Net-(J9-Pad3)
- R2 pad 1: (no net) -> Net-(J8-Pad3)
Routing:
- net VEE: track 122.9 -> 146.8 mm
- net VCC: track 112.2 -> 131.4 mm
- net vcf_ctl_raw: track 15.3 -> 28.5 mm
- net Net-(R20-Pad2): track 6.45 -> 7.20 mm
- net Net-(C9-Pad2): track 7.32 -> 8.06 mm
- net Net-(C8-Pad2): track 7.45 -> 8.06 mm
- net vcf_ctl2: track 5.54 -> 5.03 mm
