File: hardware/voice_board/voice_board.kicad_pcb (KiCad board)
At the start: 2 copper layers, 130 parts, among them J1 Conn_02x06_Odd_Even, J2 Conn_02x02_Odd_Even, J3 Conn_02x02_Odd_Even, J4 Conn_01x02_Male, J5 Conn_02x03_Odd_Even, J6 Conn_02x02_Odd_Even, J7 Conn_02x02_Odd_Even, J8 Conn_02x03_Odd_Even, J9 Conn_02x02_Odd_Even, Q1 BC327, Q10 BC557, Q11 BC557, Q12 BC557, Q13 BC557, Q14 BC557, Q15 BC557, Q16 BC557, Q17 BC547, Q18 BC547, Q19 2N7000, Q2 BC557, Q20 2N7000, Q21 BC547, Q22 BC547, Q3 BC327, Q4 BC557, Q5 BC557, Q6 BC557, Q7 BC557, Q8 BC557, Q9 BC557, U1 TL074, U2 MCP4822, U3 LM324

Commit message: flip another footprint
Parts:
- moved U3 17.0 mm to (241.3, 115.1), turned to 180 degrees
Connections:
- U3 pad 1: Net-(Q21-Pad2) -> expo_out
- U3 pad 11: VCC -> VEE
- U3 pad 12: GND -> (no net)
- U3 pad 13: Net-(Q21-Pad1) -> (no net)
- U3 pad 14: Net-(R70-Pad2) -> (no net)
- U3 pad 2: expo_raw -> Net-(Q22-Pad1)
- U3 pad 4: VEE -> VCC
- U3 pad 5: (no net) -> GND
- U3 pad 6: (no net) -> Net-(Q21-Pad1)
- U3 pad 7: (no net) -> Net-(R70-Pad2)
- U3 pad 8: expo_out -> Net-(Q21-Pad2)
- U3 pad 9: Net-(Q22-Pad1) -> expo_raw
Changed lines of the file:
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@@
   )
   (module Package_DIP:DIP-14_W7.62mm (layer B.Cu)
-    (at 233.68 130.302)
+    (at 241.3 115.062 180)
     (descr "14-lead though-hole mounted DIP package, row spacing 7.62 mm (300 mils)")
     (tags "THT DIP DIL PDIP 2.54mm 7.62mm 300mil")
@@
       (effects (font (size 1 1) (thickness 0.15)) (justify mirror))
     )
+    (fp_arc (start 3.81 1.33) (end 2.81 1.33) (angle 180) (layer B.SilkS) (width 0.12))
+    (fp_line (start 1.635 1.27) (end 6.985 1.27) (layer B.Fab) (width 0.1))
+    (fp_line (start 6.985 1.27) (end 6.985 -16.51) (layer B.Fab) (width 0.1))
+    (fp_line (start 6.985 -16.51) (end 0.635 -16.51) (layer B.Fab) (width 0.1))
+    (fp_line (start 0.635 -16.51) (end 0.635 0.27) (layer B.Fab) (width 0.1))
+    (fp_line (start 0.635 0.27) (end 1.635 1.27) (layer B.Fab) (width 0.1))
+    (fp_line (start 2.81 1.33) (end 1.16 1.33) (layer B.SilkS) (width 0.12))
+    (fp_line (start 1.16 1.33) (end 1.16 -16.57) (layer B.SilkS) (width 0.12))
+    (fp_line (start 1.16 -16.57) (end 6.46 -16.57) (layer B.SilkS) (width 0.12))
+    (fp_line (start 6.46 -16.57) (end 6.46 1.33) (layer B.SilkS) (width 0.12))
+    (fp_line (start 6.46 1.33) (end 4.81 1.33) (layer B.SilkS) (width 0.12))
+    (fp_line (start -1.1 1.55) (end -1.1 -16.8) (layer B.CrtYd) (width 0.05))
+    (fp_line (start -1.1 -16.8) (end 8.7 -16.8) (layer B.CrtYd) (width 0.05))
+    (fp_line (start 8.7 -16.8) (end 8.7 1.55) (layer B.CrtYd) (width 0.05))
+    (fp_line (start 8.7 1.55) (end -1.1 1.55) (layer B.CrtYd) (width 0.05))
     (fp_text user %R (at 3.81 -7.62) (layer B.Fab)
       (effects (font (size 1 1) (thickness 0.15)) (justify mirror))
     )
-    (fp_line (start 8.7 1.55) (end -1.1 1.55) (layer B.CrtYd) (width 0.05))
-    (fp_line (start 8.7 -16.8) (end 8.7 1.55) (layer B.CrtYd) (width 0.05))
-    (fp_line (start -1.1 -16.8) (end 8.7 -16.8) (layer B.CrtYd) (width 0.05))
-    (fp_line (start -1.1 1.55) (end -1.1 -16.8) (layer B.CrtYd) (width 0.05))
-    (fp_line (start 6.46 1.33) (end 4.81 1.33) (layer B.SilkS) (width 0.12))
-    (fp_line (start 6.46 -16.57) (end 6.46 1.33) (layer B.SilkS) (width 0.12))
-    (fp_line (start 1.16 -16.57) (end 6.46 -16.57) (layer B.SilkS) (width 0.12))
-    (fp_line (start 1.16 1.33) (end 1.16 -16.57) (layer B.SilkS) (width 0.12))
-    (fp_line (start 2.81 1.33) (end 1.16 1.33) (layer B.SilkS) (width 0.12))
-    (fp_line (start 0.635 0.27) (end 1.635 1.27) (layer B.Fab) (width 0.1))
-    (fp_line (start 0.635 -16.51) (end 0.635 0.27) (layer B.Fab) (width 0.1))
-    (fp_line (start 6.985 -16.51) (end 0.635 -16.51) (layer B.Fab) (width 0.1))
-    (fp_line (start 6.985 1.27) (end 6.985 -16.51) (layer B.Fab) (width 0.1))
-    (fp_line (start 1.635 1.27) (end 6.985 1.27) (layer B.Fab) (width 0.1))
-    (fp_arc (start 3.81 1.33) (end 2.81 1.33) (angle 180) (layer B.SilkS) (width 0.12))
-    (pad 14 thru_hole oval (at 7.62 0) (size 1.6 1.6) (drill 0.8) (layers *.Cu *.Mask)
+    (pad 1 thru_hole rect (at 0 0 180) (size 1.6 1.6) (drill 0.8) (layers *.Cu *.Mask)
+      (net 84 expo_out))
+    (pad 8 thru_hole oval (at 7.62 -15.24 180) (size 1.6 1.6) (drill 0.8) (layers *.Cu *.Mask)
+      (net 89 "Net-(Q21-Pad2)"))
+    (pad 2 thru_hole oval (at 0 -2.54 180) (size 1.6 1.6) (drill 0.8) (layers *.Cu *.Mask)
+      (net 90 "Net-(Q22-Pad1)"))
+    (pad 9 thru_hole oval (at 7.62 -12.7 180) (size 1.6 1.6) (drill 0.8) (layers *.Cu *.Mask)
+      (net 85 expo_raw))
+    (pad 3 thru_hole oval (at 0 -5.08 180) (size 1.6 1.6) (drill 0.8) (layers *.Cu *.Mask)
+      (net 19 GND))
+    (pad 10 thru_hole oval (at 7.62 -10.16 180) (size 1.6 1.6) (drill 0.8) (layers *.Cu *.Mask)
+      (net 19 GND))
+    (pad 4 thru_hole oval (at 0 -7.62 180) (size 1.6 1.6) (drill 0.8) (layers *.Cu *.Mask)
+      (net 38 VCC))
+    (pad 11 thru_hole oval (at 7.62 -7.62 180) (size 1.6 1.6) (drill 0.8) (layers *.Cu *.Mask)
+      (net 37 VEE))
+    (pad 5 thru_hole oval (at 0 -10.16 180) (size 1.6 1.6) (drill 0.8) (layers *.Cu *.Mask)
+      (net 19 GND))
+    (pad 12 thru_hole oval (at 7.62 -5.08 180) (size 1.6 1.6) (drill 0.8) (layers *.Cu *.Mask))
+    (pad 6 thru_hole oval (at 0 -12.7 180) (size 1.6 1.6) (drill 0.8) (layers *.Cu *.Mask)
+      (net 87 "Net-(Q21-Pad1)"))
+    (pad 13 thru_hole oval (at 7.62 -2.54 180) (size 1.6 1.6) (drill 0.8) (layers *.Cu *.Mask))
+    (pad 7 thru_hole oval (at 0 -15.24 180) (size 1.6 1.6) (drill 0.8) (layers *.Cu *.Mask)
       (net 92 "Net-(R70-Pad2)"))
-    (pad 7 thru_hole oval (at 0 -15.24) (size 1.6 1.6) (drill 0.8) (layers *.Cu *.Mask))
-    (pad 13 thru_hole oval (at 7.62 -2.54) (size 1.6 1.6) (drill 0.8) (layers *.Cu *.Mask)
-      (net 87 "Net-(Q21-Pad1)"))
-    (pad 6 thru_hole oval (at 0 -12.7) (size 1.6 1.6) (drill 0.8) (layers *.Cu *.Mask))
-    (pad 12 thru_hole oval (at 7.62 -5.08) (size 1.6 1.6) (drill 0.8) (layers *.Cu *.Mask)
-      (net 19 GND))
-    (pad 5 thru_hole oval (at 0 -10.16) (size 1.6 1.6) (drill 0.8) (layers *.Cu *.Mask))
-    (pad 11 thru_hole oval (at 7.62 -7.62) (size 1.6 1.6) (drill 0.8) (layers *.Cu *.Mask)
-      (net 38 VCC))
-    (pad 4 thru_hole oval (at 0 -7.62) (size 1.6 1.6) (drill 0.8) (layers *.Cu *.Mask)
-      (net 37 VEE))
-    (pad 10 thru_hole oval (at 7.62 -10.16) (size 1.6 1.6) (drill 0.8) (layers *.Cu *.Mask)
-      (net 19 GND))
-    (pad 3 thru_hole oval (at 0 -5.08) (size 1.6 1.6) (drill 0.8) (layers *.Cu *.Mask)
-      (net 19 GND))
-    (pad 9 thru_hole oval (at 7.62 -12.7) (size 1.6 1.6) (drill 0.8) (layers *.Cu *.Mask)
-      (net 90 "Net-(Q22-Pad1)"))
-    (pad 2 thru_hole oval (at 0 -2.54) (size 1.6 1.6) (drill 0.8) (layers *.Cu *.Mask)
-      (net 85 expo_raw))
-    (pad 8 thru_hole oval (at 7.62 -15.24) (size 1.6 1.6) (drill 0.8) (layers *.Cu *.Mask)
-      (net 84 expo_out))
-    (pad 1 thru_hole rect (at 0 0) (size 1.6 1.6) (drill 0.8) (layers *.Cu *.Mask)
-      (net 89 "Net-(Q21-Pad2)"))
+    (pad 14 thru_hole oval (at 7.62 0 180) (size 1.6 1.6) (drill 0.8) (layers *.Cu *.Mask))
     (model ${KISYS3DMOD}/Package_DIP.3dshapes/DIP-14_W7.62mm.wrl
       (at (xyz 0 0 0))

Commit message: replace some SMD caps with thts
Parts:
- C1: footprint Capacitor_SMD:C_0805_2012Metric_Pad1.15x1.40mm_HandSolder -> Capacitor_THT:CP_Radial_D7.5mm_P2.50mm; moved to B.Cu
- C2, C7: footprint Capacitor_SMD:CP_Elec_8x5.4 -> Capacitor_THT:CP_Radial_D7.5mm_P2.50mm; moved to B.Cu
- J8, J9, R52, R55: moved to B.Cu
- JP3: footprint Connector_PinHeader_2.54mm:PinHeader_1x04_P2.54mm_Vertical -> footprints:SolderDipJumper4alt; moved to B.Cu
- moved JP3 25.7 mm to (145.5, -10.4)
- moved C1 8.49 mm to (192.8, 54.1), turned to 0 degrees
- moved C7 1.78 mm to (242.1, 53.8)

Commit message: flip some potis
Parts:
- J3, R20: moved to B.Cu
- moved J9 112.5 mm to (233.9, 40.4), turned to 270 degrees
- moved JP3 73.4 mm to (192.5, 46.0)
- moved R20 5.00 mm to (216.5, 38.9), turned to 0 degrees
Connections:
- R18 pad 1: Net-(J9-Pad1) -> Net-(J9-Pad3)
- R19 pad 1: Net-(J9-Pad3) -> Net-(J9-Pad1)
- R20 pad 1: VCC -> VEE
- R20 pad 3: VEE -> VCC

Commit message: routing improvement
Parts:
- J8: value Conn_02x03_Odd_Even -> Conn_02x02_Odd_Even; footprint Connector_PinHeader_2.54mm:PinHeader_2x03_P2.54mm_Vertical -> Connector_PinHeader_2.54mm:PinHeader_2x02_P2.54mm_Vertical
- moved J3 111.2 mm to (210.8, 74.2), turned to 270 degrees
- moved J8 85.6 mm to (196.1, 40.1), turned to 90 degrees
- moved R5 21.5 mm to (199.6, 37.6)
- moved C2 19.3 mm to (224.2, 48.8)
- moved R22 17.4 mm to (222.8, 46.5), turned to 180 degrees
- moved R21 7.37 mm to (207.0, 37.6)
- moved J9 0.51 mm to (233.9, 39.9)
- moved R20 0.51 mm to (216.5, 38.4)
- moved R24 0.51 mm to (222.4, 34.3)
- moved R18 0.51 mm to (237.4, 31.2)
- moved R19 0.51 mm to (230.1, 31.2)
- moved R23 0.51 mm to (222.4, 36.3)
- moved R25 0.51 mm to (222.4, 32.3)
- moved R39 0.51 mm to (228.9, 43.7)
Connections:
- J8 pad 1: vca_ctl_raw -> Net-(J8-Pad1)
- J8 pad 2: vca_audio_in -> vca_ctl_raw
- J8 pad 4: (no net) -> GND
- R1 pad 1: Net-(J8-Pad5) -> Net-(J8-Pad3)
- R2 pad 1: Net-(J8-Pad3) -> Net-(J8-Pad1)
Routing:
- net GND: track 142.7 -> 222.0 mm, vias 0 -> 3
- net vcf_audio_out: track 9.32 -> 58.9 mm, vias 0 -> 1
- net vca_ctl_raw: track 12.4 -> 40.8 mm
- net Net-(C2-Pad2): track 0.00 -> 21.6 mm
- net VCC: track 131.4 -> 112.7 mm, vias 0 -> 1
- net vcf_ctl_raw: track 28.5 -> 46.1 mm
- net Net-(Q21-Pad2): track 27.9 -> 10.9 mm
- net (no net): track 17.0 -> 0.00 mm
- net Net-(J8-Pad1): track 0.00 -> 13.9 mm, vias 0 -> 2
- net Net-(J9-Pad1): track 0.00 -> 13.3 mm
- net Net-(J8-Pad3): track 0.00 -> 9.61 mm
- net Net-(J9-Pad3): track 0.00 -> 9.56 mm
- net vca_audio_in: track 0.00 -> 8.55 mm
- net Net-(C2-Pad1): track 2.14 -> 9.63 mm
- net Net-(C7-Pad1): track 0.00 -> 6.23 mm
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
Commit message: move most things together
Parts:
- moved J4 211.8 mm to (207.0, 94.5), turned to 0 degrees
- moved R54 198.4 mm to (198.9, 94.5), turned to 270 degrees
- moved R53 190.1 mm to (198.9, 87.1), turned to 270 degrees
- moved C11 188.8 mm to (193.8, 93.2), turned to 90 degrees
- moved C17 187.5 mm to (190.5, 96.3), turned to 270 degrees
- moved C10 182.8 mm to (193.8, 88.1), turned to 90 degrees
- moved C16 182.3 mm to (190.5, 92.2), turned to 90 degrees
- moved U2 181.8 mm to (188.3, 94.5), turned to 0 degrees
- moved R52 180.1 mm to (182.6, 120.7)
- moved C12 180.1 mm to (214.8, 144.6)
- moved R55 180.1 mm to (205.2, 141.5)
- moved R56 180.1 mm to (214.6, 148.1)
- moved J6 176.8 mm to (165.4, 36.8)
- moved R57 176.8 mm to (170.9, 37.6)
- moved R60 176.8 mm to (175.8, 32.3)
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Other:
- board text removed: "PerfBoard"

Commit message: lots of labels
Parts:
- moved R72 19.0 mm to (184.4, 83.8), turned to 0 degrees
- moved C16 7.62 mm to (190.5, 99.8)
- moved C8 7.62 mm to (216.7, 102.9)
- moved C9 7.62 mm to (237.5, 102.9)
- moved D1 7.62 mm to (222.8, 98.3)
- moved D2 7.62 mm to (231.4, 98.3)
- moved D3 7.62 mm to (222.5, 95.2)
- moved D4 7.62 mm to (231.6, 95.2)
- moved J1 7.62 mm to (225.8, 106.7)
- moved J2 7.62 mm to (182.4, 99.6)
- moved J4 7.62 mm to (207.0, 102.1)
- moved JP1 7.62 mm to (213.4, 105.9)
- moved JP2 7.62 mm to (240.8, 105.9)
- moved R44 7.62 mm to (222.8, 105.7)
- moved R45 7.62 mm to (231.4, 105.7)
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Routing:
- net VCC: track 112.7 -> 88.4 mm
- net VEE: track 148.2 -> 132.5 mm
- net Net-(J8-Pad3): track 9.61 -> 0.00 mm
- net expo_raw: track 36.1 -> 26.8 mm
- net Net-(Q22-Pad1): track 29.3 -> 23.8 mm
- net Net-(J8-Pad1): track 13.9 -> 8.64 mm
- net vcf_audio_out: track 58.9 -> 62.7 mm
- net vca_ctl_raw: track 40.8 -> 37.3 mm
- net Net-(R66-Pad1): track 2.88 -> 5.28 mm
- net Net-(C1-Pad2): track 8.51 -> 6.38 mm
- net Net-(Q1-Pad2): track 9.11 -> 10.3 mm
- net vca_audio_in: track 8.55 -> 7.79 mm
Other:
- board text added: "GND"
- board text added: "Vcc"
- board text added: "Vee"
- board text added: "buffered"
- board text added: "clamped"
- board text added: "feedback/ resonance"
- board text added: "in"
- board text added: "raw"
- board text added: "scale"
- board text added: "sync"
- board text added: "trim"
- board text added: "tune"
- board text removed: "3x low pass filter"

Commit message: ?
Parts:
- moved R56 35.0 mm to (194.6, 119.4)
- moved C12 35.0 mm to (194.8, 115.9)
- moved R55 22.5 mm to (199.6, 119.6)
- moved R66 17.5 mm to (165.1, 70.6)
- moved R67 17.5 mm to (162.6, 68.6)
- moved R71 17.5 mm to (158.0, 75.9)
- moved J7 17.5 mm to (162.6, 73.2)
- moved Q21 17.5 mm to (139.4, 70.9)
- moved Q22 17.5 mm to (139.4, 66.0)
- moved R68 17.5 mm to (144.0, 66.5)
- moved R69 17.5 mm to (146.8, 74.2)
- moved R70 17.5 mm to (141.0, 73.9)
- moved R72 17.5 mm to (168.1, 77.5)
- moved U3 17.5 mm to (158.0, 71.9)
Routing:
- net VCC: track 88.4 -> 277.4 mm, vias 1 -> 5
- net GND: track 222.1 -> 265.7 mm, vias 3 -> 6
- net vcf_audio_in: track 0.00 -> 29.8 mm
- net VEE: track 132.5 -> 149.9 mm
- net Net-(J8-Pad3): track 0.00 -> 12.5 mm
- net mixer_out: track 23.4 -> 35.2 mm, vias 0 -> 1
- net Net-(J8-Pad1): track 8.64 -> 17.8 mm
- net vca_ctl_raw: track 37.3 -> 43.0 mm
Other:
- board text added: "RC-lowpass"
- board text added: "V_ctl generation"
- board text added: "exponential converter"
- board text added: "mixer"
- board text added: "out"
- board text added: "square_ctl buffer and sync"

Commit message: move VCF poti to VCF side
Parts:
- moved R21 11.2 mm to (216.7, 43.2)
- moved R23 5.21 mm to (222.1, 31.1)
- moved R25 3.46 mm to (219.1, 33.3), turned to 270 degrees
- moved R20 3.05 mm to (216.7, 35.3)
- moved R24 1.17 mm to (222.1, 33.1)
Routing:
- net VCC: track 277.4 -> 247.3 mm, vias 5 -> 6
- net vcf_audio_in: track 29.8 -> 43.3 mm
- net Net-(C2-Pad2): track 21.6 -> 11.9 mm, vias 0 -> 2
- net Net-(R20-Pad2): track 7.20 -> 1.96 mm
- net vcf_ctl_raw: track 46.1 -> 50.0 mm
- net GND: track 265.7 -> 264.1 mm, vias 6 -> 4
- net vcf_ctl1: track 12.6 -> 13.8 mm
- net VEE: track 149.9 -> 151.1 mm
- net vcf_ctl2: track 5.03 -> 5.77 mm
Other:
- board text added: "pregain"
