File: hardware/voice_board/voice_board.kicad_pcb (KiCad board)
At the start: 2 copper layers, 83.8 x 72.4 mm, 133 parts, among them J1 Conn_02x06_Odd_Even, J10 Conn_01x02_Male, J2 Conn_02x02_Odd_Even, J3 Conn_02x02_Odd_Even, J4 Conn_01x02_Male, J5 Conn_02x03_Odd_Even, J6 Conn_02x02_Odd_Even, J7 Conn_02x02_Odd_Even, J8 Conn_02x02_Odd_Even, J9 Conn_02x02_Odd_Even, Q1 BC327, Q10 BC557, Q11 BC557, Q12 BC557, Q13 BC557, Q14 BC557, Q15 BC557, Q16 BC557, Q17 BC547, Q18 BC547, Q19 2N7000, Q2 BC557, Q20 2N7000, Q21 BC547, Q22 BC547, Q3 BC327, Q4 BC557, Q5 BC557, Q6 BC557, Q7 BC557, Q8 BC557, Q9 BC557, U1 TL074, U2 MCP4822, U3 LM324

Commit message: final version of voice board mk I
Parts:
- removed C12: 100n, Capacitor_SMD:C_0805_2012Metric_Pad1.15x1.40mm_HandSolder
- removed R52, R55: 1k, Potentiometer_THT:Potentiometer_Runtron_RM-065_Vertical
- removed R56: 10k, Resistor_SMD:R_0805_2012Metric_Pad1.15x1.40mm_HandSolder
- moved R35 1.82 mm to (231.1, 55.4), turned to 90 degrees
Routing:
- net GND: track 388.4 -> 443.6 mm, vias 10 -> 14
- net Net-(R26-Pad2): track 7.07 -> 9.55 mm
- net VCC: track 319.0 -> 320.5 mm
- net Net-(C7-Pad2): track 27.5 -> 26.3 mm
- net Net-(C3-Pad2): track 11.3 -> 10.8 mm
- added copper zone on B.Cu, net GND
- added copper zone on F.Cu, net GND
