File: simulation/expo/expo.sch (KiCad schematic (older format))
At the start: 15 parts, among them Q1 BC546, Q2 BC546, U1 LM324, U2 LM324, U3 LM324

Commit message: voice board: add expo
Parts:
- Q1, Q2: Spice_Lib_File /home/flo/kicad/synth/simulation/lib/BC546.lib -> ../lib/BC546.lib
- U1, U2, U3: Spice_Lib_File /home/flo/kicad/synth/simulation/lib/LM324.ti.lib -> ../lib/LM324.ti.lib
Changed lines of the file:
@@
 EESchema Schematic File Version 4
-EELAYER 29 0
+LIBS:expo-cache
+EELAYER 30 0
 EELAYER END
 $Descr A4 11693 8268
@@
 F 5 "BC546B" H 7850 2200 50  0001 C CNN "Spice_Model"
 F 6 "Y" H 7850 2200 50  0001 C CNN "Spice_Netlist_Enabled"
-F 7 "/home/flo/kicad/synth/simulation/lib/BC546.lib" H 7850 2200 50  0001 C CNN "Spice_Lib_File"
+F 7 "../lib/BC546.lib" H 7850 2200 50  0001 C CNN "Spice_Lib_File"
 	1    7850 2200
 	1    0    0    -1
@@
 F 5 "BC546B" H 8950 2200 50  0001 C CNN "Spice_Model"
 F 6 "Y" H 8950 2200 50  0001 C CNN "Spice_Netlist_Enabled"
-F 7 "/home/flo/kicad/synth/simulation/lib/BC546.lib" H 8950 2200 50  0001 C CNN "Spice_Lib_File"
+F 7 "../lib/BC546.lib" H 8950 2200 50  0001 C CNN "Spice_Lib_File"
 	1    8950 2200
 	-1   0    0    -1
@@
 F 6 "Y" H 7350 3000 50  0001 C CNN "Spice_Netlist_Enabled"
 F 7 "1 2 4 5 3" H 7350 3000 50  0001 C CNN "Spice_Node_Sequence"
-F 8 "/home/flo/kicad/synth/simulation/lib/LM324.ti.lib" H 7350 3000 50  0001 C CNN "Spice_Lib_File"
+F 8 "../lib/LM324.ti.lib" H 7350 3000 50  0001 C CNN "Spice_Lib_File"
 	1    7350 3000
 	1    0    0    1
@@
 F 6 "Y" H 9950 1700 50  0001 C CNN "Spice_Netlist_Enabled"
 F 7 "1 2 4 5 3" H 9950 1700 50  0001 C CNN "Spice_Node_Sequence"
-F 8 "/home/flo/kicad/synth/simulation/lib/LM324.ti.lib" H 9950 1700 50  0001 C CNN "Spice_Lib_File"
+F 8 "../lib/LM324.ti.lib" H 9950 1700 50  0001 C CNN "Spice_Lib_File"
 	1    9950 1700
 	1    0    0    1
@@
 F 6 "Y" H 5050 1750 50  0001 C CNN "Spice_Netlist_Enabled"
 F 7 "1 2 4 5 3" H 5050 1750 50  0001 C CNN "Spice_Node_Sequence"
-F 8 "/home/flo/kicad/synth/simulation/lib/LM324.ti.lib" H 5050 1750 50  0001 C CNN "Spice_Lib_File"
+F 8 "../lib/LM324.ti.lib" H 5050 1750 50  0001 C CNN "Spice_Lib_File"
 	1    5050 1750
 	1    0    0    1
