File: hardware/control_board_prototype/control_board_prototype.kicad_pcb (KiCad board)
At the start: 2 copper layers, 98 x 54.4 mm, 78 parts, among them J1 Conn_01x17_Male, J10 Conn_02x06_Odd_Even, J11 Conn_02x10_Odd_Even, J2 Conn_01x15_Male, J3 Conn_01x02_Male, J4 Conn_02x10_Odd_Even, J5 Conn_02x10_Odd_Even, J6 Conn_02x10_Odd_Even, J7 Conn_02x04_Odd_Even, J8 Conn_02x06_Odd_Even, J9 Conn_02x04_Odd_Even, U1 LM317_3PinPackage, U2 LM358, U3 TLE2426xLP, U4 BU2505FV, U5 BU2505FV

Commit message: last fixes for control and voice board:
control board: add 3V3 header
voice board: mcp4822 silkscreen
Parts:
- removed G***: LOGO, windfisch:windfisch_smaller
- removed REF**: KiCad-Logo2_8mm_SilkScreen, Symbol:KiCad-Logo2_8mm_SilkScreen
- removed REF**: OSHW-Logo2_14.6x12mm_SilkScreen, Symbol:OSHW-Logo2_14.6x12mm_SilkScreen
- added J12: Conn_02x04_Odd_Even, Connector_PinHeader_2.54mm:PinHeader_2x04_P2.54mm_Vertical, F.Cu at (165.4, 74.5)
- U1: value LM317_3PinPackage -> LM317
Routing:
- net +3V3: track 49.5 -> 103.5 mm, vias 2 -> 5
Other:
- board text added: "3V3"
