File: hardware/control_board_prototype/control_board_prototype.kicad_pcb (KiCad board)
At the start: 2 copper layers, 98 x 54.4 mm, 76 parts, among them J1 Conn_01x17_Male, J10 Conn_02x06_Odd_Even, J11 Conn_02x10_Odd_Even, J12 Conn_02x04_Odd_Even, J2 Conn_01x15_Male, J3 Conn_01x02_Male, J4 Conn_02x10_Odd_Even, J5 Conn_02x10_Odd_Even, J6 Conn_02x10_Odd_Even, J7 Conn_02x04_Odd_Even, J8 Conn_02x06_Odd_Even, J9 Conn_02x04_Odd_Even, U1 LM317, U2 LM358, U3 TLE2426xLP, U4 BU2505FV, U5 BU2505FV

Commit message: control board docs and rev02
Parts:
- added G***: LOGO, windfisch:windfisch_smaller, B.Cu at (204.7, 75.2)
Other:
- board text added: "rev02"
