File: hardware/control_board_prototype/control_board_prototype.kicad_pcb (KiCad board)
At the start: 2 copper layers, 98 x 54.4 mm, 77 parts, among them J1 Conn_01x17_Male, J10 Conn_02x06_Odd_Even, J11 Conn_02x10_Odd_Even, J12 Conn_02x04_Odd_Even, J2 Conn_01x15_Male, J3 Conn_01x02_Male, J4 Conn_02x10_Odd_Even, J5 Conn_02x10_Odd_Even, J6 Conn_02x10_Odd_Even, J7 Conn_02x04_Odd_Even, J8 Conn_02x06_Odd_Even, J9 Conn_02x04_Odd_Even, U1 LM317, U2 LM358, U3 TLE2426xLP, U4 BU2505FV, U5 BU2505FV

Commit message: add BU2505 dac channel labels
Other:
- board text added: "1"
- board text added: "10"
- board text added: "2"
- board text added: "8 7 6 5 4 3"
- board text added: "9"
Changed lines of the file:
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@@
   (general
     (thickness 1.6)
-    (drawings 52)
+    (drawings 61)
     (tracks 884)
     (zones 0)
@@
     (descr "Through hole straight pin header, 2x04, 2.54mm pitch, double rows")
     (tags "Through hole pin header THT 2x04 2.54mm double row")
-    (fp_text reference J9 (at 5.08 0) (layer F.SilkS)
+    (fp_text reference J9 (at -2.54 -2.54) (layer F.SilkS)
       (effects (font (size 1 1) (thickness 0.15)))
     )
@@
     (descr "Through hole straight pin header, 2x04, 2.54mm pitch, double rows")
     (tags "Through hole pin header THT 2x04 2.54mm double row")
-    (fp_text reference J7 (at 5.08 0) (layer F.SilkS)
+    (fp_text reference J7 (at -2.159 -2.413) (layer F.SilkS)
       (effects (font (size 1 1) (thickness 0.15)))
     )
@@
     )
   )
+  (gr_text "8\n7\n6\n5\n4\n3" (at 259.969 57.277) (layer F.SilkS)
+    (effects (font (size 1 1) (thickness 0.2)))
+  )
+  (gr_text 1 (at 226.822 72.898) (layer F.SilkS)
+    (effects (font (size 1 1) (thickness 0.2)))
+  )
+  (gr_text 9 (at 226.822 67.818) (layer F.SilkS)
+    (effects (font (size 1 1) (thickness 0.2)))
+  )
+  (gr_text 2 (at 226.822 75.565) (layer F.SilkS)
+    (effects (font (size 1 1) (thickness 0.2)))
+  )
+  (gr_text 10 (at 226.949 70.358) (layer F.SilkS)
+    (effects (font (size 1 1) (thickness 0.2)))
+  )
+  (gr_text 2 (at 226.822 47.117) (layer F.SilkS)
+    (effects (font (size 1 1) (thickness 0.2)))
+  )
+  (gr_text 1 (at 226.822 44.45) (layer F.SilkS)
+    (effects (font (size 1 1) (thickness 0.2)))
+  )
+  (gr_text 10 (at 226.949 41.91) (layer F.SilkS)
+    (effects (font (size 1 1) (thickness 0.2)))
+  )
+  (gr_text 9 (at 226.822 39.37) (layer F.SilkS)
+    (effects (font (size 1 1) (thickness 0.2)))
+  )
   (gr_text rev02 (at 208.788 70.104 90) (layer B.SilkS)
