File: simulation/vcf/vcf.sch (KiCad schematic (older format))
At the start: 38 parts, among them Q1 BC557B, Q10 BC557B, Q11 BC557B, Q12 BC557B, Q2 BC557B, Q3 BC557B, Q4 BC557B, Q5 BC557B, Q6 BC557B, Q7 BC557B, Q8 BC557B, Q9 BC557B, U2 LM324

Commit message: vcf simulation works :)
Parts:
- removed Q1, Q3: BC557B, symbol pspice:QPNP
- removed R1: 10k, symbol Device:R
- removed R34: 680, Resistor_SMD:R_0805_2012Metric_Pad1.15x1.40mm_HandSolder, symbol Device:R
- removed V3: -2, symbol pspice:VSOURCE
- added C6: 100u, symbol Device:C
- added I1: 100u, symbol pspice:ISOURCE
- C2, C3, C4, C5: value 47n -> 100n
- R2: value 10k -> 100k
- R7, R8: value 10k -> 1Meg
- V1, V2: value 5 -> 20
Connections:
- net 0: now also I1.1 (E1); no longer Q9.2 (B), R15.2
- net signal_preatt: now also C6.2; no longer Q5.2 (B), R5.2
- net at Q5.3 (E), Q9.3 (E): now also I1.2 (E2)
- new net: C6.1, Q5.2 (B), R5.2
- new net: Q9.2 (B), R15.2
Other:
- note removed: "Control voltage:\nVCC=closed"
- note removed: "current mirror as\nvoltage controlled\ncurrent source"

Commit message: some VCF schematic changes
Parts:
- added C7: 1u, symbol Device:C
- added R1: 20.98k, Resistor_SMD:R_0805_2012Metric_Pad1.15x1.40mm_HandSolder, symbol Device:R
- added R16: 200k, symbol Device:R
- added R17, R18: 100k, symbol Device:R
- added R19, R20: 1Meg, symbol Device:R
- added U1: LM324, symbol pspice:OPAMP
- C2, C3, C4, C5: value 100n -> 47n
- C6: value 100u -> 10u
- I1: value 100u -> 0.15m
- R10: value 1Meg -> 100k
- R7, R8: value 1Meg -> 220
- R9: value 1Meg -> 200k
- V1, V2: value 20 -> 5
Connections:
- net 0: now also R16.2, R19.2
- net VCC: now also U1.4 (V+)
- net VEE: now also R17.2, R18.2, U1.5 (V-)
- net diff1: now also C5.1, Q12.3 (E), Q4.1 (C); no longer C5.2, Q2.1 (C), Q8.3 (E)
- net diff2: now also C5.2, Q2.1 (C), Q8.3 (E); no longer C5.1, Q12.3 (E), Q4.1 (C)
- net signal_out: now also R1.1
- net at R7.1, R9.1, U2.1 (+): now also R16.1
- net at Q9.2 (B), R15.2: now also C7.2
- new net: R17.1, R19.1, U1.1 (+)
- new net: R18.1, R20.2, U1.2 (-)
- new net: C7.1, R1.2
- new net signal_out2: R20.1, U1.3
Other:
- note added: ".tran 10u 30m"
- note removed: ".tran 10u 10m"
- moved on the sheet: R9

Commit message: cleaned up vcf simulation
Parts:
- removed C1: 470n, symbol Device:C
- removed R16: 200k, symbol Device:R
- removed R17, R18: 100k, symbol Device:R
- removed R19, R20: 1Meg, symbol Device:R
- removed U1: LM324, symbol pspice:OPAMP
- R1: value 20.98k -> 1000Meg
- R9: value 200k -> 100k
Other:
- note added: "resonance control.\n(good resonance at 50k-100k)"
- moved on the sheet: R9

Commit message: reduce plot quality for speed
Parts:
- removed C7: 1u, symbol Device:C
- removed R1: 1000Meg, Resistor_SMD:R_0805_2012Metric_Pad1.15x1.40mm_HandSolder, symbol Device:R
- I1: value 0.15m -> 0.01m
- R10, R9: value 100k -> 500k
- R7, R8: value 220 -> 1k
- V4: value PULSE(-2 2 0 0m 0m 1m 2m) -> PULSE(-2 2 0 0m 0m 2m 4m)
Connections:
- net foo: now reaches Q12.2 (B), Q8.2 (B), R13.2, R14.1
Other:
- note added: "-3.9V"
- note added: "ca 0.5* I1 each"
- note added: "ca 6 uA"
- note added: "diff1,2 = -3.3V ca"
Changed lines of the file:
@@
 P 3650 3825
 F 0 "V4" H 3250 3925 50  0000 L CNN
-F 1 "PULSE(-2 2 0 0m 0m 1m 2m)" H 3225 3175 50  0000 L CNN
+F 1 "PULSE(-2 2 0 0m 0m 2m 4m)" H 3225 3175 50  0000 L CNN
 F 2 "" H 3650 3825 50  0001 C CNN
 F 3 "~" H 3650 3825 50  0001 C CNN
@@
 	5925 5450 5925 5550
 Wire Wire Line
-	6900 5450 6900 5400
-Wire Wire Line
 	5925 5450 6450 5450
 Wire Wire Line
-	6900 5550 6900 5600
-Wire Wire Line
 	6225 5550 6450 5550
-Wire Wire Line
-	6975 4700 6975 3700
 Wire Wire Line
 	6675 2950 5475 2950
@@
 P 7625 6100
 F 0 "R10" V 7525 6075 50  0000 L CNN
-F 1 "100k" V 7625 6000 50  0000 L CNN
+F 1 "500k" V 7625 6000 50  0000 L CNN
 F 2 "" V 7555 6100 50  0001 C CNN
 F 3 "~" H 7625 6100 50  0001 C CNN
@@
 P 6075 1900
 F 0 "I1" H 6305 1946 50  0000 L CNN
-F 1 "0.15m" H 6305 1855 50  0000 L CNN
+F 1 "0.01m" H 6305 1855 50  0000 L CNN
 F 2 "" H 6075 1900 50  0001 C CNN
 F 3 "~" H 6075 1900 50  0001 C CNN
@@
 Wire Wire Line
 	7275 5400 7350 5400
-$Comp
-L Device:R R1
-U 1 1 5E6485C0
-P 6975 3550
-F 0 "R1" H 6825 3550 50  0000 L CNN
-F 1 "1000Meg" V 6975 3475 50  0000 L CNN
-F 2 "Resistor_SMD:R_0805_2012Metric_Pad1.15x1.40mm_HandSolder" V 6905 3550 50  0001 C CNN
-F 3 "~" H 6975 3550 50  0001 C CNN
-	1    6975 3550
-	1    0    0    1
-$EndComp
-Wire Wire Line
-	6975 3400 6975 3175
 $Comp
 L Device:C C6
@@
 	0    1    1    0
 $EndComp
-Wire Wire Line
-	6975 2875 6975 2650
 $Comp
 L power:VEE #PWR05
@@
 	7275 5025 7275 5000
 Wire Wire Line
-	6975 4700 7950 4700
-Wire Wire Line
-	6975 2650 6675 2650
-Connection ~ 6675 2650
-$Comp
-L Device:C C7
-U 1 1 5E65CF72
-P 6975 3025
-F 0 "C7" H 6860 2979 50  0000 R CNN
-F 1 "1u" H 6860 3070 50  0000 R CNN
-F 2 "" H 7013 2875 50  0001 C CNN
-F 3 "~" H 6975 3025 50  0001 C CNN
-	1    6975 3025
-	-1   0    0    1
-$EndComp
-Wire Wire Line
 	3650 3525 4375 3525
 $Comp
@@
 P 7275 5150
 F 0 "R9" H 7325 5100 50  0000 L CNN
-F 1 "100k" V 7275 5050 50  0000 L CNN
+F 1 "500k" V 7275 5050 50  0000 L CNN
 F 2 "" V 7205 5150 50  0001 C CNN
 F 3 "~" H 7275 5150 50  0001 C CNN
@@
 	-1   0    0    1
 $EndComp
-$Comp
-L Device:R R8
-U 1 1 5D9923C5
-P 7050 5600
-F 0 "R8" V 7150 5575 50  0000 L CNN
-F 1 "220" V 7050 5500 50  0000 L CNN
-F 2 "" V 6980 5600 50  0001 C CNN
-F 3 "~" H 7050 5600 50  0001 C CNN
-	1    7050 5600
-	0    1    1    0
-$EndComp
-$Comp
-L Device:R R7
-U 1 1 5D98E38E
-P 7050 5400
-F 0 "R7" V 6950 5375 50  0000 L CNN
-F 1 "220" V 7050 5300 50  0000 L CNN
-F 2 "" V 6980 5400 50  0001 C CNN
-F 3 "~" H 7050 5400 50  0001 C CNN
-	1    7050 5400
-	0    1    1    0
-$EndComp
 Wire Wire Line
 	7950 6100 7950 5500
-Wire Wire Line
-	7950 5500 7950 4700
-Connection ~ 7950 5500
 $Comp
 L pspice:OPAMP U2
@@
 Text Notes 7050 3975 0    50   ~ 0
 resonance control.\n(good resonance at 50k-100k)
+$Comp
+L Device:R R7
+U 1 1 5D98E38E
+P 7050 5400
+F 0 "R7" V 6950 5375 50  0000 L CNN
+F 1 "1k" V 7050 5300 50  0000 L CNN
+F 2 "" V 6980 5400 50  0001 C CNN
+F 3 "~" H 7050 5400 50  0001 C CNN
+	1    7050 5400
+	0    1    1    0
+$EndComp
+$Comp
+L Device:R R8
+U 1 1 5D9923C5
+P 7050 5600
+F 0 "R8" V 7150 5575 50  0000 L CNN
+F 1 "1k" V 7050 5500 50  0000 L CNN
+F 2 "" V 6980 5600 50  0001 C CNN
+F 3 "~" H 7050 5600 50  0001 C CNN
+	1    7050 5600
+	0    1    1    0
+$EndComp
+Text Notes 7175 6300 0    50   ~ 0
+ca 6 uA
+Text Notes 6375 6325 0    50   ~ 0
+ca 0.5* I1 each
+Text Notes 6650 6475 0    50   ~ 0
+diff1,2 = -3.3V ca
+Text GLabel 5475 5950 0    50   Input ~ 0
+foo
+Text Notes 5050 5975 0    50   ~ 0
+-3.9V
+Wire Wire Line
+	6900 5400 6900 5450
+Wire Wire Line
+	6900 5550 6900 5600
 $EndSCHEMATC
