File: simulation/vcf/vcf_buffered_bjt.sch (KiCad schematic (older format))
At the start: 38 parts, among them Q10 BC557B, Q101 BC557B, Q102 BC557B, Q11 BC557B, Q12 BC557B, Q2 BC557B, Q4 BC557B, Q5 BC557B, Q6 BC557B, Q7 BC557B, Q8 BC557B, Q9 BC557B, U2 LM324

Commit message: Use TL074, not LM324 in vcf simulation
Parts:
- U2: value LM324 -> TL074; Spice_Lib_File /home/flo/analog-synth/simulation/lib/LM324.ti.lib -> /home/flo/analog-synth/simulation/lib/TL074.ti.lib; Spice_Model LM324 -> TL074
Changed lines of the file:
@@
 P 9975 5575
 F 0 "U2" H 10100 5475 50  0000 L CNN
-F 1 "LM324" H 9975 5375 50  0000 L CNN
+F 1 "TL074" H 9975 5375 50  0000 L CNN
 F 2 "" H 9975 5575 50  0001 C CNN
 F 3 "~" H 9975 5575 50  0001 C CNN
 F 4 "X" H 9975 5575 50  0001 C CNN "Spice_Primitive"
-F 5 "LM324" H 9975 5575 50  0001 C CNN "Spice_Model"
+F 5 "TL074" H 9975 5575 50  0001 C CNN "Spice_Model"
 F 6 "Y" H 9975 5575 50  0001 C CNN "Spice_Netlist_Enabled"
-F 7 "/home/flo/analog-synth/simulation/lib/LM324.ti.lib" H 9975 5575 50  0001 C CNN "Spice_Lib_File"
+F 7 "/home/flo/analog-synth/simulation/lib/TL074.ti.lib" H 9975 5575 50  0001 C CNN "Spice_Lib_File"
 F 8 "1,2,4,5,3" H 9975 5575 50  0001 C CNN "Spice_Node_Sequence"
 	1    9975 5575
