File: simulation/vcf/vcf_buffered_opamp.sch (KiCad schematic (older format))
At the start: 34 parts, among them Q10 BC557B, Q11 BC557B, Q12 BC557B, Q2 BC557B, Q4 BC557B, Q5 BC557B, Q6 BC557B, Q7 BC557B, Q8 BC557B, Q9 BC557B, U2 LM324

Commit message: Plot tooling and schematics for VCF simulation
Parts:
- added U? (x2): LM324, symbol pspice:OPAMP
- V4: value PULSE(-2 2 0 0m 0m 2m 4m) -> SIN(0 2 1000)
Connections:
- net VCC: now also U?.4 (V+), U?.4 (V+)
- net VEE: now also U?.5 (V-), U?.5 (V-)
- net diff1: now also U?.2 (-), U?.3; no longer C5.1, Q12.3 (E), Q4.1 (C)
- net diff2: now also U?.2 (-), U?.3; no longer C5.2, Q2.1 (C), Q8.3 (E)
- new net: C5.1, Q12.3 (E), Q4.1 (C), U?.1 (+)
- new net: C5.2, Q2.1 (C), Q8.3 (E), U?.1 (+)
Other:
- note removed: ".tran 10u 30m"
- moved on the sheet: R10, R7, R8, R9, U2

Commit message: Use TL074, not LM324 in vcf simulation
Parts:
- U2, U? (x2): value LM324 -> TL074; Spice_Lib_File /home/flo/analog-synth/simulation/lib/LM324.ti.lib -> /home/flo/analog-synth/simulation/lib/TL074.ti.lib; Spice_Model LM324 -> TL074
Changed lines of the file:
@@
 P 9975 5575
 F 0 "U2" H 10100 5475 50  0000 L CNN
-F 1 "LM324" H 9975 5375 50  0000 L CNN
+F 1 "TL074" H 9975 5375 50  0000 L CNN
 F 2 "" H 9975 5575 50  0001 C CNN
 F 3 "~" H 9975 5575 50  0001 C CNN
 F 4 "X" H 9975 5575 50  0001 C CNN "Spice_Primitive"
-F 5 "LM324" H 9975 5575 50  0001 C CNN "Spice_Model"
+F 5 "TL074" H 9975 5575 50  0001 C CNN "Spice_Model"
 F 6 "Y" H 9975 5575 50  0001 C CNN "Spice_Netlist_Enabled"
-F 7 "/home/flo/analog-synth/simulation/lib/LM324.ti.lib" H 9975 5575 50  0001 C CNN "Spice_Lib_File"
+F 7 "/home/flo/analog-synth/simulation/lib/TL074.ti.lib" H 9975 5575 50  0001 C CNN "Spice_Lib_File"
 F 8 "1,2,4,5,3" H 9975 5575 50  0001 C CNN "Spice_Node_Sequence"
 	1    9975 5575
@@
 P 7525 4725
 F 0 "U?" H 7650 4625 50  0000 L CNN
-F 1 "LM324" H 7525 4525 50  0000 L CNN
+F 1 "TL074" H 7525 4525 50  0000 L CNN
 F 2 "" H 7525 4725 50  0001 C CNN
 F 3 "~" H 7525 4725 50  0001 C CNN
 F 4 "X" H 7525 4725 50  0001 C CNN "Spice_Primitive"
-F 5 "LM324" H 7525 4725 50  0001 C CNN "Spice_Model"
+F 5 "TL074" H 7525 4725 50  0001 C CNN "Spice_Model"
 F 6 "Y" H 7525 4725 50  0001 C CNN "Spice_Netlist_Enabled"
-F 7 "/home/flo/analog-synth/simulation/lib/LM324.ti.lib" H 7525 4725 50  0001 C CNN "Spice_Lib_File"
+F 7 "/home/flo/analog-synth/simulation/lib/TL074.ti.lib" H 7525 4725 50  0001 C CNN "Spice_Lib_File"
 F 8 "1,2,4,5,3" H 7525 4725 50  0001 C CNN "Spice_Node_Sequence"
 	1    7525 4725
@@
 P 7525 5650
 F 0 "U?" H 7650 5550 50  0000 L CNN
-F 1 "LM324" H 7525 5450 50  0000 L CNN
+F 1 "TL074" H 7525 5450 50  0000 L CNN
 F 2 "" H 7525 5650 50  0001 C CNN
 F 3 "~" H 7525 5650 50  0001 C CNN
 F 4 "X" H 7525 5650 50  0001 C CNN "Spice_Primitive"
-F 5 "LM324" H 7525 5650 50  0001 C CNN "Spice_Model"
+F 5 "TL074" H 7525 5650 50  0001 C CNN "Spice_Model"
 F 6 "Y" H 7525 5650 50  0001 C CNN "Spice_Netlist_Enabled"
-F 7 "/home/flo/analog-synth/simulation/lib/LM324.ti.lib" H 7525 5650 50  0001 C CNN "Spice_Lib_File"
+F 7 "/home/flo/analog-synth/simulation/lib/TL074.ti.lib" H 7525 5650 50  0001 C CNN "Spice_Lib_File"
 F 8 "1,2,4,5,3" H 7525 5650 50  0001 C CNN "Spice_Node_Sequence"
 	1    7525 5650
