File: simulation/vcf/vcf_unbuffered_capacitors1.sch (KiCad schematic (older format))
At the start: 36 parts, among them Q10 BC557B, Q11 BC557B, Q12 BC557B, Q2 BC557B, Q4 BC557B, Q5 BC557B, Q6 BC557B, Q7 BC557B, Q8 BC557B, Q9 BC557B, U2 LM324

Commit message: vcf_unbuffered_capacitors* now correctly reflect patch2
Parts:
- C102: value 27p -> 2.2n
Changed lines of the file:
@@
 P 7625 6250
 F 0 "C102" V 7725 6050 50  0000 L CNN
-F 1 "27p" V 7725 6325 50  0000 L CNN
+F 1 "2.2n" V 7725 6325 50  0000 L CNN
 F 2 "" H 7625 6250 50  0001 C CNN
 F 3 "~" H 7625 6250 50  0001 C CNN

Commit message: Use TL074, not LM324 in vcf simulation
Parts:
- U2: value LM324 -> TL074; Spice_Lib_File /home/flo/analog-synth/simulation/lib/LM324.ti.lib -> /home/flo/analog-synth/simulation/lib/TL074.ti.lib; Spice_Model LM324 -> TL074
Changed lines of the file:
@@
 P 7650 5500
 F 0 "U2" H 7775 5400 50  0000 L CNN
-F 1 "LM324" H 7650 5300 50  0000 L CNN
+F 1 "TL074" H 7650 5300 50  0000 L CNN
 F 2 "" H 7650 5500 50  0001 C CNN
 F 3 "~" H 7650 5500 50  0001 C CNN
 F 4 "X" H 7650 5500 50  0001 C CNN "Spice_Primitive"
-F 5 "LM324" H 7650 5500 50  0001 C CNN "Spice_Model"
+F 5 "TL074" H 7650 5500 50  0001 C CNN "Spice_Model"
 F 6 "Y" H 7650 5500 50  0001 C CNN "Spice_Netlist_Enabled"
-F 7 "/home/flo/analog-synth/simulation/lib/LM324.ti.lib" H 7650 5500 50  0001 C CNN "Spice_Lib_File"
+F 7 "/home/flo/analog-synth/simulation/lib/TL074.ti.lib" H 7650 5500 50  0001 C CNN "Spice_Lib_File"
 F 8 "1,2,4,5,3" H 7650 5500 50  0001 C CNN "Spice_Node_Sequence"
 	1    7650 5500
