File: simulation/vca/vca.sch (KiCad schematic (older format))
At the start: 20 parts, among them Q1 BC557B, Q2 BC557B, Q3 BC557B, Q4 BC557B, U2 LM324

Commit message: Changed VCA simulation
Parts:
- R1: value 10k -> 22k
- R10, R9: value 68k -> 50k
- R7, R8: value 100k -> 10k
- V3: value 0 -> PULSE(-5 5 0 2m 2m 0.02m 4m)
- V4: value PULSE(-2 2 0 1m 1m 0.01m 2m) -> PULSE(-2 2 0 0.1m 0.1m 0.001m 0.2m)
Other:
- note added: ".tran 1u 10m"
- note removed: ".tran 10u 10m"
Changed lines of the file:
@@
 Wire Wire Line
 	8200 2825 8275 2825
-$Comp
-L Device:R R7
-U 1 1 5D98E38E
-P 8050 2625
-F 0 "R7" V 7950 2600 50  0000 L CNN
-F 1 "100k" V 8050 2525 50  0000 L CNN
-F 2 "" V 7980 2625 50  0001 C CNN
-F 3 "~" H 8050 2625 50  0001 C CNN
-	1    8050 2625
-	0    1    1    0
-$EndComp
-$Comp
-L Device:R R8
-U 1 1 5D9923C5
-P 8050 2825
-F 0 "R8" V 8150 2800 50  0000 L CNN
-F 1 "100k" V 8050 2725 50  0000 L CNN
-F 2 "" V 7980 2825 50  0001 C CNN
-F 3 "~" H 8050 2825 50  0001 C CNN
-	1    8050 2825
-	0    1    1    0
-$EndComp
-$Comp
-L Device:R R10
-U 1 1 5D992BCF
-P 8625 3325
-F 0 "R10" V 8525 3300 50  0000 L CNN
-F 1 "68k" V 8625 3225 50  0000 L CNN
-F 2 "" V 8555 3325 50  0001 C CNN
-F 3 "~" H 8625 3325 50  0001 C CNN
-	1    8625 3325
-	0    1    1    0
-$EndComp
 Wire Wire Line
 	8275 2825 8275 3325
@@
 Wire Wire Line
 	8950 3325 8950 2725
-$Comp
-L Device:R R9
-U 1 1 5D9941E7
-P 8275 2375
-F 0 "R9" H 8100 2325 50  0000 L CNN
-F 1 "68k" V 8275 2275 50  0000 L CNN
-F 2 "" V 8205 2375 50  0001 C CNN
-F 3 "~" H 8275 2375 50  0001 C CNN
-	1    8275 2375
-	-1   0    0    1
-$EndComp
 Wire Wire Line
 	8275 2525 8275 2625
@@
 $EndComp
 $Comp
-L Device:R R1
-U 1 1 5D94CF4E
-P 5775 1600
-F 0 "R1" V 5675 1550 50  0000 L CNN
-F 1 "10k" V 5775 1525 50  0000 L CNN
-F 2 "" V 5705 1600 50  0001 C CNN
-F 3 "~" H 5775 1600 50  0001 C CNN
-	1    5775 1600
-	0    1    1    0
-$EndComp
-$Comp
-L Device:R R4
-U 1 1 5D97C329
-P 6675 3000
-F 0 "R4" H 6745 3046 50  0000 L CNN
-F 1 "10k" V 6675 2925 50  0000 L CNN
-F 2 "" V 6605 3000 50  0001 C CNN
-F 3 "~" H 6675 3000 50  0001 C CNN
-	1    6675 3000
-	1    0    0    1
-$EndComp
-$Comp
 L power:VEE #PWR07
 U 1 1 5D9809F3
@@
 $EndComp
 Text Notes 10200 650  0    50   ~ 0
-.tran 10u 10m
+.tran 1u 10m
 $Comp
 L pspice:VSOURCE V1
@@
 P 4450 1900
 F 0 "V3" H 4050 2000 50  0000 L CNN
-F 1 "0" H 4050 1750 50  0000 L CNN
+F 1 "PULSE(-5 5 0 2m 2m 0.02m 4m)" H 4050 1750 50  0000 L CNN
 F 2 "" H 4450 1900 50  0001 C CNN
 F 3 "~" H 4450 1900 50  0001 C CNN
 	1    4450 1900
-	1    0    0    -1
-$EndComp
-$Comp
-L pspice:VSOURCE V4
-U 1 1 5E4DBEAC
-P 5100 2550
-F 0 "V4" H 4700 2650 50  0000 L CNN
-F 1 "PULSE(-2 2 0 1m 1m 0.01m 2m)" H 4675 1900 50  0000 L CNN
-F 2 "" H 5100 2550 50  0001 C CNN
-F 3 "~" H 5100 2550 50  0001 C CNN
-	1    5100 2550
 	1    0    0    -1
 $EndComp
@@
 Wire Wire Line
 	6675 1900 6825 1900
+Connection ~ 6825 1900
+Wire Wire Line
+	6825 1900 6975 1900
+Wire Wire Line
+	6975 2825 7900 2825
+Wire Wire Line
+	6675 2625 7900 2625
+$Comp
+L Device:R R10
+U 1 1 5D992BCF
+P 8625 3325
+F 0 "R10" V 8525 3300 50  0000 L CNN
+F 1 "50k" V 8625 3225 50  0000 L CNN
+F 2 "" V 8555 3325 50  0001 C CNN
+F 3 "~" H 8625 3325 50  0001 C CNN
+	1    8625 3325
+	0    1    1    0
+$EndComp
+$Comp
+L Device:R R9
+U 1 1 5D9941E7
+P 8275 2375
+F 0 "R9" H 8100 2325 50  0000 L CNN
+F 1 "50k" V 8275 2275 50  0000 L CNN
+F 2 "" V 8205 2375 50  0001 C CNN
+F 3 "~" H 8275 2375 50  0001 C CNN
+	1    8275 2375
+	-1   0    0    1
+$EndComp
+$Comp
+L Device:R R1
+U 1 1 5D94CF4E
+P 5775 1600
+F 0 "R1" V 5675 1550 50  0000 L CNN
+F 1 "22k" V 5775 1525 50  0000 L CNN
+F 2 "" V 5705 1600 50  0001 C CNN
+F 3 "~" H 5775 1600 50  0001 C CNN
+	1    5775 1600
+	0    1    1    0
+$EndComp
 $Comp
 L Device:R R5
@@
 	-1   0    0    -1
 $EndComp
-Connection ~ 6825 1900
-Wire Wire Line
-	6825 1900 6975 1900
 $Comp
 L Device:R R6
@@
 	1    0    0    1
 $EndComp
-Wire Wire Line
-	6975 2825 7900 2825
-Wire Wire Line
-	6675 2625 7900 2625
+$Comp
+L Device:R R4
+U 1 1 5D97C329
+P 6675 3000
+F 0 "R4" H 6745 3046 50  0000 L CNN
+F 1 "10k" V 6675 2925 50  0000 L CNN
+F 2 "" V 6605 3000 50  0001 C CNN
+F 3 "~" H 6675 3000 50  0001 C CNN
+	1    6675 3000
+	1    0    0    1
+$EndComp
+$Comp
+L Device:R R8
+U 1 1 5D9923C5
+P 8050 2825
+F 0 "R8" V 8150 2800 50  0000 L CNN
+F 1 "10k" V 8050 2725 50  0000 L CNN
+F 2 "" V 7980 2825 50  0001 C CNN
+F 3 "~" H 8050 2825 50  0001 C CNN
+	1    8050 2825
+	0    1    1    0
+$EndComp
+$Comp
+L Device:R R7
+U 1 1 5D98E38E
+P 8050 2625
+F 0 "R7" V 7950 2600 50  0000 L CNN
+F 1 "10k" V 8050 2525 50  0000 L CNN
+F 2 "" V 7980 2625 50  0001 C CNN
+F 3 "~" H 8050 2625 50  0001 C CNN
+	1    8050 2625
+	0    1    1    0
+$EndComp
+$Comp
+L pspice:VSOURCE V4
+U 1 1 5E4DBEAC
+P 5100 2550
+F 0 "V4" H 4700 2650 50  0000 L CNN
+F 1 "PULSE(-2 2 0 0.1m 0.1m 0.001m 0.2m)" H 4675 1900 50  0000 L CNN
+F 2 "" H 5100 2550 50  0001 C CNN
+F 3 "~" H 5100 2550 50  0001 C CNN
+	1    5100 2550
+	1    0    0    -1
+$EndComp
 $EndSCHEMATC
