File: simulation/vca2/vca.sch (KiCad schematic (older format))
At the start: 34 parts, among them Q1 BC557B, Q2 BC557B, Q3 BC557B, Q4 BC557B, Q5 BC557B, Q6 BC557B, Q7 BC557B, Q8 BC557B, U1 LM324, U2 LM324

Commit message: vca simulation++
Parts:
- removed Q1: BC557B, symbol pspice:QPNP
- removed R1: 22k, symbol Device:R
- added R?: 10k, symbol Device:R
- R17, R18: value 22k -> 33k
- V3: value PULSE(-5 5 0 10m 10m 0.01m 20m) -> PULSE(4.37 4.45 0 10m 10m 0.01m 20m)
Connections:
- net cv_pregain: now also R?.2
- net at Q3.2 (B): now also R?.1

Commit message: changed vca2 to exponential input
Parts:
- removed Q5, Q7: BC557B, symbol pspice:QPNP
- added Q1: BC557B, symbol pspice:QPNP
- added R19, R20: 1k, symbol Device:R
- R11: value 22k -> 10k
- V3: value PULSE(4.37 4.45 0 10m 10m 0.01m 20m) -> PULSE(-2 0 0 10m 10m 0.01m 20m)
- V5: value PULSE(0 5 0 0.5m 0.5m 0.1m 4m) -> PULSE(-1.5 -1.5 0 0.5m 0.5m 0.1m 4m)
- gave numbers to parts that had none: 1
Connections:
- net VCC: now also Q1.3 (E), R19.2, R20.2
- net cv_pregain2: now reaches Q3.2 (B), R1.1
- net cv_pregain2: now also R19.1
- net cv_postgain2: now reaches R11.1
- net cv_postgain2: now also Q1.2 (B), R20.1
- net at R13.1: now also Q1.1 (C)
Other:
- note removed: "Control voltage:\nVCC=closed"
Changed lines of the file:
@@
 L power:VCC #PWR03
 U 1 1 5D942900
-P 6375 850
-F 0 "#PWR03" H 6375 700 50  0001 C CNN
-F 1 "VCC" H 6392 1023 50  0000 C CNN
-F 2 "" H 6375 850 50  0001 C CNN
-F 3 "" H 6375 850 50  0001 C CNN
-	1    6375 850
+P 5950 700
+F 0 "#PWR03" H 5950 550 50  0001 C CNN
+F 1 "VCC" H 5967 873 50  0000 C CNN
+F 2 "" H 5950 700 50  0001 C CNN
+F 3 "" H 5950 700 50  0001 C CNN
+	1    5950 700
 	1    0    0    -1
 $EndComp
@@
 $EndComp
 Wire Wire Line
-	6375 1250 6375 1600
-Wire Wire Line
 	6825 850  6825 900
-Wire Wire Line
-	6375 850  6825 850
 $Comp
 L Device:R R3
@@
 Wire Wire Line
 	8350 2625 8275 2625
-Text Notes 6925 4250 0    50   ~ 0
-current mirror as\nvoltage controlled\ncurrent source
-$Comp
-L power:VCC #PWR013
-U 1 1 601FFDF6
-P 6375 3775
-F 0 "#PWR013" H 6375 3625 50  0001 C CNN
-F 1 "VCC" H 6392 3948 50  0000 C CNN
-F 2 "" H 6375 3775 50  0001 C CNN
-F 3 "" H 6375 3775 50  0001 C CNN
-	1    6375 3775
-	1    0    0    -1
-$EndComp
-$Comp
-L pspice:QPNP Q7
-U 1 1 601FFE12
-P 6675 4175
-F 0 "Q7" H 6575 4475 50  0000 L CNN
-F 1 "BC557B" H 6225 4325 50  0001 L CNN
-F 2 "" H 6675 4175 50  0001 C CNN
-F 3 "~" H 6675 4175 50  0001 C CNN
-F 4 "Q" H 6675 4175 50  0001 C CNN "Spice_Primitive"
-F 5 "BC557b" H 6675 4175 50  0001 C CNN "Spice_Model"
-F 6 "Y" H 6675 4175 50  0001 C CNN "Spice_Netlist_Enabled"
-F 7 "/home/flo/analog-synth/simulation/lib/BC547_557.lib" H 6675 4175 50  0001 C CNN "Spice_Lib_File"
-	1    6675 4175
-	1    0    0    1
-$EndComp
-Wire Wire Line
-	6375 4175 6375 4525
-Wire Wire Line
-	6825 3775 6825 3825
-Wire Wire Line
-	6375 3775 6825 3775
-Text Notes 5175 4400 0    50   ~ 0
-Control voltage:\nVCC=closed
 Text GLabel 4825 4525 1    50   Input ~ 0
 cv_postgain
@@
 Text GLabel 5000 5200 3    50   Input ~ 0
 signal_intermediate
-Wire Wire Line
-	4450 4525 5625 4525
-Wire Wire Line
-	6375 4525 5925 4525
-$Comp
-L Device:R R11
-U 1 1 601FFE33
-P 5775 4525
-F 0 "R11" V 5675 4475 50  0000 L CNN
-F 1 "22k" V 5775 4450 50  0000 L CNN
-F 2 "" V 5705 4525 50  0001 C CNN
-F 3 "~" H 5775 4525 50  0001 C CNN
-	1    5775 4525
-	0    1    1    0
-$EndComp
 $Comp
 L pspice:VSOURCE V5
@@
 P 4450 4825
 F 0 "V5" H 4050 4925 50  0000 L CNN
-F 1 "PULSE(0 5 0 0.5m 0.5m 0.1m 4m)" H 2975 4500 50  0000 L CNN
+F 1 "PULSE(-1.5 -1.5 0 0.5m 0.5m 0.1m 4m)" H 2975 4500 50  0000 L CNN
 F 2 "" H 4450 4825 50  0001 C CNN
 F 3 "~" H 4450 4825 50  0001 C CNN
@@
 	1    0    0    -1
 $EndComp
-Connection ~ 6375 3775
-Wire Wire Line
-	5925 3775 6375 3775
-Wire Wire Line
-	5925 3825 5925 3775
-Connection ~ 6375 4175
-Connection ~ 5925 4525
-$Comp
-L pspice:QPNP Q5
-U 1 1 601FFE04
-P 6075 4175
-F 0 "Q5" H 5975 4475 50  0000 L CNN
-F 1 "BC557B" H 5625 4050 50  0000 L CNN
-F 2 "" H 6075 4175 50  0001 C CNN
-F 3 "~" H 6075 4175 50  0001 C CNN
-F 4 "Q" H 6075 4175 50  0001 C CNN "Spice_Primitive"
-F 5 "BC557b" H 6075 4175 50  0001 C CNN "Spice_Model"
-F 6 "Y" H 6075 4175 50  0001 C CNN "Spice_Netlist_Enabled"
-F 7 "/home/flo/analog-synth/simulation/lib/BC547_557.lib" H 6075 4175 50  0001 C CNN "Spice_Lib_File"
-	1    6075 4175
-	-1   0    0    1
-$EndComp
-Wire Wire Line
-	4450 1600 5025 1600
-Wire Wire Line
-	5025 1600 5025 2175
-Wire Wire Line
-	5025 2175 4625 2175
-Wire Wire Line
-	4625 2175 4625 2725
-Wire Wire Line
-	4625 2725 4125 2725
-$Comp
-L Device:R R?
+Wire Wire Line
+	5825 1600 5950 1600
+Wire Wire Line
+	6375 1025 5950 1025
+Wire Wire Line
+	5950 1025 5950 1000
+Wire Wire Line
+	6375 1025 6375 1250
+Wire Wire Line
+	5950 1025 5950 1600
+Connection ~ 5950 1025
+Text GLabel 5950 1275 0    50   Input ~ 0
+cv_pregain2
+$Comp
+L power:VCC #PWR022
+U 1 1 6025EFEC
+P 6825 850
+F 0 "#PWR022" H 6825 700 50  0001 C CNN
+F 1 "VCC" H 6842 1023 50  0000 C CNN
+F 2 "" H 6825 850 50  0001 C CNN
+F 3 "" H 6825 850 50  0001 C CNN
+	1    6825 850
+	1    0    0    -1
+$EndComp
+Wire Wire Line
+	4450 1600 5525 1600
+$Comp
+L Device:R R19
+U 1 1 6024AD39
+P 5950 850
+F 0 "R19" H 6020 896 50  0000 L CNN
+F 1 "1k" V 5950 775 50  0000 L CNN
+F 2 "" V 5880 850 50  0001 C CNN
+F 3 "~" H 5950 850 50  0001 C CNN
+	1    5950 850
+	1    0    0    1
+$EndComp
+$Comp
+L Device:R R1
 U 1 1 60243ADC
 P 5675 1600
-F 0 "R?" H 5745 1646 50  0000 L CNN
+F 0 "R1" H 5745 1646 50  0000 L CNN
 F 1 "10k" V 5675 1525 50  0000 L CNN
 F 2 "" V 5605 1600 50  0001 C CNN
@@
 	0    1    -1   0
 $EndComp
-Connection ~ 5025 1600
-Wire Wire Line
-	5525 1600 5025 1600
-Wire Wire Line
-	5825 1600 6375 1600
 $Comp
 L pspice:VSOURCE V3
@@
 P 4450 1900
 F 0 "V3" H 4050 2000 50  0000 L CNN
-F 1 "PULSE(4.37 4.45 0 10m 10m 0.01m 20m)" H 2975 1575 50  0000 L CNN
+F 1 "PULSE(-2 0 0 10m 10m 0.01m 20m)" H 2975 1575 50  0000 L CNN
 F 2 "" H 4450 1900 50  0001 C CNN
 F 3 "~" H 4450 1900 50  0001 C CNN
@@
 	1    0    0    -1
 $EndComp
+Text Notes 6925 4250 0    50   ~ 0
+current mirror as\nvoltage controlled\ncurrent source
+$Comp
+L power:VCC #PWR013
+U 1 1 602674B9
+P 5950 3625
+F 0 "#PWR013" H 5950 3475 50  0001 C CNN
+F 1 "VCC" H 5967 3798 50  0000 C CNN
+F 2 "" H 5950 3625 50  0001 C CNN
+F 3 "" H 5950 3625 50  0001 C CNN
+	1    5950 3625
+	1    0    0    -1
+$EndComp
+$Comp
+L pspice:QPNP Q1
+U 1 1 602674C7
+P 6675 4175
+F 0 "Q1" H 6575 4475 50  0000 L CNN
+F 1 "BC557B" H 6225 4325 50  0001 L CNN
+F 2 "" H 6675 4175 50  0001 C CNN
+F 3 "~" H 6675 4175 50  0001 C CNN
+F 4 "Q" H 6675 4175 50  0001 C CNN "Spice_Primitive"
+F 5 "BC557b" H 6675 4175 50  0001 C CNN "Spice_Model"
+F 6 "Y" H 6675 4175 50  0001 C CNN "Spice_Netlist_Enabled"
+F 7 "/home/flo/analog-synth/simulation/lib/BC547_557.lib" H 6675 4175 50  0001 C CNN "Spice_Lib_File"
+	1    6675 4175
+	1    0    0    1
+$EndComp
+Wire Wire Line
+	6825 3775 6825 3825
+Wire Wire Line
+	6375 3950 5950 3950
+Wire Wire Line
+	5950 3950 5950 3925
+Wire Wire Line
+	6375 3950 6375 4175
+Wire Wire Line
+	5950 3950 5950 4525
+Connection ~ 5950 3950
+Text GLabel 5950 4200 0    50   Input ~ 0
+cv_postgain2
+$Comp
+L power:VCC #PWR023
+U 1 1 602674D8
+P 6825 3775
+F 0 "#PWR023" H 6825 3625 50  0001 C CNN
+F 1 "VCC" H 6842 3948 50  0000 C CNN
+F 2 "" H 6825 3775 50  0001 C CNN
+F 3 "" H 6825 3775 50  0001 C CNN
+	1    6825 3775
+	1    0    0    -1
+$EndComp
+$Comp
+L Device:R R20
+U 1 1 602674E2
+P 5950 3775
+F 0 "R20" H 6020 3821 50  0000 L CNN
+F 1 "1k" V 5950 3700 50  0000 L CNN
+F 2 "" V 5880 3775 50  0001 C CNN
+F 3 "~" H 5950 3775 50  0001 C CNN
+	1    5950 3775
+	1    0    0    1
+$EndComp
+$Comp
+L Device:R R11
+U 1 1 602674EC
+P 5675 4525
+F 0 "R11" H 5745 4571 50  0000 L CNN
+F 1 "10k" V 5675 4450 50  0000 L CNN
+F 2 "" V 5605 4525 50  0001 C CNN
+F 3 "~" H 5675 4525 50  0001 C CNN
+	1    5675 4525
+	0    1    -1   0
+$EndComp
+Wire Wire Line
+	5825 4525 5950 4525
+Wire Wire Line
+	4450 4525 5525 4525
 $EndSCHEMATC

Commit message: vca with voltage controlled distortion that does not affect volume
Parts:
- added Q?: BC557B, symbol pspice:QPNP
- added R21, R22, R24: 10k, symbol Device:R
- added R23: 15k, symbol Device:R
- added R?: 1k, symbol Device:R
- added U3, U?: LM324, symbol pspice:OPAMP
- added V6: 2, symbol pspice:VSOURCE
- added V?: -0.8, symbol pspice:VSOURCE
- V5: value PULSE(-1.5 -1.5 0 0.5m 0.5m 0.1m 4m) -> PULSE(1.5 1.5 0 0.5m 0.5m 0.1m 4m)
Connections:
- net 0: now also U3.1 (+), V6.2 (E2), V?.2 (E2)
- net VCC: now also U3.4 (V+), U?.4 (V+)
- net VEE: now also U3.5 (V-), U?.5 (V-)
- net cv_postgain: now also R22.1, U3.3; no longer V5.1 (E1)
- net cv_pregain: now also R?.1
- new net: R21.2, V5.1 (E1)
- new net: R21.1, R22.2, R23.1, R24.1, U3.2 (-)
- new net: R24.2, U?.2 (-), U?.3
- new net: R23.2, V6.1 (E1)
- new net: Q?.3 (E), V?.1 (E1)
- new net cv_pregain_clamped: Q?.1 (C), Q?.2 (B), R?.2, U?.1 (+)
Other:
- moved on the sheet: V5

Commit message: that opamp buffer seems unneeded
Parts:
- removed U?: LM324, symbol pspice:OPAMP
- R24: value 10k -> 9k
- V5: value PULSE(1.5 1.5 0 0.5m 0.5m 0.1m 4m) -> PULSE(1.5 1.5 0 5.9m 0.01m 0.01m 6m)
- V?: value -0.8 -> -0.66
Connections:
- net cv_pregain_clamped: now also R24.2
Changed lines of the file:
@@
 Text GLabel 5000 5200 3    50   Input ~ 0
 signal_intermediate
-$Comp
-L pspice:VSOURCE V5
-U 1 1 601FFE26
-P 3200 4925
-F 0 "V5" H 2800 5025 50  0000 L CNN
-F 1 "PULSE(1.5 1.5 0 0.5m 0.5m 0.1m 4m)" H 1725 4600 50  0000 L CNN
-F 2 "" H 3200 4925 50  0001 C CNN
-F 3 "~" H 3200 4925 50  0001 C CNN
-	1    3200 4925
-	1    0    0    -1
-$EndComp
 Wire Wire Line
 	5825 1600 5950 1600
@@
 	1    0    0    -1
 $EndComp
-Text Notes 6925 4250 0    50   ~ 0
-current mirror as\nvoltage controlled\ncurrent source
 $Comp
 L power:VCC #PWR013
@@
 	0    1    -1   0
 $EndComp
-Wire Wire Line
-	3850 4625 3750 4625
 $Comp
 L power:GND #PWR027
@@
 P 3275 3825
 F 0 "R24" V 3150 3775 50  0000 L CNN
-F 1 "10k" V 3275 3750 50  0000 L CNN
+F 1 "9k" V 3275 3750 50  0000 L CNN
 F 2 "" V 3205 3825 50  0001 C CNN
 F 3 "~" H 3275 3825 50  0001 C CNN
@@
 	0    1    -1   0
 $EndComp
-Wire Wire Line
-	3750 4625 3750 4450
-Wire Wire Line
-	3750 4450 3550 4450
-Connection ~ 3750 4625
-Wire Wire Line
-	3750 4625 3675 4625
 Text GLabel 925  3425 0    50   Input ~ 0
 cv_pregain
@@
 	3550 4175 3750 4175
 Wire Wire Line
-	3750 4175 3750 4450
-Connection ~ 3750 4450
-Wire Wire Line
 	3425 3825 3750 3825
 Wire Wire Line
 	3750 3825 3750 4175
-Connection ~ 3750 4175
 $Comp
 L Device:R R?
@@
 	0    -1   1    0
 $EndComp
-Wire Wire Line
-	1225 3425 1475 3425
-Connection ~ 1475 3425
-Wire Wire Line
-	1475 3425 2250 3425
 $Comp
 L pspice:VSOURCE V?
@@
 P 800 2300
 F 0 "V?" H 400 2400 50  0000 L CNN
-F 1 "-0.8" H 425 1875 50  0000 L CNN
+F 1 "-0.66" H 425 1875 50  0000 L CNN
 F 2 "" H 800 2300 50  0001 C CNN
 F 3 "~" H 800 2300 50  0001 C CNN
@@
 Text GLabel 2075 3425 1    50   Input ~ 0
 cv_pregain_clamped
-$Comp
-L pspice:OPAMP U?
-U 1 1 602DF9C3
-P 2550 3525
-F 0 "U?" H 2675 3425 50  0000 L CNN
-F 1 "LM324" H 2550 3325 50  0000 L CNN
-F 2 "" H 2550 3525 50  0001 C CNN
-F 3 "~" H 2550 3525 50  0001 C CNN
-F 4 "X" H 2550 3525 50  0001 C CNN "Spice_Primitive"
-F 5 "LM324" H 2550 3525 50  0001 C CNN "Spice_Model"
-F 6 "Y" H 2550 3525 50  0001 C CNN "Spice_Netlist_Enabled"
-F 7 "/home/flo/analog-synth/simulation/lib/LM324.ti.lib" H 2550 3525 50  0001 C CNN "Spice_Lib_File"
-F 8 "1,2,4,5,3" H 2550 3525 50  0001 C CNN "Spice_Node_Sequence"
-	1    2550 3525
-	1    0    0    -1
-$EndComp
-$Comp
-L power:VCC #PWR?
-U 1 1 602DFE9F
-P 2450 3225
-F 0 "#PWR?" H 2450 3075 50  0001 C CNN
-F 1 "VCC" H 2350 3275 50  0000 C CNN
-F 2 "" H 2450 3225 50  0001 C CNN
-F 3 "" H 2450 3225 50  0001 C CNN
-	1    2450 3225
-	-1   0    0    -1
-$EndComp
-$Comp
-L power:VEE #PWR?
-U 1 1 602DFEA9
-P 2450 3825
-F 0 "#PWR?" H 2450 3675 50  0001 C CNN
-F 1 "VEE" H 2550 3875 50  0000 C CNN
-F 2 "" H 2450 3825 50  0001 C CNN
-F 3 "" H 2450 3825 50  0001 C CNN
-	1    2450 3825
-	1    0    0    1
-$EndComp
-Wire Wire Line
-	2250 3625 2250 4025
-Wire Wire Line
-	2250 4025 2850 4025
-Wire Wire Line
-	2850 4025 2850 3525
 Wire Wire Line
 	2850 3525 3125 3525
-Connection ~ 2850 3525
 Wire Wire Line
 	3125 3525 3125 3825
-Wire Wire Line
-	1925 2925 1925 2575
-Wire Wire Line
-	1925 2575 1475 2575
-Connection ~ 1475 2575
 $Comp
 L pspice:QPNP Q?
@@
 Wire Wire Line
 	1475 3250 1475 3275
+Wire Wire Line
+	2850 3425 2850 3525
+$Comp
+L pspice:VSOURCE V5
+U 1 1 601FFE26
+P 3200 4925
+F 0 "V5" H 2800 5025 50  0000 L CNN
+F 1 "PULSE(1.5 1.5 0 5.9m 0.01m 0.01m 6m)" H 1725 4600 50  0000 L CNN
+F 2 "" H 3200 4925 50  0001 C CNN
+F 3 "~" H 3200 4925 50  0001 C CNN
+	1    3200 4925
+	1    0    0    -1
+$EndComp
+Wire Wire Line
+	3850 4625 3750 4625
+Wire Wire Line
+	3750 4625 3675 4625
+Connection ~ 3750 4625
+Connection ~ 3750 4175
+Wire Wire Line
+	3750 4175 3750 4625
+Wire Wire Line
+	1475 3425 2850 3425
+Wire Wire Line
+	1225 3425 1475 3425
+Connection ~ 1475 3425
 Connection ~ 1475 3275
 Wire Wire Line

Commit message: thermally compensated expo current source for VCA, pinch off resistor
Parts:
- removed Q3: BC557B, symbol pspice:QPNP
- removed R1: 10k, symbol Device:R
- removed R19: 1k, symbol Device:R
- added C2: 10n, symbol Device:C
- added Q10, Q9: BC557B, symbol pspice:QPNP
- added R26: 1.5Meg, symbol Device:R
- added R27: 100, symbol Device:R
- added R28: 100k, symbol Device:R
- added R29, R30: 2.2k, symbol Device:R
- added R555: 10k, symbol Device:R
- added U4: LM324, symbol pspice:OPAMP
- added V8: 2.5, symbol pspice:VSOURCE
- R21, R22: value 10k -> 100k
- R23: value 15k -> 10k
- R5: value 10k -> 100
- V3: value PULSE(-2 0 0 10m 10m 0.01m 20m) -> PULSE(2.4 2.5 0 10m 10m 0.01m 20m)
- V6: value 2 -> -2.55
- V7: renamed from V?; value -0.66 -> 2.6
- gave numbers to parts that had none: 2
Connections:
- net 0: now also R30.2, R555.2, U4.1 (+), V8.2 (E2)
- net VCC: now also R29.1, U4.4 (V+)
- net VEE: now also R26.2, R28.2, U4.5 (V-)
- net cv_pregain: now also Q10.2 (B)
- net R5bot: now reaches Q2.3 (E), Q4.3 (E), R5.2
- net R5bot: now also R555.1
- net R5top: now reaches R5.1
- net R5top: now also Q10.1 (C)
- net at Q1.1 (C), R13.1: now also R26.1
- new net: Q9.2 (B), R29.2, R30.1
- new net +2V5: V8.1 (E1)
- new net bla1: Q10.3 (E), Q9.3 (E), R27.2
- new net opamp: C2.1, R27.1, U4.3
- new net opampminus: C2.2, Q9.1 (C), R28.1, U4.2 (-)
Other:
- note added: ".temp 30\n.tran 1u 10m"
- note removed: ".tran 1u 10m"
- note removed: "current mirror as\nvoltage controlled\ncurrent source"
- moved on the sheet: R5, V3
