File: simulation/vca2/vca3.sch (KiCad schematic (older format))
At the start: 59 parts, among them Q1 PNP, Q2 PNP, Q3 PNP, Q4 PNP, Q5 PNP, Q6 PNP, Q7 PNP, Q8 PNP, U1 LM324, U2 LM324, U3 LM324, U4 LM324, U5 LM324, U6 LM324

Commit message: improved gain compensation
Parts:
- removed R16, R36, R37: 2.2k, symbol Device:R
- removed R?: 1k, symbol Device:R
- added Q9: PNP, symbol Device:Q_PNP_CBE
- added R22: 2.2k, symbol Device:R
- added R25: 22k, symbol Device:R
- added R40: 47k, symbol Device:R
- added U7: LM324, symbol pspice:OPAMP
- R17: value 2.2k -> 1k
- R18: value 470k -> 4.325k
- R20: value 1k -> 2k
- R38: value 1Meg -> 4.325k
Connections:
- net cv_pregain2_adj is gone; now on net VCC: R20.2
- net 0: now also U2.1 (+), U5.1 (+), Q9.3 (E), R22.1; no longer R17.1
- net VCC: now also U7.4 (V+); no longer R18.1, R38.1
- net VEE: now also R18.1, R38.1, U7.5 (V-)
- net cv_pregain2: now also U7.1 (+)
- net fnord2: now reaches R17.2
- net fnord2: now also Q9.1 (C), Q9.2 (B), R40.1; no longer U2.1 (+)
- net at R35.1, R38.2, R39.2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: now also R40.2; no longer R20.1
- new net: R20.1, R22.2, R25.1, U7.2 (-)
- new net fnord: R17.1, R25.2, U7.3
